Commit message: Reduce gaps in collisions

File: urdf/legs.xacro (robot description, xacro)
@@ -126,8 +126,8 @@
       <collision>
         <origin
-          xyz="-0.1 -0.075 -0.07"
+          xyz="-0.0975 -0.075 -0.07"
           rpy="0 ${PI/2} ${PI/4}" />
         <geometry>
-          <box size="0.025 0.05 0.135"/>
+          <box size="0.025 0.05 0.14"/>
         </geometry>
       </collision>
@@ -409,8 +409,8 @@
       <collision>
         <origin
-          xyz="-0.1 -0.075 +0.07"
+          xyz="-0.0975 -0.075 +0.07"
           rpy="0 ${PI/2} ${PI/4}" />
         <geometry>
-          <box size="0.025 0.05 0.135"/>
+          <box size="0.025 0.05 0.14"/>
         </geometry>
       </collision>

Commit message: Invert meshes of hind hips

File: urdf/legs.xacro (robot description, xacro)
@@ -30,4 +30,12 @@
           rpy="0 0 0" />
         <geometry>
+          <xacro:if value="${FH == 'F'}">
+            <mesh
+              filename="package://ayg_description/meshes/L_Hip.STL" />
+          </xacro:if>
+          <xacro:unless value="${FH == 'F'}">
+            <mesh
+              filename="package://ayg_description/meshes/R_Hip.STL" />
+          </xacro:unless>
           <mesh
             filename="package://ayg_description/meshes/L_Hip.STL" />
@@ -313,6 +321,12 @@
           rpy="0 0 0" />
         <geometry>
-          <mesh
-            filename="package://ayg_description/meshes/R_Hip.STL" />
+          <xacro:if value="${FH == 'F'}">
+            <mesh
+              filename="package://ayg_description/meshes/R_Hip.STL" />
+          </xacro:if>
+          <xacro:unless value="${FH == 'F'}">
+            <mesh
+              filename="package://ayg_description/meshes/L_Hip.STL" />
+          </xacro:unless>
         </geometry>
         <material

Commit message: Fix feet's visual geometry

File: urdf/legs.xacro (robot description, xacro)
@@ -261,5 +261,5 @@
           rpy="${PI/2} 0 0" />
         <geometry>
-          <sphere radius="0.030"/>
+          <cylinder length="0.025" radius="0.030"/>
         </geometry>
         <material
@@ -552,5 +552,5 @@
           rpy="${PI/2} 0 0" />
         <geometry>
-          <sphere radius="0.030"/>
+          <cylinder length="0.025" radius="0.030"/>
         </geometry>
         <material
