Commit message: Update meshes and xacro

File: urdf/ayg.xacro (robot description, xacro)
@@ -1,1114 +1,1114 @@
 <?xml version="1.0" encoding="utf-8"?>
 <robot name="ayg" xmlns:xacro="http://www.ros.org/wiki/xacro">
-	<xacro:arg name="use_gazebo" default="False" />
-	<xacro:property name="use_gazebo" default="$(arg use_gazebo)" />
-	<xacro:arg name="initial_configuration" default="lying_down" />
-	<xacro:property name="initial_configuration" value="$(arg initial_configuration)" />
-	<xacro:arg name="controller" default="default" />
-	<xacro:property name="controller" default="$(arg controller)" />
-	<xacro:property name="effort_lim" value="50.0" />
-	<xacro:property name="velocity_lim" value="10.0" />
-	<xacro:property name="PI" value="3.1415926535897931" />
-	<xacro:if value="${use_gazebo}">
-		<xacro:include filename="$(find ayg_description)/urdf/ayg_gazebo.xacro" />
-	</xacro:if>
-	<link
-		name="Base">
-		<inertial>
-			<origin
-				xyz="-4.4505E-17 9.7011E-18 -0.0030849"
-				rpy="0 0 0" />
-			<mass
-				value="5.6129" />
-			<inertia
-				ixx="0.010298"
-				ixy="-2.8049E-19"
-				ixz="-8.004E-19"
-				iyy="0.015742"
-				iyz="1.5043E-18"
-				izz="0.019645" />
-		</inertial>
-		<visual>
-			<origin
-				xyz="0 0 0"
-				rpy="0 0 0" />
-			<geometry>
-				<mesh
-					filename="package://ayg_description/meshes/Base.STL" />
-			</geometry>
-			<material
-				name="">
-				<color
-					rgba="0.69804 0.69804 0.69804 1" />
-			</material>
-		</visual>
-		<collision>
-			<origin
-				xyz="0 0 0"
-				rpy="0 0 0" />
-			<geometry>
-				<mesh
-					filename="package://ayg_description/meshes/Base.STL" />
-			</geometry>
-		</collision>
-	</link>
-	<link
-		name="LF_Hip">
-		<inertial>
-			<origin
-				xyz="0.071418 6.5097E-16 0.002654"
-				rpy="0 0 0" />
-			<mass
-				value="1.0061" />
-			<inertia
-				ixx="0.00057848"
-				ixy="-1.7535E-21"
-				ixz="3.7047E-21"
-				iyy="0.00058006"
-				iyz="8.655E-21"
-				izz="0.0010176" />
-		</inertial>
-		<visual>
-			<origin
-				xyz="0 0 0"
-				rpy="0 0 0" />
-			<geometry>
-				<mesh
-					filename="package://ayg_description/meshes/LF_Hip.STL" />
-			</geometry>
-			<material
-				name="">
-				<color
-					rgba="0.69804 0.69804 0.69804 1" />
-			</material>
-		</visual>
-		<collision>
-			<origin
-				xyz="0 0 0"
-				rpy="0 0 0" />
-			<geometry>
-				<mesh
-					filename="package://ayg_description/meshes/LF_Hip.STL" />
-			</geometry>
-		</collision>
-	</link>
-	<joint
-		name="LF_HAA"
-		type="revolute">
-		<origin
-			xyz="0.15192 0.054 0"
-			rpy="1.5708 0 0" />
-		<parent
-			link="Base" />
-		<child
-			link="LF_Hip" />
-		<axis
-			xyz="1 0 0" />
-		<limit
-			lower="-0.34907"
-			upper="0.17453"
-			effort="${effort_lim}"
-			velocity="${velocity_lim}" />
-	</joint>
-	<link
-		name="LF_Thigh">
-		<inertial>
-			<origin
-				xyz="-0.0079041 -0.006894 -0.04243"
-				rpy="0 0 0" />
-			<mass
-				value="1.1334" />
-			<inertia
-				ixx="0.0008397"
-				ixy="-0.00023737"
-				ixz="-1.4658E-09"
-				iyy="0.00084564"
-				iyz="-1.2252E-06"
-				izz="0.001546" />
-		</inertial>
-		<visual>
-			<origin
-				xyz="0 0 0"
-				rpy="0 0 0" />
-			<geometry>
-				<mesh
-					filename="package://ayg_description/meshes/LF_Thigh.STL" />
-			</geometry>
-			<material
-				name="">
-				<color
-					rgba="0.69804 0.69804 0.69804 1" />
-			</material>
-		</visual>
-		<collision>
-			<origin
-				xyz="0 0 0"
-				rpy="0 0 0" />
-			<geometry>
-				<mesh
-					filename="package://ayg_description/meshes/LF_Thigh.STL" />
-			</geometry>
-		</collision>
-	</link>
-	<joint
-		name="LF_HFE"
-		type="revolute">
-		<origin
-			xyz="0.077085 0 -0.017"
-			rpy="0 0 0" />
-		<parent
-			link="LF_Hip" />
-		<child
-			link="LF_Thigh" />
-		<axis
-			xyz="0 0 1" />
-		<limit
-			lower="-2.618"
-			upper="0.34907"
-			effort="${effort_lim}"
-			velocity="${velocity_lim}" />
-	</joint>
-	<link
-		name="LF_Shank">
-		<inertial>
-			<origin
-				xyz="0.070616 -0.05127 -0.0201"
-				rpy="0 0 0" />
-			<mass
-				value="0.058285" />
-			<inertia
-				ixx="0.00018414"
-				ixy="0.00018535"
-				ixz="9.8667E-20"
-				iyy="0.00020942"
-				iyz="-9.1978E-20"
-				izz="0.00039291" />
-		</inertial>
-		<visual>
-			<origin
-				xyz="0 0 0"
-				rpy="0 0 0" />
-			<geometry>
-				<mesh
-					filename="package://ayg_description/meshes/LF_Shank.STL" />
-			</geometry>
-			<material
-				name="">
-				<color
-					rgba="0.69804 0.69804 0.69804 1" />
-			</material>
-		</visual>
-		<collision>
-			<origin
-				xyz="0 0 0"
-				rpy="0 0 0" />
-			<geometry>
-				<mesh
-					filename="package://ayg_description/meshes/LF_Shank.STL" />
-			</geometry>
-		</collision>
-	</link>
-	<joint
-		name="LF_KFE"
-		type="revolute">
-		<origin
-			xyz="-0.1494 -0.16021 -0.0539"
-			rpy="0 0 0" />
-		<parent
-			link="LF_Thigh" />
-		<child
-			link="LF_Shank" />
-		<axis
-			xyz="0 0 1" />
-		<limit
-			lower="-0.43633"
-			upper="1.2217"
-			effort="${effort_lim}"
-			velocity="${velocity_lim}" />
-	</joint>
-	<link
-		name="LF_Foot">
-		<inertial>
-			<origin
-				xyz="0.012 0 -5.5511E-17"
-				rpy="0 0 0" />
-			<mass
-				value="0.088055" />
-			<inertia
-				ixx="4.0957E-05"
-				ixy="6.4789E-21"
-				ixz="1.0527E-20"
-				iyy="2.4705E-05"
-				iyz="-4.2352E-21"
-				izz="2.4705E-05" />
-		</inertial>
-		<visual>
-			<origin
-				xyz="0 0 0"
-				rpy="0 0 0" />
-			<geometry>
-				<cylinder length="0.025" radius="0.030" />
-			</geometry>
-			<material
-				name="">
-				<color
-					rgba="0.25098 0.25098 0.25098 1" />
-			</material>
-		</visual>
-		<collision>
-			<origin
-				xyz="0 0 0"
-				rpy="0 0 0" />
-			<geometry>
-				<cylinder length="0.025" radius="0.030" />
-			</geometry>
-		</collision>
-	</link>
-	<joint
-		name="LF_Shank_2_Foot"
-		type="fixed">
-		<origin
-			xyz="0.165 -0.151 -0.0201"
-			rpy="0 0 0" />
-		<parent
-			link="LF_Shank" />
-		<child
-			link="LF_Foot" />
-		<axis
-			xyz="0 0 0" />
-	</joint>
-	<link
-		name="RF_Hip">
-		<inertial>
-			<origin
-				xyz="0.0714175198878489 6.86607544823498E-16 0.00265399811396266"
-				rpy="0 0 0" />
-			<mass
-				value="1.00611999358686" />
-			<inertia
-				ixx="0.000578475326629041"
-				ixy="2.38284951842656E-20"
-				ixz="-4.58376353579811E-20"
-				iyy="0.000580062231241837"
-				iyz="-1.65786496242045E-21"
-				izz="0.00101761251741825" />
-		</inertial>
-		<visual>
-			<origin
-				xyz="0 0 0"
-				rpy="0 0 0" />
-			<geometry>
-				<mesh
-					filename="package://ayg_description/meshes/RF_Hip.STL" />
-			</geometry>
-			<material
-				name="">
-				<color
-					rgba="0.698039215686274 0.698039215686274 0.698039215686274 1" />
-			</material>
-		</visual>
-		<collision>
-			<origin
-				xyz="0 0 0"
-				rpy="0 0 0" />
-			<geometry>
-				<mesh
-					filename="package://ayg_description/meshes/RF_Hip.STL" />
-			</geometry>
-		</collision>
-	</link>
-	<joint
-		name="RF_HAA"
-		type="revolute">
-		<origin
-			xyz="0.15192 -0.054 0"
-			rpy="-1.5708 0 0" />
-		<parent
-			link="Base" />
-		<child
-			link="RF_Hip" />
-		<axis
-			xyz="1 0 0" />
-		<limit
-			lower="-0.17453"
-			upper="0.34907"
-			effort="${effort_lim}"
-			velocity="${velocity_lim}" />
-	</joint>
-	<link
-		name="RF_Thigh">
-		<inertial>
-			<origin
-				xyz="-0.00790410799025601 -0.00689399183089042 0.0424302203258587"
-				rpy="0 0 0" />
-			<mass
-				value="1.13336000773924" />
-			<inertia
-				ixx="0.000839701004100924"
-				ixy="-0.000237368706450857"
-				ixz="1.4657628001327E-09"
-				iyy="0.000845643609366733"
-				iyz="1.22524486883543E-06"
-				izz="0.00154598364653309" />
-		</inertial>
-		<visual>
-			<origin
-				xyz="0 0 0"
-				rpy="0 0 0" />
-			<geometry>
-				<mesh
-					filename="package://ayg_description/meshes/RF_Thigh.STL" />
-			</geometry>
-			<material
-				name="">
-				<color
-					rgba="0.698039215686274 0.698039215686274 0.698039215686274 1" />
-			</material>
-		</visual>
-		<collision>
-			<origin
-				xyz="0 0 0"
-				rpy="0 0 0" />
-			<geometry>
-				<mesh
-					filename="package://ayg_description/meshes/RF_Thigh.STL" />
-			</geometry>
-		</collision>
-	</link>
-	<joint
-		name="RF_HFE"
-		type="revolute">
-		<origin
-			xyz="0.077085 0 -0.017"
-			rpy="3.1416 0 0" />
-		<parent
-			link="RF_Hip" />
-		<child
-			link="RF_Thigh" />
-		<axis
-			xyz="0 0 1" />
-		<limit
-			lower="-0.34907"
-			upper="2.618"
-			effort="${effort_lim}"
-			velocity="${velocity_lim}" />
-	</joint>
-	<link
-		name="RF_Shank">
-		<inertial>
-			<origin
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
Commit message: Update camera + add argument to rviz launch file

File: urdf/ayg.xacro (robot description, xacro)
@@ -3,6 +3,6 @@
   <xacro:arg name="use_gazebo" default="False" />
   <xacro:property name="use_gazebo" default="$(arg use_gazebo)" />
-  <xacro:arg name="has_camera" default="False" />
-  <xacro:property name="has_camera" default="$(arg has_camera)" />
+  <xacro:arg name="camera" default="False" />
+  <xacro:property name="camera" default="$(arg camera)" />
   <xacro:arg name="initial_configuration" default="lying_down" />
   <xacro:property name="initial_configuration" value="$(arg initial_configuration)" />
@@ -99,5 +99,5 @@
   </joint>
   <xacro:include filename="$(find ayg_description)/urdf/legs.xacro" />
-  <xacro:if value="${has_camera}">
+  <xacro:if value="${camera}">
     <xacro:include filename="$(find ayg_description)/urdf/camera.xacro" />
   </xacro:if>

File: urdf/camera.xacro (robot description, xacro)
@@ -1,63 +1,19 @@
 <?xml version="1.0"?>
 <robot xmlns:xacro="http://www.ros.org/wiki/xacro">
-  <link
-    name="Neck">
-    <inertial>
-      <origin
-        xyz="0 0 0"
-        rpy="0 0 0" />
-      <mass
-        value="0" />
-      <inertia
-        ixx="0"
-        ixy="0"
-        ixz="0"
-        iyy="0"
-        iyz="0"
-        izz="0" />
-    </inertial>
-    <visual>
-      <origin
-        xyz="0 0 0"
-        rpy="0 0 0" />
-      <geometry>
-        <mesh
-          filename="package://ayg_description/meshes/Neck.STL" />
-      </geometry>
-      <material
-        name="">
-        <color
-          rgba="0.69804 0.69804 0.69804 1" />
-      </material>
-    </visual>
-  </link>
-  <joint
-    name="Base_2_Neck"
-    type="fixed">
-    <origin
-      xyz="0.2615 0 0.0249999999999999"
-      rpy="1.5707963267949 0 1.5707963267949" />
-    <parent
-      link="Base" />
-    <child
-      link="Neck" />
-    <axis
-      xyz="0 0 0" />
-  </joint>
   <link
     name="Camera">
     <inertial>
       <origin
-        xyz="7.0525E-18 -2.7756E-17 0.013"
+        xyz="0.027539 -0.0054988 -1.4524E-08"
         rpy="0 0 0" />
       <mass
-        value="0.16948" />
+        value="0.3912" />
       <inertia
-        ixx="2.085E-05"
-        ixy="5.6809E-20"
-        ixz="-7.2863E-20"
-        iyy="0.00020719"
-        iyz="3.3881E-21"
-        izz="0.00020895" />
+        ixx="0.00080723"
+        ixy="4.4453E-06"
+        ixz="-1.7833E-09"
+        iyy="0.00082275"
+        iyz="2.4795E-09"
+        izz="0.00010329" />
     </inertial>
     <visual>
@@ -72,24 +28,25 @@
         name="">
         <color
-          rgba="0.25098 0.25098 0.25098 1" />
+          rgba="0.69804 0.69804 0.69804 1" />
       </material>
     </visual>
     <collision>
       <origin
-        xyz="0 -0.0025 0"
-        rpy="-0.288975409992567 0 0" />
+        xyz="0 0 0"
+        rpy="0 0 0" />
       <geometry>
-        <box size="0.13 0.035 0.05"/>
+        <mesh
+          filename="package://ayg_description/meshes/Camera.STL" />
       </geometry>
     </collision>
   </link>
   <joint
-    name="Neck_2_Camera"
+    name="Base_2_Camera"
     type="fixed">
     <origin
-      xyz="0 0.0166603444360147 0.0804068913666247"
-      rpy="0.288975409992567 0 0" />
+      xyz="0.2475 0 0.095"
+      rpy="1.5708 0 0" />
     <parent
-      link="Neck" />
+      link="Base" />
     <child
       link="Camera" />

Commit message: Add ros2 control for hardware + change arg name

File: urdf/ayg.xacro (robot description, xacro)
@@ -1,6 +1,6 @@
 <?xml version="1.0" encoding="utf-8"?>
 <robot name="ayg" xmlns:xacro="http://www.ros.org/wiki/xacro">
-  <xacro:arg name="use_gazebo" default="False" />
-  <xacro:property name="use_gazebo" default="$(arg use_gazebo)" />
+  <xacro:arg name="sim" default="False" />
+  <xacro:property name="sim" default="$(arg sim)" />
   <xacro:arg name="camera" default="False" />
   <xacro:property name="camera" default="$(arg camera)" />
@@ -12,7 +12,16 @@
   <xacro:property name="velocity_lim" value="10.0" />
   <xacro:property name="PI" value="3.1415926535897931" />
-  <xacro:if value="${use_gazebo}">
+  <xacro:if value="${sim}">
     <xacro:include filename="$(find ayg_description)/urdf/ayg_gazebo.xacro" />
   </xacro:if>
+  <xacro:unless value="${sim}">
+    <xacro:include filename="$(find robstride_hardware)/urdf/robstride_ros2_control.xacro"/>
+    <xacro:robstride_ros2_control
+      can_interface="can0"
+      actuator_type="3"
+      default_kp="40.0"
+      default_kd="1.0"
+    />
+  </xacro:unless>
   <link
     name="Base">

File: urdf/ayg_gazebo.xacro (robot description, xacro)
@@ -62,5 +62,5 @@
         <gazebo>
             <plugin filename="libgz_ros2_control-system.so" name="gz_ros2_control::GazeboSimROS2ControlPlugin">
-                <parameters>$(find ayg_control)/config/gazebo/ayg_control.yaml</parameters>
+                <parameters>$(find ayg_control)/config/gazebo/ayg_sw_controllers.yaml</parameters>
             </plugin>
         </gazebo>

Commit message: Use macro for batteries

File: urdf/ayg.xacro (robot description, xacro)
@@ -60,4 +60,5 @@
         xyz="0.00057686 -0.00018498 0.0026529"
         rpy="0 0 0" />
+      <!-- Measured: 9.148 kg (CAD: 9.1298 kg) -->
       <mass
         value="9.148" />
@@ -137,73 +138,43 @@
       xyz="0 0 0" />
   </joint>
-  <!-- Batteries (2x, front-to-back inside body cavity, under top hatches) -->
-  <link name="Battery_Front">
-    <inertial>
-      <origin xyz="${battery_com_x} ${battery_com_y} ${battery_com_z}" rpy="0 0 0" />
-      <mass value="${battery_real_mass}" />
-      <inertia
-        ixx="${battery_cad_ixx * battery_inertia_scale}"
-        ixy="${battery_cad_ixy * battery_inertia_scale}"
-        ixz="${battery_cad_ixz * battery_inertia_scale}"
-        iyy="${battery_cad_iyy * battery_inertia_scale}"
-        iyz="${battery_cad_iyz * battery_inertia_scale}"
-        izz="${battery_cad_izz * battery_inertia_scale}" />
-    </inertial>
-    <visual>
-      <origin xyz="0 0 0" rpy="0 0 0" />
-      <geometry>
-        <box size="0.079 0.177 0.096" />
-      </geometry>
-      <material name="battery_color">
-        <color rgba="0.2 0.2 0.3 1" />
-      </material>
-    </visual>
-    <collision>
-      <origin xyz="0 0 0" rpy="0 0 0" />
-      <geometry>
-        <box size="0.079 0.177 0.096" />
-      </geometry>
-    </collision>
-  </link>
-  <joint name="Base_2_Battery_Front" type="fixed">
-    <origin xyz="${battery_front_x} 0 ${battery_pos_z}" rpy="0 0 0" />
-    <parent link="Base" />
-    <child link="Battery_Front" />
-    <axis xyz="0 0 0" />
-  </joint>
-  <link name="Battery_Rear">
-    <inertial>
-      <origin xyz="${battery_com_x} ${battery_com_y} ${battery_com_z}" rpy="0 0 0" />
-      <mass value="${battery_real_mass}" />
-      <inertia
-        ixx="${battery_cad_ixx * battery_inertia_scale}"
-        ixy="${battery_cad_ixy * battery_inertia_scale}"
-        ixz="${battery_cad_ixz * battery_inertia_scale}"
-        iyy="${battery_cad_iyy * battery_inertia_scale}"
-        iyz="${battery_cad_iyz * battery_inertia_scale}"
-        izz="${battery_cad_izz * battery_inertia_scale}" />
-    </inertial>
-    <visual>
-      <origin xyz="0 0 0" rpy="0 0 0" />
-      <geometry>
-        <box size="0.079 0.177 0.096" />
-      </geometry>
-      <material name="battery_color">
-        <color rgba="0.2 0.2 0.3 1" />
-      </material>
-    </visual>
-    <collision>
-      <origin xyz="0 0 0" rpy="0 0 0" />
-      <geometry>
-        <box size="0.079 0.177 0.096" />
-      </geometry>
-    </collision>
-  </link>
-  <joint name="Base_2_Battery_Rear" type="fixed">
-    <origin xyz="${battery_rear_x} 0 ${battery_pos_z}" rpy="0 0 0" />
-    <parent link="Base" />
-    <child link="Battery_Rear" />
-    <axis xyz="0 0 0" />
-  </joint>
+  <!-- Battery macro (2x identical packs, front and rear) -->
+  <xacro:macro name="battery" params="name pos_x">
+    <link name="Battery_${name}">
+      <inertial>
+        <origin xyz="${battery_com_x} ${battery_com_y} ${battery_com_z}" rpy="0 0 0" />
+        <mass value="${battery_real_mass}" />
+        <inertia
+          ixx="${battery_cad_ixx * battery_inertia_scale}"
+          ixy="${battery_cad_ixy * battery_inertia_scale}"
+          ixz="${battery_cad_ixz * battery_inertia_scale}"
+          iyy="${battery_cad_iyy * battery_inertia_scale}"
+          iyz="${battery_cad_iyz * battery_inertia_scale}"
+          izz="${battery_cad_izz * battery_inertia_scale}" />
+      </inertial>
+      <visual>
+        <origin xyz="0 0 0" rpy="0 0 0" />
+        <geometry>
+          <box size="0.079 0.177 0.096" />
+        </geometry>
+        <material name="battery_color">
+          <color rgba="0.2 0.2 0.3 1" />
+        </material>
+      </visual>
+      <collision>
+        <origin xyz="0 0 0" rpy="0 0 0" />
+        <geometry>
+          <box size="0.079 0.177 0.096" />
+        </geometry>
+      </collision>
+    </link>
+    <joint name="Base_2_Battery_${name}" type="fixed">
+      <origin xyz="${pos_x} 0 ${battery_pos_z}" rpy="0 0 0" />
+      <parent link="Base" />
+      <child link="Battery_${name}" />
+      <axis xyz="0 0 0" />
+    </joint>
+  </xacro:macro>
+  <xacro:battery name="Front" pos_x="${battery_front_x}" />
+  <xacro:battery name="Rear"  pos_x="${battery_rear_x}" />
   <xacro:include filename="$(find ayg_description)/urdf/legs.xacro" />
   <xacro:if value="${camera}">

Commit message: Add arg for gazebo version

File: urdf/ayg.xacro (robot description, xacro)
@@ -5,4 +5,6 @@
   <xacro:arg name="sim_backend" default="gazebo" />
   <xacro:property name="sim_backend" value="$(arg sim_backend)" />
+  <xacro:arg name="gazebo_version" default="fortress" />
+  <xacro:property name="gazebo_version" value="$(arg gazebo_version)" />
   <xacro:arg name="camera" default="False" />
   <xacro:property name="camera" default="$(arg camera)" />

File: urdf/ayg_sim_ros2_control.xacro (robot description, xacro)
@@ -87,16 +87,33 @@
             </gazebo>
         </xacro:if>
-        <gazebo>
-            <plugin filename="gz-sim-odometry-publisher-system" name="gz::sim::systems::OdometryPublisher">
-                <odom_frame>Base</odom_frame>
-                <robot_base_frame>Base</robot_base_frame>
-                <odom_publish_frequency>500</odom_publish_frequency>
-                <dimensions>3</dimensions>
-            </plugin>
-        </gazebo>
-        <gazebo>
-            <plugin filename="gz-sim-imu-system" name="gz::sim::systems::Imu">
-            </plugin>
-        </gazebo>
+        <xacro:if value="${gazebo_version == 'fortress'}">
+            <gazebo>
+                <plugin filename="ignition-gazebo-odometry-publisher-system"
+                        name="ignition::gazebo::systems::OdometryPublisher">
+                    <odom_frame>Base</odom_frame>
+                    <robot_base_frame>Base</robot_base_frame>
+                    <odom_publish_frequency>500</odom_publish_frequency>
+                    <dimensions>3</dimensions>
+                </plugin>
+            </gazebo>
+            <gazebo>
+                <plugin filename="ignition-gazebo-imu-system"
+                        name="ignition::gazebo::systems::Imu"/>
+            </gazebo>
+        </xacro:if>
+        <xacro:unless value="${gazebo_version == 'fortress'}">
+            <gazebo>
+                <plugin filename="gz-sim-odometry-publisher-system" name="gz::sim::systems::OdometryPublisher">
+                    <odom_frame>Base</odom_frame>
+                    <robot_base_frame>Base</robot_base_frame>
+                    <odom_publish_frequency>500</odom_publish_frequency>
+                    <dimensions>3</dimensions>
+                </plugin>
+            </gazebo>
+            <gazebo>
+                <plugin filename="gz-sim-imu-system" name="gz::sim::systems::Imu">
+                </plugin>
+            </gazebo>
+        </xacro:unless>
         <gazebo reference="Base">
             <sensor name="imu_sensor" type="imu">
