Commit message: feat: certification-grade MuJoCo plant — armature, handles, RS-03 motor-curve params
- mujoco/ayg.xml: joint armature 0.02 (the certified mujoco_val value; 0 was the
  documented snap/fail sim2sim gap) + handle_F/handle_R collision meshes, matching
  the cf_lab validation model (full-diff verified physically identical).
- ayg.xacro + ayg_sim_ros2_control.xacro: motor_curve / motor_curve_tau /
  motor_curve_tau_knee args -> MujocoSystem hardware params (RS-03 four-quadrant
  torque-speed curve; tau follows the controller clamp: 20/16 cert, 30/30 HW plan).

File: urdf/ayg.xacro (robot description, xacro)
@@ -18,4 +18,15 @@
   <xacro:arg name="publish_current" default="false" />
   <xacro:property name="publish_current" value="$(arg publish_current)" />
+  <!-- MuJoCo backend only: enable the RS-03 four-quadrant torque-speed curve in the plant
+       (the certification-condition velocity envelope). Off by default so walking sims keep
+       their historical plant; recovery rehearsals should pass motor_curve:=true. -->
+  <xacro:arg name="motor_curve" default="false" />
+  <xacro:property name="motor_curve" value="$(arg motor_curve)" />
+  <!-- Per-joint clamp used inside the curve math — keep in sync with the controller's
+       effort limits (cert condition 20/16, planned HW config 30/30). -->
+  <xacro:arg name="motor_curve_tau" default="20.0" />
+  <xacro:property name="motor_curve_tau" value="$(arg motor_curve_tau)" />
+  <xacro:arg name="motor_curve_tau_knee" default="16.0" />
+  <xacro:property name="motor_curve_tau_knee" value="$(arg motor_curve_tau_knee)" />
   <xacro:property name="effort_lim" value="30.0" />
   <xacro:property name="velocity_lim" value="18.849" />

File: urdf/ayg_sim_ros2_control.xacro (robot description, xacro)
@@ -28,4 +28,13 @@
             <xacro:if value="${sim_backend == 'mujoco'}">
                 <param name="mujoco_model_path">$(find ayg_description)/mujoco/ayg.xml</param>
+                <xacro:if value="${motor_curve}">
+                    <!-- RS-03 four-quadrant curve = certification plant (mujoco_val
+                         eval_phased_recovery with vcap 20 + motor_curve, tau 20/16). -->
+                    <param name="motor_curve">true</param>
+                    <param name="motor_curve_vcap">20.0</param>
+                    <param name="motor_curve_tau_sat">60.0</param>
+                    <param name="motor_curve_tau">${motor_curve_tau}</param>
+                    <param name="motor_curve_tau_knee">${motor_curve_tau_knee}</param>
+                </xacro:if>
             </xacro:if>
         </hardware>

Commit message: Add model_version tag

File: urdf/ayg.xacro (robot description, xacro)
@@ -17,4 +17,6 @@
   <xacro:property name="velocity_lim" value="10.0" />
   <xacro:property name="PI" value="3.1415926535897931" />
+  <xacro:property name="model_version" value="1.3" />
+  <model_version>${model_version}</model_version>
   <!-- Battery inertial properties (CAD export → URDF frame)
        CAD frame: X=forward, Y=up, Z=left  |  URDF frame: X=forward, Y=left, Z=up

Commit message: camera: gate the sim stereo IR pair on a stereo_ir arg; fix stale script refs

File: urdf/ayg.xacro (robot description, xacro)
@@ -9,4 +9,12 @@
   <xacro:arg name="camera" default="True" />
   <xacro:property name="camera" default="$(arg camera)" />
+  <!--
+    Simulated stereo IR pair (the cuVSLAM input). Off by default: two extra
+    640x360 renderers at 30 Hz cost real gz frame time, and only Visual SLAM
+    consumes them. ayg_gazebo passes stereo_ir:=true when enable_vslam:=true.
+    Only meaningful with camera:=true and sim:=true.
+  -->
+  <xacro:arg name="stereo_ir" default="False" />
+  <xacro:property name="stereo_ir" default="$(arg stereo_ir)" />
   <xacro:arg name="initial_configuration" default="lying_down" />
   <xacro:property name="initial_configuration" value="$(arg initial_configuration)" />

File: urdf/camera.xacro (robot description, xacro)
@@ -210,5 +210,5 @@
           of the configured 640x360/87deg. NOTE gz applies this only to the K
           matrix, not P; a small republisher copies K->P (ayg_gazebo
-          fix_depth_camera_info.py + depth_cloud.launch.py) so depth_image_proc
+          fix_camera_info.py + depth_cloud.launch.py) so depth_image_proc
           and RViz reconstruct an aligned point cloud.
           fx=fy=(width/2)/tan(hfov/2)=337.2, cx=width/2, cy=height/2.
@@ -317,7 +317,7 @@
     Topic names match real hardware (realsense2_camera, camera_name=Camera,
     enable_infra1/2): /camera/Camera/infra{1,2}/image_rect_raw. gz leaves
-    CameraInfo.P at its default, so ayg_gazebo's stereo_camera_info node fixes P
-    up and writes the right camera's Tx = -fx * baseline — see
-    ayg_gazebo/scripts/fix_depth_camera_info.py.
+    CameraInfo.P at its default, so ayg_gazebo's stereo_camera_info.launch.py
+    fixes P up and writes the right camera's Tx = -fx * baseline — see
+    ayg_gazebo/scripts/fix_camera_info.py.
     The real projector must be OFF for stereo VO (its dot pattern is a
     camera-fixed texture that corrupts feature tracking); in sim there is no
@@ -358,10 +358,19 @@
     </gazebo>
   </xacro:macro>
-  <xacro:infra_sensor name="infra1"
-                      frame="Camera_infra1_frame"
-                      optical_frame="Camera_infra1_optical_frame"/>
-  <xacro:infra_sensor name="infra2"
-                      frame="Camera_infra2_frame"
-                      optical_frame="Camera_infra2_optical_frame"/>
+  <!--
+    Gated on its own arg, not on `camera`: two extra 640x360 renderers at 30 Hz
+    is a real cost in gz, and only cuVSLAM consumes them. ayg_gazebo turns this
+    on when enable_vslam:=true, so a depth-only sim run does not pay for it. The
+    infra *frames* above stay unconditional: massless frames are free, and
+    keeping them means the TF tree matches hardware either way.
+  -->
+  <xacro:if value="${stereo_ir}">
+    <xacro:infra_sensor name="infra1"
+                        frame="Camera_infra1_frame"
+                        optical_frame="Camera_infra1_optical_frame"/>
+    <xacro:infra_sensor name="infra2"
+                        frame="Camera_infra2_frame"
+                        optical_frame="Camera_infra2_optical_frame"/>
+  </xacro:if>
   </xacro:if>
 </robot>

Commit message: Drop the inert gazebo_version fortress/harmonic switch
Applies origin/main's 951ab48 to the shared sim_ros2_control.xacro,
which my restructure had carried over from the pre-951ab48 1.3 branch.
On this branch the switch was NOT inert: its default (gazebo_version
fortress) emitted Ignition-era plugin names (ignition-gazebo-*) on
both 1.2 and 1.3, breaking odometry and IMU on the Harmonic/Jazzy
platform this now targets. Collapse to the single gz-sim-* block and
drop the gazebo_version arg/property.

File: urdf/ayg.xacro (robot description, xacro)
@@ -5,6 +5,4 @@
   <xacro:arg name="sim_backend" default="gazebo" />
   <xacro:property name="sim_backend" value="$(arg sim_backend)" />
-  <xacro:arg name="gazebo_version" default="fortress" />
-  <xacro:property name="gazebo_version" value="$(arg gazebo_version)" />
   <!-- Which Ayg model to build: "1.2" or "1.3". Selects the whole per-version
        subtree (root xacro, legs, meshes, mujoco/rviz configs) - see the

File: urdf/sim_ros2_control.xacro (robot description, xacro)
@@ -65,33 +65,15 @@
             </gazebo>
         </xacro:if>
-        <xacro:if value="${gazebo_version == 'fortress'}">
-            <gazebo>
-                <plugin filename="ignition-gazebo-odometry-publisher-system"
-                        name="ignition::gazebo::systems::OdometryPublisher">
-                    <odom_frame>Base</odom_frame>
-                    <robot_base_frame>Base</robot_base_frame>
-                    <odom_publish_frequency>500</odom_publish_frequency>
-                    <dimensions>3</dimensions>
-                </plugin>
-            </gazebo>
-            <gazebo>
-                <plugin filename="ignition-gazebo-imu-system"
-                        name="ignition::gazebo::systems::Imu"/>
-            </gazebo>
-        </xacro:if>
-        <xacro:unless value="${gazebo_version == 'fortress'}">
-            <gazebo>
-                <plugin filename="gz-sim-odometry-publisher-system" name="gz::sim::systems::OdometryPublisher">
-                    <odom_frame>Base</odom_frame>
-                    <robot_base_frame>Base</robot_base_frame>
-                    <odom_publish_frequency>500</odom_publish_frequency>
-                    <dimensions>3</dimensions>
-                </plugin>
-            </gazebo>
-            <gazebo>
-                <plugin filename="gz-sim-imu-system" name="gz::sim::systems::Imu">
-                </plugin>
-            </gazebo>
-        </xacro:unless>
+        <gazebo>
+            <plugin filename="gz-sim-odometry-publisher-system" name="gz::sim::systems::OdometryPublisher">
+                <odom_frame>Base</odom_frame>
+                <robot_base_frame>Base</robot_base_frame>
+                <odom_publish_frequency>500</odom_publish_frequency>
+                <dimensions>3</dimensions>
+            </plugin>
+        </gazebo>
+        <gazebo>
+            <plugin filename="gz-sim-imu-system" name="gz::sim::systems::Imu"/>
+        </gazebo>
         <gazebo reference="Base">
             <sensor name="imu_sensor" type="imu">
