Commit message: Tune MuJoCo contact params and add sim_backend support to xacro
- Increase foot/floor friction and use condim=6 with noslip solver
  for stable ground contact
- Change foot collision from sphere to cylinder for flatter contact
- Lower spawn height to 0.18m (closer to standing)
- Add sim_backend xacro arg to select gazebo or mujoco ros2_control
- Add .gitignore for MuJoCo runtime artifacts

Co-Authored-By: Claude Opus 4.6 (1M context) <noreply@anthropic.com>

File: urdf/ayg.xacro (robot description, xacro)
@@ -3,4 +3,6 @@
   <xacro:arg name="sim" default="False" />
   <xacro:property name="sim" default="$(arg sim)" />
+  <xacro:arg name="sim_backend" default="gazebo" />
+  <xacro:property name="sim_backend" value="$(arg sim_backend)" />
   <xacro:arg name="camera" default="False" />
   <xacro:property name="camera" default="$(arg camera)" />
@@ -12,6 +14,13 @@
   <xacro:property name="velocity_lim" value="10.0" />
   <xacro:property name="PI" value="3.1415926535897931" />
-  <xacro:if value="${sim}">
+  <xacro:if value="${sim and sim_backend == 'gazebo'}">
     <xacro:include filename="$(find ayg_description)/urdf/ayg_gazebo.xacro" />
+  </xacro:if>
+  <xacro:if value="${sim and sim_backend == 'mujoco'}">
+    <xacro:include filename="$(find ayg_mujoco)/urdf/ayg_mujoco_ros2_control.xacro" />
+    <xacro:ayg_mujoco_ros2_control
+      mujoco_model_path="$(find ayg_description)/mujoco/ayg.xml"
+      use_viewer="true"
+    />
   </xacro:if>
   <xacro:unless value="${sim}">

Commit message: Add MuJoCo-compatible XML robot description (#4)
* Add MuJoCo-compatible XML robot description

Convert URDF to MuJoCo MJCF format with:
- Floating base (freejoint) for simulation
- Ground plane with checker texture
- 12 torque actuators matching URDF effort limits
- IMU (accelerometer + gyro), foot touch, joint pos/vel sensors
- Visual STL meshes (Base, Hip, Thigh, Shank) separated from
  collision primitives (group 1 vs group 3)
- Camera visual mesh at front of base
- Foot visual cylinders matching URDF

Co-Authored-By: Claude Opus 4.6 (1M context) <noreply@anthropic.com>

* Tune MuJoCo contact params and add sim_backend support to xacro

- Increase foot/floor friction and use condim=6 with noslip solver
  for stable ground contact
- Change foot collision from sphere to cylinder for flatter contact
- Lower spawn height to 0.18m (closer to standing)
- Add sim_backend xacro arg to select gazebo or mujoco ros2_control
- Add .gitignore for MuJoCo runtime artifacts

Co-Authored-By: Claude Opus 4.6 (1M context) <noreply@anthropic.com>

* Reduce joint damping and armature for more responsive control

Co-Authored-By: Claude Opus 4.6 (1M context) <noreply@anthropic.com>

* Adjust joint damping and armature for stable simulation

Co-Authored-By: Claude Opus 4.6 (1M context) <noreply@anthropic.com>

* Remove joint damping and armature to match Isaac Lab training config

Co-Authored-By: Claude Opus 4.6 (1M context) <noreply@anthropic.com>

* Remove unused arg

* Unify gazebo and mujoco ros2_control xacro files

---------

Co-authored-by: Davide De Benedittis <davide.debenedittis@gmail.com>

File: urdf/ayg.xacro (robot description, xacro)
@@ -3,4 +3,6 @@
   <xacro:arg name="sim" default="False" />
   <xacro:property name="sim" default="$(arg sim)" />
+  <xacro:arg name="sim_backend" default="gazebo" />
+  <xacro:property name="sim_backend" value="$(arg sim_backend)" />
   <xacro:arg name="camera" default="False" />
   <xacro:property name="camera" default="$(arg camera)" />
@@ -14,5 +16,5 @@
   <xacro:property name="PI" value="3.1415926535897931" />
   <xacro:if value="${sim}">
-    <xacro:include filename="$(find ayg_description)/urdf/ayg_gazebo.xacro" />
+    <xacro:include filename="$(find ayg_description)/urdf/ayg_sim_ros2_control.xacro" />
   </xacro:if>
   <xacro:unless value="${sim}">

Commit message: fix: model fidelity for RL fall-recovery sim-to-sim transfer
Three changes that align the Gazebo/URDF model with the cf_lab Isaac
training model, fixing failed recovery-policy transfer:

- ayg.xacro: add Battery_Front/Rear inertial links (2x1.6 kg, fixed to
  Base). They were missing here, leaving the base ~3.2 kg light (~35% of
  base-body mass) with ~half the pitch inertia. Also correct joint limits
  to the RS-03 datasheet: effort 50->30 N.m, velocity 10->18.849 rad/s.
- legs.xacro: add joint Coulomb friction 0.2 (damping 0.0) on all 12
  leg joints, matching the training actuator friction.
- ayg_gazebo.xacro: add contact friction mu=1.0 on the links that touch
  the ground during a belly-up flip (Base, thighs, shanks, feet). The
  collisions previously had no friction spec, so the robot slid instead
  of gripping to push upright. Matches Isaac ground static_friction=1.0.

Co-Authored-By: Claude Opus 4.8 (1M context) <noreply@anthropic.com>

File: urdf/ayg.xacro (robot description, xacro)
@@ -9,6 +9,6 @@
   <xacro:arg name="controller" default="default" />
   <xacro:property name="controller" default="$(arg controller)" />
-  <xacro:property name="effort_lim" value="50.0" />
-  <xacro:property name="velocity_lim" value="10.0" />
+  <xacro:property name="effort_lim" value="30.0" />
+  <xacro:property name="velocity_lim" value="18.849" />
   <xacro:property name="PI" value="3.1415926535897931" />
   <xacro:if value="${sim}">
@@ -63,4 +63,36 @@
     </collision>
   </link>
+  <!-- Battery packs (fixed to Base). Present in the cf_lab training model but were
+       missing here, leaving the Gazebo/real base ~3.2 kg light (~35% of base-body mass)
+       with ~half the pitch inertia, which broke RL fall-recovery transfer. Inertial-only
+       (no visual/collision: they sit inside the Base collision box). -->
+  <link name="Battery_Front">
+    <inertial>
+      <origin rpy="0 0 0" xyz="-0.00002 -0.00421 0.04143" />
+      <mass value="1.6" />
+      <inertia ixx="0.0044576" ixy="-4.1873E-06" ixz="-5.2038E-06"
+               iyy="0.0076771" iyz="-0.00026672" izz="0.0044479" />
+    </inertial>
+  </link>
+  <joint name="Base_2_Battery_Front" type="fixed">
+    <origin rpy="0 0 0" xyz="0.10070 0 -0.00900" />
+    <parent link="Base" />
+    <child link="Battery_Front" />
+    <axis xyz="0 0 0" />
+  </joint>
+  <link name="Battery_Rear">
+    <inertial>
+      <origin rpy="0 0 0" xyz="-0.00002 -0.00421 0.04143" />
+      <mass value="1.6" />
+      <inertia ixx="0.0044576" ixy="-4.1873E-06" ixz="-5.2038E-06"
+               iyy="0.0076771" iyz="-0.00026672" izz="0.0044479" />
+    </inertial>
+  </link>
+  <joint name="Base_2_Battery_Rear" type="fixed">
+    <origin rpy="0 0 0" xyz="-0.10070 0 -0.00900" />
+    <parent link="Base" />
+    <child link="Battery_Rear" />
+    <axis xyz="0 0 0" />
+  </joint>
   <link
     name="IMU">

File: urdf/ayg_gazebo.xacro (robot description, xacro)
@@ -148,3 +148,26 @@
         </sensor>
     </gazebo>
+    <!-- Contact friction: the robot collisions had NO friction spec, so during RL fall-recovery
+         the body/legs slid on the floor instead of gripping to push upright. Set ~1.0 to match the
+         Isaac training ground friction (static_friction=1.0). Covers the links that contact the
+         ground during a belly-up flip (body, thighs, shanks, feet). -->
+    <xacro:macro name="ground_friction" params="link">
+        <gazebo reference="${link}">
+            <mu1>1.0</mu1>
+            <mu2>1.0</mu2>
+        </gazebo>
+    </xacro:macro>
+    <xacro:ground_friction link="Base"/>
+    <xacro:ground_friction link="LF_Foot"/>
+    <xacro:ground_friction link="LH_Foot"/>
+    <xacro:ground_friction link="RF_Foot"/>
+    <xacro:ground_friction link="RH_Foot"/>
+    <xacro:ground_friction link="LF_Shank"/>
+    <xacro:ground_friction link="LH_Shank"/>
+    <xacro:ground_friction link="RF_Shank"/>
+    <xacro:ground_friction link="RH_Shank"/>
+    <xacro:ground_friction link="LF_Thigh"/>
+    <xacro:ground_friction link="LH_Thigh"/>
+    <xacro:ground_friction link="RF_Thigh"/>
+    <xacro:ground_friction link="RH_Thigh"/>
 </robot>

File: urdf/legs.xacro (robot description, xacro)
@@ -101,4 +101,5 @@
           velocity="${velocity_lim}" />
       </xacro:unless>
+      <dynamics damping="0.0" friction="0.2"/>
     </joint>
     <link
@@ -174,4 +175,5 @@
           velocity="${velocity_lim}" />
       </xacro:unless>
+      <dynamics damping="0.0" friction="0.2"/>
     </joint>
     <link
@@ -239,4 +241,5 @@
         effort="${effort_lim}"
         velocity="${velocity_lim}" />
+      <dynamics damping="0.0" friction="0.2"/>
     </joint>
     <link
@@ -392,4 +395,5 @@
           velocity="${velocity_lim}" />
       </xacro:unless>
+      <dynamics damping="0.0" friction="0.2"/>
     </joint>
     <link
@@ -465,4 +469,5 @@
           velocity="${velocity_lim}" />
       </xacro:unless>
+      <dynamics damping="0.0" friction="0.2"/>
     </joint>
     <link
@@ -530,4 +535,5 @@
         effort="${effort_lim}"
         velocity="${velocity_lim}" />
+      <dynamics damping="0.0" friction="0.2"/>
     </joint>
     <link

Commit message: feat: handle-collision model + publish_current arg for recovery HW deploy
Add the top-mounted carry handles (handle_F/handle_R, collision-only exact-CAD
meshes on the Base link) so the deployment model matches the hd_ctrl_s1 training
model — the robot physically has these handles and they change belly-up recovery
contact. Propagated from cf_lab ayg_description@f09472e (branch handle-collision),
which was never pushed to origin (the cf_lab<->Ayg divergence).

Also thread the publish_current xacro arg/property through to the robstride macro
(default false) to pair with the motor_states current/effort work in the Ayg repo.

Co-Authored-By: Claude Opus 4.8 (1M context) <noreply@anthropic.com>

File: urdf/ayg.xacro (robot description, xacro)
@@ -9,4 +9,8 @@
   <xacro:arg name="controller" default="default" />
   <xacro:property name="controller" default="$(arg controller)" />
+  <!-- Hardware measurement mode: publish per-motor q-axis current on motor_states.
+       Off by default; enable only for HW fidelity measurement runs (see recovery_hw). -->
+  <xacro:arg name="publish_current" default="false" />
+  <xacro:property name="publish_current" value="$(arg publish_current)" />
   <xacro:property name="effort_lim" value="30.0" />
   <xacro:property name="velocity_lim" value="18.849" />
@@ -24,4 +28,5 @@
       default_kp="40.0"
       default_kd="1.0"
+      publish_current="${publish_current}"
       calibration_file="$(find robstride_hardware)/calibration/joint_calibration.yaml"
     />
@@ -63,4 +68,21 @@
       <geometry>
         <box size="0.4 0.23 0.12" />
+      </geometry>
+    </collision>
+    <!-- Top-mounted carry handles — EXACT CAD collision mesh (two end arches extracted
+         from Base.STL; handle_F front, handle_R rear, each PhysX convex-hulled). Collision
+         ONLY (mass already in Base). Propagated from cf_lab ayg_description@f09472e
+         (branch handle-collision) so the deployment model matches the hd_ctrl_s1 training
+         model — the robot physically has these handles and they change belly-up contact. -->
+    <collision>
+      <origin xyz="0 0 0" rpy="0 0 0" />
+      <geometry>
+        <mesh filename="package://ayg_description/meshes/handle_F.STL" />
+      </geometry>
+    </collision>
+    <collision>
+      <origin xyz="0 0 0" rpy="0 0 0" />
+      <geometry>
+        <mesh filename="package://ayg_description/meshes/handle_R.STL" />
       </geometry>
     </collision>

Commit message: feat: top-handle collision model + recovery joint limits + publish_current
For recovery deployment on the real robot (which has the top-mounted carry handles):

- Top-handle collision (handle_F/handle_R, collision-only exact-CAD meshes on the
  Base link) so the model matches the handle-trained recovery policy.
- Recovery joint limits: velocity_lim 10 -> 18.849 rad/s, effort_lim 50 -> 30 N*m.
  velocity_lim=10 is a placeholder the Gazebo/ros2_control stack OBEYS, clamping
  joints below the ~15.25 rad/s recovery needs. 18.849/30 match the trained model.
- publish_current xacro arg -> robstride_ros2_control macro (default false).

Cross-repo: publish_current pass-through needs the robstride_hardware macro param
(Ayg branch hardware-deployment).

Co-Authored-By: Claude Opus 4.8 (1M context) <noreply@anthropic.com>

File: urdf/ayg.xacro (robot description, xacro)
@@ -14,6 +14,10 @@
   <xacro:property name="controller" default="$(arg controller)" />
   <xacro:arg name="use_csp" default="false" />
-  <xacro:property name="effort_lim" value="50.0" />
-  <xacro:property name="velocity_lim" value="10.0" />
+  <!-- Hardware measurement mode: publish per-motor q-axis current on motor_states.
+       Off by default; enable only for HW fidelity measurement runs (see recovery_hw). -->
+  <xacro:arg name="publish_current" default="false" />
+  <xacro:property name="publish_current" value="$(arg publish_current)" />
+  <xacro:property name="effort_lim" value="30.0" />
+  <xacro:property name="velocity_lim" value="18.849" />
   <xacro:property name="PI" value="3.1415926535897931" />
   <!-- Battery inertial properties (CAD export → URDF frame)
@@ -53,4 +57,5 @@
       default_kd="1.0"
       use_csp="$(arg use_csp)"
+      publish_current="${publish_current}"
       calibration_file="$(find robstride_hardware)/calibration/joint_calibration.yaml"
     />
@@ -93,4 +98,21 @@
       <geometry>
         <box size="0.4 0.23 0.12" />
+      </geometry>
+    </collision>
+    <!-- Top-mounted carry handles — EXACT CAD collision mesh (two end arches extracted
+         from Base.STL; handle_F front, handle_R rear, each PhysX convex-hulled). Collision
+         ONLY (mass already in Base). Propagated from cf_lab ayg_description@f09472e
+         (branch handle-collision) so the deployment model matches the hd_ctrl_s1 training
+         model — the robot physically has these handles and they change belly-up contact. -->
+    <collision>
+      <origin xyz="0 0 0" rpy="0 0 0" />
+      <geometry>
+        <mesh filename="package://ayg_description/meshes/handle_F.STL" />
+      </geometry>
+    </collision>
+    <collision>
+      <origin xyz="0 0 0" rpy="0 0 0" />
+      <geometry>
+        <mesh filename="package://ayg_description/meshes/handle_R.STL" />
       </geometry>
     </collision>

Commit message: urdf: drop the inert gazebo_version switch
The fortress/harmonic branches in ayg_sim_ros2_control.xacro were
byte-identical — the fortress arm never carried Ignition-era plugin names,
so the switch has been a no-op duplication since it was added, and the
platform is Harmonic-only (Jazzy) now anyway. Collapse to one block and
remove the never-passed gazebo_version arg and its README entry.

Co-Authored-By: Claude Fable 5 <noreply@anthropic.com>

File: urdf/ayg.xacro (robot description, xacro)
@@ -5,6 +5,4 @@
   <xacro:arg name="sim_backend" default="gazebo" />
   <xacro:property name="sim_backend" value="$(arg sim_backend)" />
-  <xacro:arg name="gazebo_version" default="fortress" />
-  <xacro:property name="gazebo_version" value="$(arg gazebo_version)" />
   <xacro:arg name="camera" default="True" />
   <xacro:property name="camera" default="$(arg camera)" />

File: urdf/ayg_sim_ros2_control.xacro (robot description, xacro)
@@ -87,33 +87,15 @@
             </gazebo>
         </xacro:if>
-        <xacro:if value="${gazebo_version == 'fortress'}">
-            <gazebo>
-                <plugin filename="gz-sim-odometry-publisher-system"
-                        name="gz::sim::systems::OdometryPublisher">
-                    <odom_frame>Base</odom_frame>
-                    <robot_base_frame>Base</robot_base_frame>
-                    <odom_publish_frequency>500</odom_publish_frequency>
-                    <dimensions>3</dimensions>
-                </plugin>
-            </gazebo>
-            <gazebo>
-                <plugin filename="gz-sim-imu-system"
-                        name="gz::sim::systems::Imu"/>
-            </gazebo>
-        </xacro:if>
-        <xacro:unless value="${gazebo_version == 'fortress'}">
-            <gazebo>
-                <plugin filename="gz-sim-odometry-publisher-system" name="gz::sim::systems::OdometryPublisher">
-                    <odom_frame>Base</odom_frame>
-                    <robot_base_frame>Base</robot_base_frame>
-                    <odom_publish_frequency>500</odom_publish_frequency>
-                    <dimensions>3</dimensions>
-                </plugin>
-            </gazebo>
-            <gazebo>
-                <plugin filename="gz-sim-imu-system" name="gz::sim::systems::Imu">
-                </plugin>
-            </gazebo>
-        </xacro:unless>
+        <gazebo>
+            <plugin filename="gz-sim-odometry-publisher-system" name="gz::sim::systems::OdometryPublisher">
+                <odom_frame>Base</odom_frame>
+                <robot_base_frame>Base</robot_base_frame>
+                <odom_publish_frequency>500</odom_publish_frequency>
+                <dimensions>3</dimensions>
+            </plugin>
+        </gazebo>
+        <gazebo>
+            <plugin filename="gz-sim-imu-system" name="gz::sim::systems::Imu"/>
+        </gazebo>
         <gazebo reference="Base">
             <sensor name="imu_sensor" type="imu">
