Commit message: Carry both Ayg 1.2 and 1.3 robot descriptions (#14)
Restructures ayg_description into per-version 1.2/ and 1.3/ subtrees behind ayg.xacro's version:= dispatch, so one checkout serves both chassis (Ayg #306).

Co-Authored-By: Claude Opus 5 (1M context) <noreply@anthropic.com>

File: urdf/ayg.xacro (robot description, xacro)
@@ -5,6 +5,18 @@
   <xacro:arg name="sim_backend" default="gazebo" />
   <xacro:property name="sim_backend" value="$(arg sim_backend)" />
+  <!-- Which Ayg model to build: "1.2" or "1.3". Selects the whole per-version
+       subtree (root xacro, legs, meshes, mujoco/rviz configs) - see the
+       dispatch include at the bottom of this file.
+       Default mirrors ayg_utils.robot_version.DEFAULT in the Ayg repo. -->
+  <xacro:arg name="version" default="1.2" />
+  <!-- Ayg 1.2's RealSense D555 depth camera. Consumed only by urdf/1.2/*;
+       a harmless no-op when version:=1.3. -->
   <xacro:arg name="camera" default="True" />
   <xacro:property name="camera" default="$(arg camera)" />
+  <!-- Ayg 1.3 replaced the D555 depth camera with a LiDAR on a new front
+       mount; the argument follows the hardware. Consumed only by
+       urdf/1.3/*; a harmless no-op when version:=1.2. -->
+  <xacro:arg name="lidar" default="True" />
+  <xacro:property name="lidar" default="$(arg lidar)" />
   <xacro:arg name="initial_configuration" default="lying_down" />
   <xacro:property name="initial_configuration" value="$(arg initial_configuration)" />
@@ -12,33 +24,19 @@
   <xacro:property name="controller" default="$(arg controller)" />
   <xacro:arg name="use_csp" default="false" />
+  <!-- Robstride MIT gains the hardware interface applies until a controller
+       claims the kp/kd command interfaces (none of the shipped ones does, so in
+       practice these ARE the gains). kp=0 leaves the motors enabled but
+       torque-free, which is how the joints are moved by hand for calibration:
+       robstride_hardware/launch/quadruped.launch.py free_joints:=true. -->
+  <xacro:arg name="default_kp" default="40.0" />
+  <xacro:arg name="default_kd" default="1.0" />
   <xacro:property name="effort_lim" value="50.0" />
   <xacro:property name="velocity_lim" value="10.0" />
   <xacro:property name="PI" value="3.1415926535897931" />
-  <xacro:property name="model_version" value="1.3" />
-  <model_version>${model_version}</model_version>
-  <!-- Battery inertial properties (CAD export → URDF frame)
-       CAD frame: X=forward, Y=up, Z=left  |  URDF frame: X=forward, Y=left, Z=up
-       Mapping: (URDF_x, URDF_y, URDF_z) = (CAD_x, CAD_z, CAD_y)
-       CAD mass: 1.55217 kg  |  Weighed: 1.6 kg each  |  Housing mass is in Base -->
-  <xacro:property name="battery_cad_mass" value="1.55217" />
-  <xacro:property name="battery_real_mass" value="1.6" />
-  <xacro:property name="battery_inertia_scale" value="${battery_real_mass / battery_cad_mass}" />
-  <!-- CoM in battery link frame (URDF, meters) -->
-  <xacro:property name="battery_com_x" value="-0.00002" />
-  <xacro:property name="battery_com_y" value="-0.00421" />
-  <xacro:property name="battery_com_z" value="0.04143" />
-  <!-- Inertia at CoM, at CAD mass, URDF frame (kg·m²) -->
-  <xacro:property name="battery_cad_ixx" value="0.0043243903" />
-  <xacro:property name="battery_cad_ixy" value="-0.0000040621" />
-  <xacro:property name="battery_cad_ixz" value="-0.0000050483" />
-  <xacro:property name="battery_cad_iyy" value="0.0074475647" />
-  <xacro:property name="battery_cad_iyz" value="-0.0002587481" />
-  <xacro:property name="battery_cad_izz" value="0.0043149743" />
-  <!-- Battery positions relative to Base (URDF, meters) -->
-  <xacro:property name="battery_front_x" value="0.10070" />
-  <xacro:property name="battery_rear_x" value="-0.10070" />
-  <xacro:property name="battery_pos_z" value="-0.00900" />
+  <!-- $(arg version) substituted as TEXT, not read back through a property:
+       see the dispatch include below for why. -->
+  <model_version>$(arg version)</model_version>
   <xacro:if value="${sim}">
-    <xacro:include filename="$(find ayg_description)/urdf/ayg_sim_ros2_control.xacro" />
+    <xacro:include filename="$(find ayg_description)/urdf/sim_ros2_control.xacro" />
   </xacro:if>
   <xacro:unless value="${sim}">
@@ -50,136 +48,18 @@
       rh_can_interface="can3"
       actuator_type="3"
-      default_kp="40.0"
-      default_kd="1.0"
+      default_kp="$(arg default_kp)"
+      default_kd="$(arg default_kd)"
       use_csp="$(arg use_csp)"
       calibration_file="$(find robstride_hardware)/calibration/joint_calibration.yaml"
     />
   </xacro:unless>
-  <link
-    name="Base">
-    <inertial>
-      <origin
-        xyz="0.00057686 -0.00018498 0.0026529"
-        rpy="0 0 0" />
-      <!-- Measured: 9.148 kg (CAD: 9.1298 kg) -->
-      <mass
-        value="9.148" />
-      <inertia
-        ixx="0.022082"
-        ixy="3.2369E-07"
-        ixz="6.8653E-05"
-        iyy="0.031986"
-        iyz="2.8565E-07"
-        izz="0.040389" />
-    </inertial>
-    <visual>
-      <origin
-        xyz="0 0 0"
-        rpy="0 0 0" />
-      <geometry>
-        <mesh
-          filename="package://ayg_description/meshes/Base.STL" />
-      </geometry>
-      <material
-        name="">
-        <color
-          rgba="0.69804 0.69804 0.69804 1" />
-      </material>
-    </visual>
-    <collision>
-      <origin
-        xyz="0 0 0"
-        rpy="0 0 0" />
-      <geometry>
-        <box size="0.4 0.23 0.12" />
-      </geometry>
-    </collision>
-  </link>
-  <link
-    name="IMU">
-    <inertial>
-      <origin
-        xyz="-1.26817788945405E-05 -3.05893593341006E-06 0.00502425421604302"
-        rpy="0 0 0" />
-      <mass
-        value="0.0181381899874512" />
-      <inertia
-        ixx="4.80017459218422E-06"
-        ixy="-6.17315963282016E-11"
-        ixz="-1.66852937330168E-09"
-        iyy="3.40477341509462E-06"
-        iyz="-3.279931989329E-11"
-        izz="7.92679226862755E-06" />
-    </inertial>
-    <visual>
-      <origin
-        xyz="0 0 0"
-        rpy="0 0 0" />
-      <geometry>
-        <mesh
-          filename="package://ayg_description/meshes/IMU.STL" />
-      </geometry>
-      <material
-        name="">
-        <color
-          rgba="0.792156862745098 0.819607843137255 0.933333333333333 1" />
-      </material>
-    </visual>
-  </link>
-  <joint
-    name="Base_2_IMU"
-    type="fixed">
-    <origin
-      xyz="-3.79309829856879E-05 0 -0.0172341687059438"
-      rpy="0 0 0" />
-    <parent
-      link="Base" />
-    <child
-      link="IMU" />
-    <axis
-      xyz="0 0 0" />
-  </joint>
-  <!-- Battery macro (2x identical packs, front and rear) -->
-  <xacro:macro name="battery" params="name pos_x">
-    <link name="Battery_${name}">
-      <inertial>
-        <origin xyz="${battery_com_x} ${battery_com_y} ${battery_com_z}" rpy="0 0 0" />
-        <mass value="${battery_real_mass}" />
-        <inertia
-          ixx="${battery_cad_ixx * battery_inertia_scale}"
-          ixy="${battery_cad_ixy * battery_inertia_scale}"
-          ixz="${battery_cad_ixz * battery_inertia_scale}"
-          iyy="${battery_cad_iyy * battery_inertia_scale}"
-          iyz="${battery_cad_iyz * battery_inertia_scale}"
-          izz="${battery_cad_izz * battery_inertia_scale}" />
-      </inertial>
-      <visual>
-        <origin xyz="0 0 0" rpy="0 0 0" />
-        <geometry>
-          <box size="0.079 0.177 0.096" />
-        </geometry>
-        <material name="battery_color">
-          <color rgba="0.2 0.2 0.3 1" />
-        </material>
-      </visual>
-      <collision>
-        <origin xyz="0 0 0" rpy="0 0 0" />
-        <geometry>
-          <box size="0.079 0.177 0.096" />
-        </geometry>
-      </collision>
-    </link>
-    <joint name="Base_2_Battery_${name}" type="fixed">
-      <origin xyz="${pos_x} 0 ${battery_pos_z}" rpy="0 0 0" />
-      <parent link="Base" />
-      <child link="Battery_${name}" />
-      <axis xyz="0 0 0" />
-    </joint>
-  </xacro:macro>
-  <xacro:battery name="Front" pos_x="${battery_front_x}" />
-  <xacro:battery name="Rear"  pos_x="${battery_rear_x}" />
-  <xacro:include filename="$(find ayg_description)/urdf/legs.xacro" />
-  <xacro:if value="${camera}">
-    <xacro:include filename="$(find ayg_description)/urdf/camera.xacro" />
-  </xacro:if>
+  <!-- Per-version dispatch (Base/IMU/battery/legs/camera-or-lidar): urdf/ayg1.2.xacro
+       or urdf/ayg1.3.xacro, chosen by substituting $(arg version) into the
+       INCLUDE FILENAME, as plain text before xacro ever runs. This must stay a
+       filename substitution and NEVER become a `${version == '1.3'}` xacro:if -
+       xacro coerces xacro:property values that parse as numbers, so a property
+       built from $(arg version) holds the FLOAT 1.3 and an equality check
+       against the string '1.3' silently evaluates false. Confirmed in the
+       container; do not "simplify" this. -->
+  <xacro:include filename="$(find ayg_description)/urdf/ayg$(arg version).xacro" />
 </robot>

File: urdf/ayg1.2.urdf (robot description, URDF)
Before this commit: robot ayg, 25 links, 24 joints
Links:
- link Base: geometry collision box size=0.4 0.23 0.12; visual mesh filename=package://ayg_description/meshes/1.2/Base.STL
- link Camera: geometry collision box size=0.0571 0.0443 0.167; visual mesh filename=package://ayg_description/meshes/1.2/Camera.STL
- link IMU: geometry visual mesh filename=package://ayg_description/meshes/1.2/IMU.STL
- link LF_Hip: geometry collision cylinder length=0.148 radius=0.05; visual mesh filename=package://ayg_description/meshes/1.2/L_Hip.STL
- link LF_Shank: geometry collision box size=0.025 0.165 0.0125; collision cylinder length=0.03 radius=0.025
- link LF_Thigh: geometry collision box size=0.025 0.05 0.14; visual mesh filename=package://ayg_description/meshes/1.2/L_Thigh.STL
- link LH_Hip: geometry collision cylinder length=0.148 radius=0.05; visual mesh filename=package://ayg_description/meshes/1.2/R_Hip.STL
- link LH_Shank: geometry collision box size=0.025 0.165 0.0125; collision cylinder length=0.03 radius=0.025
- link LH_Thigh: geometry collision box size=0.025 0.05 0.14; visual mesh filename=package://ayg_description/meshes/1.2/L_Thigh.STL
- link RF_Hip: geometry collision cylinder length=0.148 radius=0.05; visual mesh filename=package://ayg_description/meshes/1.2/R_Hip.STL
- link RF_Shank: geometry collision box size=0.025 0.165 0.0125; collision cylinder length=0.03 radius=0.025
- link RF_Thigh: geometry collision box size=0.025 0.05 0.14; visual mesh filename=package://ayg_description/meshes/1.2/R_Thigh.STL
- link RH_Hip: geometry collision cylinder length=0.148 radius=0.05; visual mesh filename=package://ayg_description/meshes/1.2/L_Hip.STL
- link RH_Shank: geometry collision box size=0.025 0.165 0.0125; collision cylinder length=0.03 radius=0.025
- link RH_Thigh: geometry collision box size=0.025 0.05 0.14; visual mesh filename=package://ayg_description/meshes/1.2/R_Thigh.STL

File: urdf/sim_ros2_control.xacro (robot description, xacro)
@@ -27,35 +27,13 @@
             <plugin>${system_plugin}</plugin>
             <xacro:if value="${sim_backend == 'mujoco'}">
-                <param name="mujoco_model_path">$(find ayg_description)/mujoco/ayg.xml</param>
+                <param name="mujoco_model_path">$(find ayg_description)/mujoco/$(arg version)/ayg.xml</param>
             </xacro:if>
         </hardware>
-        <xacro:if value="${initial_configuration == 'lying_down'}">
-            <xacro:ros2_control_joint joint_name="LF_HAA" effort_lim="${effort_lim}" initial_value="-0.00"/>
-            <xacro:ros2_control_joint joint_name="LF_HFE" effort_lim="${effort_lim}" initial_value="-0.36"/>
-            <xacro:ros2_control_joint joint_name="LF_KFE" effort_lim="${effort_lim}" initial_value=" 1.09"/>
-            <xacro:ros2_control_joint joint_name="RF_HAA" effort_lim="${effort_lim}" initial_value=" 0.00"/>
-            <xacro:ros2_control_joint joint_name="RF_HFE" effort_lim="${effort_lim}" initial_value="-0.36"/>
-            <xacro:ros2_control_joint joint_name="RF_KFE" effort_lim="${effort_lim}" initial_value=" 1.09"/>
-            <xacro:ros2_control_joint joint_name="LH_HAA" effort_lim="${effort_lim}" initial_value=" 0.00"/>
-            <xacro:ros2_control_joint joint_name="LH_HFE" effort_lim="${effort_lim}" initial_value="-0.48"/>
-            <xacro:ros2_control_joint joint_name="LH_KFE" effort_lim="${effort_lim}" initial_value=" 1.20"/>
-            <xacro:ros2_control_joint joint_name="RH_HAA" effort_lim="${effort_lim}" initial_value=" 0.00"/>
-            <xacro:ros2_control_joint joint_name="RH_HFE" effort_lim="${effort_lim}" initial_value="-0.48"/>
-            <xacro:ros2_control_joint joint_name="RH_KFE" effort_lim="${effort_lim}" initial_value=" 1.20"/>
-        </xacro:if>
-        <xacro:if value="${initial_configuration == 'standing'}">
-            <xacro:ros2_control_joint joint_name="LF_HAA" effort_lim="${effort_lim}" initial_value="-0.00"/>
-            <xacro:ros2_control_joint joint_name="LF_HFE" effort_lim="${effort_lim}" initial_value="-0.00"/>
-            <xacro:ros2_control_joint joint_name="LF_KFE" effort_lim="${effort_lim}" initial_value=" 0.00"/>
-            <xacro:ros2_control_joint joint_name="RF_HAA" effort_lim="${effort_lim}" initial_value=" 0.00"/>
-            <xacro:ros2_control_joint joint_name="RF_HFE" effort_lim="${effort_lim}" initial_value="-0.00"/>
-            <xacro:ros2_control_joint joint_name="RF_KFE" effort_lim="${effort_lim}" initial_value=" 0.00"/>
-            <xacro:ros2_control_joint joint_name="LH_HAA" effort_lim="${effort_lim}" initial_value=" 0.00"/>
-            <xacro:ros2_control_joint joint_name="LH_HFE" effort_lim="${effort_lim}" initial_value="-0.00"/>
-            <xacro:ros2_control_joint joint_name="LH_KFE" effort_lim="${effort_lim}" initial_value=" 0.00"/>
-            <xacro:ros2_control_joint joint_name="RH_HAA" effort_lim="${effort_lim}" initial_value=" 0.00"/>
-            <xacro:ros2_control_joint joint_name="RH_HFE" effort_lim="${effort_lim}" initial_value="-0.00"/>
-            <xacro:ros2_control_joint joint_name="RH_KFE" effort_lim="${effort_lim}" initial_value=" 0.00"/>
-        </xacro:if>
+        <!-- initial_configuration poses (lying_down / standing) are per-version:
+             the 1.2 and 1.3 leg geometries need different joint values to reach
+             the same named pose (see each version's file for the derivation).
+             Filename substitution on $(arg version), same convention and same
+             reason as the ayg$(arg version).xacro dispatch in ayg.xacro. -->
+        <xacro:include filename="$(find ayg_description)/urdf/$(arg version)/initial_configuration.xacro" />
         <sensor name="imu_sensor">
             <state_interface name="orientation.x"/>
@@ -76,5 +54,8 @@
             <gazebo>
                 <plugin filename="libgz_ros2_control-system.so" name="gz_ros2_control::GazeboSimROS2ControlPlugin">
-                    <parameters>$(find ayg_control)/config/gazebo/ayg_sw_controllers.yaml</parameters>
+                    <!-- ayg_control#306 split this config per-version; $(arg version)
+                         text substitution, same convention as the dispatch sites above
+                         (do NOT read this back through a ${...} property). -->
+                    <parameters>$(find ayg_control)/config/$(arg version)/gazebo/ayg_sw_controllers.yaml</parameters>
                 </plugin>
             </gazebo>

Commit message: urdf: payload_mass xacro arg, a load carried on Base (Ayg 1.3)
Default 0 kg: the rendered sim and hardware URDFs are byte-identical to
before. A payload is added to Base the same way as extra_base_mass,
uniform over the Base collision box at the CAD centre of mass, so 15 kg
takes Base from 12.02 to 27.02 kg. Used by Gazebo to test the DreamWaQ
payload policy under load.

Co-Authored-By: Claude Opus 5.5 <noreply@anthropic.com>

File: urdf/ayg.xacro (robot description, xacro)
@@ -19,4 +19,7 @@
   <xacro:arg name="lidar" default="True" />
   <xacro:property name="lidar" default="$(arg lidar)" />
+  <!-- Payload carried on Base, in kg (Ayg 1.3 only; a no-op when version:=1.2).
+       0 is the bare robot; set it in simulation to test a policy under load. -->
+  <xacro:arg name="payload_mass" default="0.0" />
   <xacro:arg name="initial_configuration" default="lying_down" />
   <xacro:property name="initial_configuration" value="$(arg initial_configuration)" />

File: urdf/ayg1.3.xacro (robot description, xacro)
@@ -15,8 +15,13 @@
        position inside the trunk equally likely, that is the expected inertia.
        Each diagonal term gains m (a^2 + b^2) / 12; the centre of mass and the
-       products of inertia keep their CAD values. -->
+       products of inertia keep their CAD values.
+       The payload_mass xacro arg (default 0) adds a carried load on top of it,
+       modelled the same way: uniform over the Base box at the CAD centre of
+       mass. -->
   <xacro:property name="base_mass_cad"   value="11.02" />
   <xacro:property name="extra_base_mass" value="1.0" />
-  <xacro:property name="base_mass"       value="${base_mass_cad + extra_base_mass}" />
+  <xacro:property name="payload_mass"    value="$(arg payload_mass)" />
+  <xacro:property name="added_base_mass" value="${extra_base_mass + payload_mass}" />
+  <xacro:property name="base_mass"       value="${base_mass_cad + added_base_mass}" />
   <xacro:property name="base_box_x"      value="0.423" />
   <xacro:property name="base_box_y"      value="0.239" />
@@ -40,10 +45,10 @@
         value="${base_mass}" />
       <inertia
-        ixx="${round(0.035479 + extra_base_mass * (base_box_y**2 + base_box_z**2) / 12, 6)}"
+        ixx="${round(0.035479 + added_base_mass * (base_box_y**2 + base_box_z**2) / 12, 6)}"
         ixy="-3.4801E-06"
         ixz="8.3812E-05"
-        iyy="${round(0.032555 + extra_base_mass * (base_box_x**2 + base_box_z**2) / 12, 6)}"
+        iyy="${round(0.032555 + added_base_mass * (base_box_x**2 + base_box_z**2) / 12, 6)}"
         iyz="0.00043953"
-        izz="${round(0.055613 + extra_base_mass * (base_box_x**2 + base_box_y**2) / 12, 6)}" />
+        izz="${round(0.055613 + added_base_mass * (base_box_x**2 + base_box_y**2) / 12, 6)}" />
     </inertial>
     <visual>
