Commit message: Update urdf

File: urdf/ayg.urdf (robot description, URDF)
Before this commit: robot ayg, 20 links, 19 joints
Links:
- link Base: mass 5.6129 -> 8.43904999246817
- link LF_Foot: mass 0.088055 -> 0.088054927521184
- link LF_Hip: mass 1.0061 -> 1.00401999005125; geometry collision mesh filename=package://ayg_description/meshes/L_Hip.STL; visual mesh filename=package://ayg_description/meshes/L_Hip.STL
- link LF_Shank: mass 0.058285 -> 0.102570008997248; geometry collision mesh filename=package://ayg_description/meshes/L_Shank.STL; visual mesh filename=package://ayg_description/meshes/L_Shank.STL
- link LF_Thigh: mass 1.1334 -> 1.15974999242447; geometry collision mesh filename=package://ayg_description/meshes/L_Thigh.STL; visual mesh filename=package://ayg_description/meshes/L_Thigh.STL
- link LH_Foot: mass 0.0880549275211839 -> 0.088054927521184
- link LH_Hip: mass 1.00611999358686 -> 1.00401999005125; geometry collision mesh filename=package://ayg_description/meshes/L_Hip.STL; visual mesh filename=package://ayg_description/meshes/L_Hip.STL
- link LH_Shank: mass 0.0582850645781694 -> 0.102570008997248; geometry collision mesh filename=package://ayg_description/meshes/L_Shank.STL; visual mesh filename=package://ayg_description/meshes/L_Shank.STL
- link LH_Thigh: mass 1.13336000771446 -> 1.15974999242447; geometry collision mesh filename=package://ayg_description/meshes/L_Thigh.STL; visual mesh filename=package://ayg_description/meshes/L_Thigh.STL
- link Neck: mass 0.36577 -> 0
- link RF_Foot: mass 0.0880549275211839 -> 0.088054927521184
- link RF_Hip: mass 1.00611999358686 -> 1.00401999005125; geometry collision mesh filename=package://ayg_description/meshes/R_Hip.STL; visual mesh filename=package://ayg_description/meshes/R_Hip.STL
- link RF_Shank: mass 0.0582850645781695 -> 0.102570008997248; geometry collision mesh filename=package://ayg_description/meshes/R_Shank.STL; visual mesh filename=package://ayg_description/meshes/R_Shank.STL
- link RF_Thigh: mass 1.13336000773924 -> 1.15974999242447; geometry collision mesh filename=package://ayg_description/meshes/R_Thigh.STL; visual mesh filename=package://ayg_description/meshes/R_Thigh.STL
- link RH_Foot: mass 0.0880549275211839 -> 0.088054927521184
- link RH_Hip: mass 1.00611999358686 -> 1.00401999005125; geometry collision mesh filename=package://ayg_description/meshes/R_Hip.STL; visual mesh filename=package://ayg_description/meshes/R_Hip.STL
- link RH_Shank: mass 0.0582850645781694 -> 0.102570008997248; geometry collision mesh filename=package://ayg_description/meshes/R_Shank.STL; visual mesh filename=package://ayg_description/meshes/R_Shank.STL
- link RH_Thigh: mass 1.13336000773924 -> 1.15974999242447; geometry collision mesh filename=package://ayg_description/meshes/R_Thigh.STL; visual mesh filename=package://ayg_description/meshes/R_Thigh.STL
Joints:
- joint Base_2_IMU: origin xyz=0 0 -0.001 rpy=-1.5708 0 -1.5708 -> xyz=0 0 0.006 rpy=-1.5708 0 1.5708
- joint Base_2_Neck: origin xyz=0.2265 0 0.02 rpy=1.5708 0 1.5708 -> xyz=0.2615 0 0.0249999999999999 rpy=1.5707963267949 0 1.5707963267949
- joint LF_HAA: limit lower=-0.34907 upper=0.17453 effort=50.0 velocity=10.0 -> lower=-0.5236 upper=0.34907 effort=50.0 velocity=10.0; origin xyz=0.15192 0.054 0 rpy=1.5708 0 0 -> xyz=0.197 0.054 0 rpy=-1.5708 0 0
- joint LF_HFE: limit lower=-2.618 upper=0.34907 effort=50.0 velocity=10.0 -> lower=-0.87266 upper=2.5307 effort=50.0 velocity=10.0; origin xyz=0.077085 0 -0.017 rpy=0 0 0 -> xyz=0.0665 0 0.019 rpy=3.1416 0 0
- joint LF_KFE: limit lower=-0.43633 upper=1.2217 effort=50.0 velocity=10.0 -> lower=-0.7854 upper=1.2217 effort=50.0 velocity=10.0; origin xyz=-0.1494 -0.16021 -0.0539 rpy=0 0 0 -> xyz=-0.14936 -0.16017 -0.052 rpy=0 0 0
- joint LF_Shank_2_Foot: origin xyz=0.165 -0.151 -0.0201 rpy=0 0 0 -> xyz=0.165 -0.151 -0.0185 rpy=0 0 0
- joint LH_HAA: limit lower=-0.69813 upper=0.34907 effort=50.0 velocity=10.0 -> lower=-0.87266 upper=0.5236 effort=50.0 velocity=10.0; origin xyz=-0.15192 0.054 0 rpy=-1.5708 0 3.1416 -> xyz=-0.197 0.054 0 rpy=-1.5708 0 3.1416
- joint LH_HFE: limit lower=-0.87266 upper=2.618 effort=50.0 velocity=10.0 -> lower=-2.5307 upper=0.87266 effort=50.0 velocity=10.0; origin xyz=0.077085 0 -0.017 rpy=0 0 3.1416 -> xyz=0.0665 0 -0.019 rpy=0 0 3.1416
- joint LH_KFE: limit lower=-0.43633 upper=1.2217 effort=50.0 velocity=10.0 -> lower=-0.7854 upper=1.2217 effort=50.0 velocity=10.0; origin xyz=-0.1494 -0.16021 -0.0539 rpy=0 0 0 -> xyz=-0.14936 -0.16017 -0.052 rpy=0 0 0
- joint LH_Shank_2_Foot: origin xyz=0.165 -0.151 -0.0201 rpy=0 0 0 -> xyz=0.164999999999998 -0.151000000000002 -0.0185 rpy=0 0 0
- joint Neck_2_Camera: origin xyz=0 0.01666 0.080407 rpy=0.28898 0 0 -> xyz=0 0.0166603444360147 0.0804068913666247 rpy=0.288975409992567 0 0
- joint RF_HAA: limit lower=-0.17453 upper=0.34907 effort=50.0 velocity=10.0 -> lower=-0.34907 upper=0.5236 effort=50.0 velocity=10.0; origin xyz=0.15192 -0.054 0 rpy=-1.5708 0 0 -> xyz=0.197 -0.054 0 rpy=-1.5708 0 0
- joint RF_HFE: limit lower=-0.34907 upper=2.618 effort=50.0 velocity=10.0 -> lower=-0.87266 upper=2.5307 effort=50.0 velocity=10.0; origin xyz=0.077085 0 -0.017 rpy=3.1416 0 0 -> xyz=0.0665 0 -0.019 rpy=3.1416 0 0
- joint RF_KFE: limit lower=-0.43633 upper=1.2217 effort=50.0 velocity=10.0 -> lower=-0.7854 upper=1.2217 effort=50.0 velocity=10.0; origin xyz=-0.1494 -0.16021 0.0539 rpy=0 0 0 -> xyz=-0.14936 -0.16017 0.052 rpy=0 0 0
- joint RF_Shank_2_Foot: origin xyz=0.165 -0.151 0.0201 rpy=0 0 0 -> xyz=0.165 -0.151 0.0185 rpy=0 0 0
- joint RH_HAA: limit lower=-0.34907 upper=0.69813 effort=50.0 velocity=10.0 -> lower=-0.5236 upper=0.87266 effort=50.0 velocity=10.0; origin xyz=-0.15192 -0.054 0 rpy=1.5708 0 3.1416 -> xyz=-0.197 -0.054 0 rpy=-1.5708 0 3.1416
- joint RH_HFE: limit lower=-2.618 upper=0.87266 effort=50.0 velocity=10.0 -> lower=-2.5307 upper=0.87266 effort=50.0 velocity=10.0; origin xyz=0.077085 0 -0.017 rpy=3.1416 0 3.1416 -> xyz=0.0665 0 0.019 rpy=0 0 3.1416
- joint RH_KFE: limit lower=-0.43633 upper=1.2217 effort=50.0 velocity=10.0 -> lower=-0.7854 upper=1.2217 effort=50.0 velocity=10.0; origin xyz=-0.1494 -0.16021 0.0539 rpy=0 0 0 -> xyz=-0.14936 -0.16017 0.052 rpy=0 0 0
- joint RH_Shank_2_Foot: origin xyz=0.165 -0.151 0.0201 rpy=0 0 0 -> xyz=0.165 -0.151 0.0185 rpy=0 0 0

Commit message: Use xacro macros for left and right legs

File: urdf/ayg.urdf (robot description, URDF)
Before this commit: robot ayg, 20 links, 19 joints
Links:
- link Base: geometry collision box size=0.4 0.23 0.12; visual mesh filename=package://ayg_description/meshes/Base.STL
- link IMU: geometry visual mesh filename=package://ayg_description/meshes/IMU.STL
Joints:
- joint LH_Shank_2_Foot: origin xyz=0.164999999999998 -0.151000000000002 -0.0185 rpy=0 0 0 -> xyz=0.165 -0.151 -0.0185 rpy=0 0 0

File: urdf/ayg.xacro (robot description, xacro)
@@ -48,909 +48,9 @@
         rpy="0 0 0" />
       <geometry>
-        <mesh
-          filename="package://ayg_description/meshes/Base.STL" />
+        <box size="0.4 0.23 0.12" />
       </geometry>
     </collision>
   </link>
-  <link
-    name="LF_Hip">
-    <inertial>
-      <origin
-        xyz="0.0624625305028617 0.000263588472359728 -0.00241409757946361"
-        rpy="0 0 0" />
-      <mass
-        value="1.00401999005125" />
-      <inertia
-        ixx="0.000584357699669872"
-        ixy="1.71578981310067E-06"
-        ixz="-2.61675027998363E-19"
-        iyy="0.000584539401732687"
-        iyz="-3.57751728713357E-20"
-        izz="0.00102756652010595" />
-    </inertial>
-    <visual>
-      <origin
-        xyz="0 0 0"
-        rpy="0 0 0" />
-      <geometry>
-        <mesh
-          filename="package://ayg_description/meshes/L_Hip.STL" />
-      </geometry>
-      <material
-        name="">
-        <color
-          rgba="0.698039215686274 0.698039215686274 0.698039215686274 1" />
-      </material>
-    </visual>
-    <collision>
-      <origin
-        xyz="0 0 0"
-        rpy="0 0 0" />
-      <geometry>
-        <mesh
-          filename="package://ayg_description/meshes/L_Hip.STL" />
-      </geometry>
-    </collision>
-  </link>
-  <joint
-    name="LF_HAA"
-    type="revolute">
-    <origin
-      xyz="0.197 0.054 0"
-      rpy="-1.5708 0 0" />
-    <parent
-      link="Base" />
-    <child
-      link="LF_Hip" />
-    <axis
-      xyz="1 0 0" />
-    <limit
-      lower="-0.5236"
-      upper="0.34907"
-      effort="${effort_lim}"
-      velocity="${velocity_lim}" />
-  </joint>
-  <link
-    name="LF_Thigh">
-    <inertial>
-      <origin
-        xyz="-0.00815740476229621 -0.00912689407030123 -0.0420066354122466"
-        rpy="0 0 0" />
-      <mass
-        value="1.15974999242447" />
-      <inertia
-        ixx="0.000911992879302287"
-        ixy="-0.000310524680951164"
-        ixz="-4.3266057977693E-16"
-        iyy="0.00091897366461706"
-        iyz="-1.93894477964206E-06"
-        izz="0.00169326046596367" />
-    </inertial>
-    <visual>
-      <origin
-        xyz="0 0 0"
-        rpy="0 0 0" />
-      <geometry>
-        <mesh
-          filename="package://ayg_description/meshes/L_Thigh.STL" />
-      </geometry>
-      <material
-        name="">
-        <color
-          rgba="0.698039215686274 0.698039215686274 0.698039215686274 1" />
-      </material>
-    </visual>
-    <collision>
-      <origin
-        xyz="0 0 0"
-        rpy="0 0 0" />
-      <geometry>
-        <mesh
-          filename="package://ayg_description/meshes/L_Thigh.STL" />
-      </geometry>
-    </collision>
-  </link>
-  <joint
-    name="LF_HFE"
-    type="revolute">
-    <origin
-      xyz="0.0665 0 0.019"
-      rpy="3.1416 0 0" />
-    <parent
-      link="LF_Hip" />
-    <child
-      link="LF_Thigh" />
-    <axis
-      xyz="0 0 1" />
-    <limit
-      lower="-0.87266"
-      upper="2.5307"
-      effort="${effort_lim}"
-      velocity="${velocity_lim}" />
-  </joint>
-  <link
-    name="LF_Shank">
-    <inertial>
-      <origin
-        xyz="0.0630329536265654 -0.047817827674744 -0.0185"
-        rpy="0 0 0" />
-      <mass
-        value="0.102570008997248" />
-      <inertia
-        ixx="0.00029767764878727"
-        ixy="0.000296980915761884"
-        ixz="1.63288326545704E-19"
-        iyy="0.000327832614532812"
-        iyz="-1.54063121876522E-19"
-        izz="0.000624546801244392" />
-    </inertial>
-    <visual>
-      <origin
-        xyz="0 0 0"
-        rpy="0 0 0" />
-      <geometry>
-        <mesh
-          filename="package://ayg_description/meshes/L_Shank.STL" />
-      </geometry>
-      <material
-        name="">
-        <color
-          rgba="0.698039215686274 0.698039215686274 0.698039215686274 1" />
-      </material>
-    </visual>
-    <collision>
-      <origin
-        xyz="0 0 0"
-        rpy="0 0 0" />
-      <geometry>
-        <mesh
-          filename="package://ayg_description/meshes/L_Shank.STL" />
-      </geometry>
-    </collision>
-  </link>
-  <joint
-    name="LF_KFE"
-    type="revolute">
-    <origin
-      xyz="-0.14936 -0.16017 -0.052"
-      rpy="0 0 0" />
-    <parent
-      link="LF_Thigh" />
-    <child
-      link="LF_Shank" />
-    <axis
-      xyz="0 0 1" />
-    <limit
-      lower="-0.7854"
-      upper="1.2217"
-      effort="${effort_lim}"
-      velocity="${velocity_lim}" />
-  </joint>
-  <link
-    name="LF_Foot">
-    <inertial>
-      <origin
-        xyz="-2.77555756156289E-17 5.55111512312578E-17 0"
-        rpy="0 ${PI/2} 0" />
-      <mass
-        value="0.088054927521184" />
-      <inertia
-        ixx="4.09565481632907E-05"
-        ixy="-8.61058027358505E-21"
-        ixz="2.27932697045296E-20"
-        iyy="2.47049106026622E-05"
-        iyz="5.04870979341448E-29"
-        izz="2.47049106026622E-05" />
-    </inertial>
-    <visual>
-      <origin
-        xyz="0 0 0"
-        rpy="0 0 0" />
-      <geometry>
-        <cylinder length="0.025" radius="0.030" />
-      </geometry>
-      <material
-        name="">
-        <color
-          rgba="0.250980392156863 0.250980392156863 0.250980392156863 1" />
-      </material>
-    </visual>
-    <collision>
-      <origin
-        xyz="0 0 0"
-        rpy="0 0 0" />
-      <geometry>
-        <cylinder length="0.025" radius="0.030" />
-      </geometry>
-    </collision>
-  </link>
-  <joint
-    name="LF_Shank_2_Foot"
-    type="fixed">
-    <origin
-      xyz="0.165 -0.151 -0.0185"
-      rpy="0 0 0" />
-    <parent
-      link="LF_Shank" />
-    <child
-      link="LF_Foot" />
-    <axis
-      xyz="0 0 0" />
-  </joint>
-  <link
-    name="RF_Hip">
-    <inertial>
-      <origin
-        xyz="0.062462530502862 0.000263588472360484 0.00241409757946365"
-        rpy="0 0 0" />
-      <mass
-        value="1.00401999005125" />
-      <inertia
-        ixx="0.000584357699669871"
-        ixy="1.71578981310067E-06"
-        ixz="-3.08533699148142E-19"
-        iyy="0.000584539401732687"
-        iyz="1.3310433650471E-20"
-        izz="0.00102756652010595" />
-    </inertial>
-    <visual>
-      <origin
-        xyz="0 0 0"
-        rpy="0 0 0" />
-      <geometry>
-        <mesh
-          filename="package://ayg_description/meshes/R_Hip.STL" />
-      </geometry>
-      <material
-        name="">
-        <color
-          rgba="0.698039215686274 0.698039215686274 0.698039215686274 1" />
-      </material>
-    </visual>
-    <collision>
-      <origin
-        xyz="0 0 0"
-        rpy="0 0 0" />
-      <geometry>
-        <mesh
-          filename="package://ayg_description/meshes/R_Hip.STL" />
-      </geometry>
-    </collision>
-  </link>
-  <joint
-    name="RF_HAA"
-    type="revolute">
-    <origin
-      xyz="0.197 -0.054 0"
-      rpy="-1.5708 0 0" />
-    <parent
-      link="Base" />
-    <child
-      link="RF_Hip" />
-    <axis
-      xyz="1 0 0" />
-    <limit
-      lower="-0.34907"
-      upper="0.5236"
-      effort="${effort_lim}"
-      velocity="${velocity_lim}" />
-  </joint>
-  <link
-    name="RF_Thigh">
-    <inertial>
-      <origin
-        xyz="-0.00815740475775473 -0.0091268940561607 0.0420066354122466"
-        rpy="0 0 0" />
-      <mass
-        value="1.15974999242447" />
-      <inertia
-        ixx="0.000911992879285499"
-        ixy="-0.000310524680969909"
-        ixz="4.28891709883383E-15"
-        iyy="0.000918973664621895"
-        iyz="1.93894536662709E-06"
-        izz="0.00169326046595172" />
-    </inertial>
-    <visual>
-      <origin
-        xyz="0 0 0"
-        rpy="0 0 0" />
-      <geometry>
-        <mesh
-          filename="package://ayg_description/meshes/R_Thigh.STL" />
-      </geometry>
-      <material
-        name="">
-        <color
-          rgba="0.698039215686274 0.698039215686274 0.698039215686274 1" />
-      </material>
-    </visual>
-    <collision>
-      <origin
-        xyz="0 0 0"
-        rpy="0 0 0" />
-      <geometry>
-        <mesh
-          filename="package://ayg_description/meshes/R_Thigh.STL" />
-      </geometry>
-    </collision>
-  </link>
-  <joint
-    name="RF_HFE"
-    type="revolute">
-    <origin
-      xyz="0.0665 0 -0.019"
-      rpy="3.1416 0 0" />
-    <parent
-      link="RF_Hip" />
-    <child
-      link="RF_Thigh" />
-    <axis
-      xyz="0 0 1" />
-    <limit
-      lower="-0.87266"
-      upper="2.5307"
-      effort="${effort_lim}"
-      velocity="${velocity_lim}" />
-  </joint>
-  <link
-    name="RF_Shank">
-    <inertial>
-      <origin
-        xyz="0.0630329536265653 -0.047817827674744 0.0185"
-        rpy="0 0 0" />
-      <mass
-        value="0.102570008997248" />
-      <inertia
-        ixx="0.000297677648787269"
-        ixy="0.000296980915761884"
-        ixz="1.63489615161778E-19"
-        iyy="0.000327832614532812"
-        iyz="-1.53587053010883E-19"
-        izz="0.000624546801244392" />
-    </inertial>
-    <visual>
-      <origin
-        xyz="0 0 0"
-        rpy="0 0 0" />
-      <geometry>
-        <mesh
-          filename="package://ayg_description/meshes/R_Shank.STL" />
-      </geometry>
-      <material
-        name="">
-        <color
-          rgba="0.698039215686274 0.698039215686274 0.698039215686274 1" />
-      </material>
-    </visual>
-    <collision>
-      <origin
-        xyz="0 0 0"
-        rpy="0 0 0" />
-      <geometry>
-        <mesh
-          filename="package://ayg_description/meshes/R_Shank.STL" />
-      </geometry>
-    </collision>
-  </link>
-  <joint
-    name="RF_KFE"
-    type="revolute">
-    <origin
-      xyz="-0.14936 -0.16017 0.052"
-      rpy="0 0 0" />
-    <parent
-      link="RF_Thigh" />
-    <child
-      link="RF_Shank" />
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
Commit message: Use primitive geometries as collisions

File: urdf/ayg.urdf (robot description, URDF)
Before this commit: robot ayg, 20 links, 19 joints
Links:
- link Camera: geometry collision box size=0.13 0.035 0.05; visual mesh filename=package://ayg_description/meshes/Camera.STL
- link LF_Hip: geometry collision cylinder length=0.13 radius=0.05; visual mesh filename=package://ayg_description/meshes/L_Hip.STL
- link LF_Shank: geometry collision box size=0.025 0.165 0.0125; collision cylinder length=0.03 radius=0.025
- link LF_Thigh: geometry collision box size=0.025 0.05 0.135; visual mesh filename=package://ayg_description/meshes/L_Thigh.STL
- link LH_Hip: geometry collision cylinder length=0.13 radius=0.05; visual mesh filename=package://ayg_description/meshes/L_Hip.STL
- link LH_Shank: geometry collision box size=0.025 0.165 0.0125; collision cylinder length=0.03 radius=0.025
- link LH_Thigh: geometry collision box size=0.025 0.05 0.135; visual mesh filename=package://ayg_description/meshes/L_Thigh.STL
- link Neck: geometry visual mesh filename=package://ayg_description/meshes/Neck.STL
- link RF_Hip: geometry collision cylinder length=0.13 radius=0.05; visual mesh filename=package://ayg_description/meshes/R_Hip.STL
- link RF_Shank: geometry collision box size=0.025 0.165 0.0125; collision cylinder length=0.03 radius=0.025
- link RF_Thigh: geometry collision box size=0.025 0.05 0.135; visual mesh filename=package://ayg_description/meshes/R_Thigh.STL
- link RH_Hip: geometry collision cylinder length=0.13 radius=0.05; visual mesh filename=package://ayg_description/meshes/R_Hip.STL
- link RH_Shank: geometry collision box size=0.025 0.165 0.0125; collision cylinder length=0.03 radius=0.025
- link RH_Thigh: geometry collision box size=0.025 0.05 0.135; visual mesh filename=package://ayg_description/meshes/R_Thigh.STL

File: urdf/ayg.xacro (robot description, xacro)
@@ -127,13 +127,4 @@
       </material>
     </visual>
-    <collision>
-      <origin
-        xyz="0 0 0"
-        rpy="0 0 0" />
-      <geometry>
-        <mesh
-          filename="package://ayg_description/meshes/Neck.STL" />
-      </geometry>
-    </collision>
   </link>
   <joint
@@ -182,9 +173,8 @@
     <collision>
       <origin
-        xyz="0 0 0"
-        rpy="0 0 0" />
+        xyz="0 -0.0025 0"
+        rpy="-0.288975409992567 0 0" />
       <geometry>
-        <mesh
-          filename="package://ayg_description/meshes/Camera.STL" />
+        <box size="0.13 0.035 0.05"/>
       </geometry>
     </collision>

File: urdf/legs.xacro (robot description, xacro)
@@ -39,13 +39,24 @@
         </material>
       </visual>
-      <collision>
-        <origin
-          xyz="0 0 0"
-          rpy="0 0 0" />
-        <geometry>
-          <mesh
-            filename="package://ayg_description/meshes/L_Hip.STL" />
-        </geometry>
-      </collision>
+      <xacro:if value="${FH == 'F'}">
+        <collision>
+          <origin
+            xyz="0.0665 0 ${0.019+0.015}"
+            rpy="0 0 0" />
+          <geometry>
+            <cylinder radius="0.05" length="0.13"/>
+          </geometry>
+        </collision>
+      </xacro:if>
+      <xacro:unless value="${FH == 'F'}">
+        <collision>
+          <origin
+            xyz="0.0665 0 ${-0.019-0.015}"
+            rpy="0 0 0" />
+          <geometry>
+            <cylinder radius="0.05" length="0.13"/>
+          </geometry>
+        </collision>
+      </xacro:unless>
     </link>
     <joint
@@ -115,9 +126,8 @@
       <collision>
         <origin
-          xyz="0 0 0"
-          rpy="0 0 0" />
-        <geometry>
-          <mesh
-            filename="package://ayg_description/meshes/L_Thigh.STL" />
+          xyz="-0.1 -0.075 -0.07"
+          rpy="0 ${PI/2} ${PI/4}" />
+        <geometry>
+          <box size="0.025 0.05 0.135"/>
         </geometry>
       </collision>
@@ -189,9 +199,16 @@
       <collision>
         <origin
-          xyz="0 0 0"
-          rpy="0 0 0" />
-        <geometry>
-          <mesh
-            filename="package://ayg_description/meshes/L_Shank.STL" />
+          xyz="0 0 -0.02"
+          rpy="0 0 0" />
+        <geometry>
+          <cylinder radius="0.025" length="0.03"/>
+        </geometry>
+      </collision>
+      <collision>
+        <origin
+          xyz="0.08 -0.075 -0.02"
+          rpy="0 0 ${PI/4}" />
+        <geometry>
+          <box size="0.025 0.165 0.0125"/>
         </geometry>
       </collision>
@@ -305,13 +322,24 @@
         </material>
       </visual>
-      <collision>
-        <origin
-          xyz="0 0 0"
-          rpy="0 0 0" />
-        <geometry>
-          <mesh
-            filename="package://ayg_description/meshes/R_Hip.STL" />
-        </geometry>
-      </collision>
+      <xacro:if value="${FH == 'F'}">
+        <collision>
+          <origin
+            xyz="0.0665 0 ${-0.019-0.015}"
+            rpy="0 0 0" />
+          <geometry>
+            <cylinder radius="0.05" length="0.13"/>
+          </geometry>
+        </collision>
+      </xacro:if>
+      <xacro:unless value="${FH == 'F'}">
+        <collision>
+          <origin
+            xyz="0.0665 0 ${+0.019+0.015}"
+            rpy="0 0 0" />
+          <geometry>
+            <cylinder radius="0.05" length="0.13"/>
+          </geometry>
+        </collision>
+      </xacro:unless>
     </link>
     <joint
@@ -381,9 +409,8 @@
       <collision>
         <origin
-          xyz="0 0 0"
-          rpy="0 0 0" />
-        <geometry>
-          <mesh
-            filename="package://ayg_description/meshes/R_Thigh.STL" />
+          xyz="-0.1 -0.075 +0.07"
+          rpy="0 ${PI/2} ${PI/4}" />
+        <geometry>
+          <box size="0.025 0.05 0.135"/>
         </geometry>
       </collision>
@@ -455,9 +482,16 @@
       <collision>
         <origin
-          xyz="0 0 0"
-          rpy="0 0 0" />
-        <geometry>
-          <mesh
-            filename="package://ayg_description/meshes/R_Shank.STL" />
+          xyz="0 0 +0.02"
+          rpy="0 0 0" />
+        <geometry>
+          <cylinder radius="0.025" length="0.03"/>
+        </geometry>
+      </collision>
+      <collision>
+        <origin
+          xyz="0.08 -0.075 +0.02"
+          rpy="0 0 ${PI/4}" />
+        <geometry>
+          <box size="0.025 0.165 0.0125"/>
         </geometry>
       </collision>
