Commit message: Small change + update URDF

File: urdf/ayg.urdf (robot description, URDF)
Before this commit: robot ayg, 20 links, 19 joints
Links:
- link LF_Thigh: geometry collision box size=0.025 0.05 0.14; visual mesh filename=package://ayg_description/meshes/L_Thigh.STL
- link LH_Hip: geometry collision cylinder length=0.13 radius=0.05; visual mesh filename=package://ayg_description/meshes/R_Hip.STL
- link LH_Thigh: geometry collision box size=0.025 0.05 0.14; visual mesh filename=package://ayg_description/meshes/L_Thigh.STL
- link RF_Thigh: geometry collision box size=0.025 0.05 0.14; visual mesh filename=package://ayg_description/meshes/R_Thigh.STL
- link RH_Hip: geometry collision cylinder length=0.13 radius=0.05; visual mesh filename=package://ayg_description/meshes/L_Hip.STL
- link RH_Thigh: geometry collision box size=0.025 0.05 0.14; visual mesh filename=package://ayg_description/meshes/R_Thigh.STL

File: urdf/legs.xacro (robot description, xacro)
@@ -38,6 +38,4 @@
               filename="package://ayg_description/meshes/R_Hip.STL" />
           </xacro:unless>
-          <mesh
-            filename="package://ayg_description/meshes/L_Hip.STL" />
         </geometry>
         <material

Commit message: Update frame orientations

File: urdf/ayg.urdf (robot description, URDF)
Before this commit: robot ayg, 20 links, 19 joints
Joints:
- joint LH_HAA: axis 1 0 0 -> -1 0 0
- joint RH_HAA: axis 1 0 0 -> -1 0 0

File: urdf/legs.xacro (robot description, xacro)
@@ -83,7 +83,7 @@
       <child
         link="L${FH}_Hip" />
-      <axis
+      <xacro:if value="${FH == 'F'}">
+        <axis
         xyz="1 0 0" />
-      <xacro:if value="${FH == 'F'}">
         <limit
           lower="-0.5236"
@@ -93,4 +93,6 @@
       </xacro:if>
       <xacro:unless value="${FH == 'F'}">
+        <axis
+        xyz="-1 0 0" />
         <limit
           lower="-0.87266"
@@ -372,7 +374,7 @@
       <child
         link="R${FH}_Hip" />
-      <axis
+      <xacro:if value="${FH == 'F'}">
+        <axis
         xyz="1 0 0" />
-      <xacro:if value="${FH == 'F'}">
         <limit
           lower="-0.34907"
@@ -382,4 +384,6 @@
       </xacro:if>
       <xacro:unless value="${FH == 'F'}">
+        <axis
+        xyz="-1 0 0" />
         <limit
           lower="-0.5236"
