Commit message: Update urdf (camera is not default, new base, add legs reinforcements)

File: urdf/ayg.urdf (robot description, URDF)
Before this commit: robot ayg, 20 links, 19 joints
Links:
- removed link Camera
- removed link Neck
- link Base: mass 8.43904999246817 -> 9.1298
- link IMU: mass 0.08 -> 0.0181381899874512
- link LF_Foot: mass 0.088054927521184 -> 0.0701295110066971
- link LF_Hip: mass 1.00401999005125 -> 1.0709
- link LF_Shank: mass 0.102570008997248 -> 0.19753
- link LF_Thigh: mass 1.15974999242447 -> 1.361
- link LH_Foot: mass 0.088054927521184 -> 0.0701295110066971
- link LH_Hip: mass 1.00401999005125 -> 1.0709
- link LH_Shank: mass 0.102570008997248 -> 0.19753
- link LH_Thigh: mass 1.15974999242447 -> 1.361
- link RF_Foot: mass 0.088054927521184 -> 0.07013
- link RF_Hip: mass 1.00401999005125 -> 1.071
- link RF_Shank: mass 0.102570008997248 -> 0.19753
- link RF_Thigh: mass 1.15974999242447 -> 1.361
- link RH_Foot: mass 0.088054927521184 -> 0.07013
- link RH_Hip: mass 1.00401999005125 -> 1.071
- link RH_Shank: mass 0.102570008997248 -> 0.19753
- link RH_Thigh: mass 1.15974999242447 -> 1.361
Joints:
- removed joint Base_2_Neck
- removed joint Neck_2_Camera
- joint Base_2_IMU: origin xyz=0 0 0.006 rpy=-1.5708 0 1.5708 -> xyz=-3.79309829856879E-05 0 -0.0172341687059438 rpy=0 0 0
- joint LF_HAA: limit lower=-0.5236 upper=0.34907 effort=50.0 velocity=10.0 -> lower=-0.5236 upper=0.43633 effort=50.0 velocity=10.0; origin xyz=0.197 0.054 0 rpy=-1.5708 0 0 -> xyz=0.2021 0.054 0 rpy=0 0 0
- joint LF_HFE: axis 0 0 1 -> 0 -1 0; limit lower=-0.87266 upper=2.5307 effort=50.0 velocity=10.0 -> lower=-1.6668 upper=3.2376 effort=50.0 velocity=10.0; origin xyz=0.0665 0 0.019 rpy=3.1416 0 0 -> xyz=0.0679 0.01985 0 rpy=0 0 0
- joint LF_KFE: axis 0 0 1 -> 0 -1 0; limit lower=-0.7854 upper=1.2217 effort=50.0 velocity=10.0 -> lower=-0.74002 upper=1.1868 effort=50.0 velocity=10.0; origin xyz=-0.14936 -0.16017 -0.052 rpy=0 0 0 -> xyz=-0.14936 0.058 -0.16017 rpy=0 0 0
- joint LF_Shank_2_Foot: origin xyz=0.165 -0.151 -0.0185 rpy=0 0 0 -> xyz=0.165 0.0205 -0.151 rpy=0 0 0
- joint LH_HAA: limit lower=-0.87266 upper=0.5236 effort=50.0 velocity=10.0 -> lower=-0.5236 upper=0.83776 effort=50.0 velocity=10.0; origin xyz=-0.197 0.054 0 rpy=-1.5708 0 3.1416 -> xyz=-0.2021 0.054 0 rpy=0 0 3.1416
- joint LH_HFE: axis 0 0 1 -> 0 -1 0; limit lower=-2.5307 upper=0.87266 effort=50.0 velocity=10.0 -> lower=-2.4522 upper=2.4522 effort=50.0 velocity=10.0; origin xyz=0.0665 0 -0.019 rpy=0 0 3.1416 -> xyz=0.0679 0.01985 0 rpy=0 0 3.1416
- joint LH_KFE: axis 0 0 1 -> 0 -1 0; limit lower=-0.7854 upper=1.2217 effort=50.0 velocity=10.0 -> lower=-0.74002 upper=1.1868 effort=50.0 velocity=10.0; origin xyz=-0.14936 -0.16017 -0.052 rpy=0 0 0 -> xyz=-0.14936 0.058 -0.16017 rpy=0 0 0
- joint LH_Shank_2_Foot: origin xyz=0.165 -0.151 -0.0185 rpy=0 0 0 -> xyz=0.165 0.0205 -0.151 rpy=0 0 0
- joint RF_HAA: limit lower=-0.34907 upper=0.5236 effort=50.0 velocity=10.0 -> lower=-0.43633 upper=0.5236 effort=50.0 velocity=10.0; origin xyz=0.197 -0.054 0 rpy=-1.5708 0 0 -> xyz=0.2021 -0.054 0 rpy=0 0 0
- joint RF_HFE: axis 0 0 1 -> 0 -1 0; limit lower=-0.87266 upper=2.5307 effort=50.0 velocity=10.0 -> lower=-1.6668 upper=3.2376 effort=50.0 velocity=10.0; origin xyz=0.0665 0 -0.019 rpy=3.1416 0 0 -> xyz=0.0679 -0.01985 0 rpy=0 0 0
- joint RF_KFE: axis 0 0 1 -> 0 -1 0; limit lower=-0.7854 upper=1.2217 effort=50.0 velocity=10.0 -> lower=-0.74002 upper=1.1868 effort=50.0 velocity=10.0; origin xyz=-0.14936 -0.16017 0.052 rpy=0 0 0 -> xyz=-0.14936 -0.058 -0.16017 rpy=0 0 0
- joint RF_Shank_2_Foot: origin xyz=0.165 -0.151 0.0185 rpy=0 0 0 -> xyz=0.165 -0.0205 -0.151 rpy=0 0 0
- joint RH_HAA: limit lower=-0.5236 upper=0.87266 effort=50.0 velocity=10.0 -> lower=-0.83776 upper=0.5236 effort=50.0 velocity=10.0; origin xyz=-0.197 -0.054 0 rpy=-1.5708 0 3.1416 -> xyz=-0.2021 -0.054 0 rpy=0 0 3.1416
- joint RH_HFE: axis 0 0 1 -> 0 -1 0; limit lower=-2.5307 upper=0.87266 effort=50.0 velocity=10.0 -> lower=-2.4522 upper=2.4522 effort=50.0 velocity=10.0; origin xyz=0.0665 0 0.019 rpy=0 0 3.1416 -> xyz=0.0665 -0.01985 0 rpy=0 0 3.1416
- joint RH_KFE: axis 0 0 1 -> 0 -1 0; limit lower=-0.7854 upper=1.2217 effort=50.0 velocity=10.0 -> lower=-0.74002 upper=1.1868 effort=50.0 velocity=10.0; origin xyz=-0.14936 -0.16017 0.052 rpy=0 0 0 -> xyz=-0.14936 -0.058 -0.16017 rpy=0 0 0
- joint RH_Shank_2_Foot: origin xyz=0.165 -0.151 0.0185 rpy=0 0 0 -> xyz=0.165 -0.0205 -0.151 rpy=0 0 0

File: urdf/ayg.xacro (robot description, xacro)
@@ -3,4 +3,6 @@
   <xacro:arg name="use_gazebo" default="False" />
   <xacro:property name="use_gazebo" default="$(arg use_gazebo)" />
+  <xacro:arg name="has_camera" default="False" />
+  <xacro:property name="has_camera" default="$(arg has_camera)" />
   <xacro:arg name="initial_configuration" default="lying_down" />
   <xacro:property name="initial_configuration" value="$(arg initial_configuration)" />
@@ -17,15 +19,15 @@
     <inertial>
       <origin
-        xyz="0.000442764791303709 0.00323410160779704 0.000245694936587104"
+        xyz="0.00057686 -0.00018498 0.0026529"
         rpy="0 0 0" />
       <mass
-        value="8.43904999246817" />
+        value="9.1298" />
       <inertia
-        ixx="0.020065303439704"
-        ixy="4.08404656288191E-05"
-        ixz="-2.29078687506071E-14"
-        iyy="0.0384358501598642"
-        iyz="-2.71859452435122E-15"
-        izz="0.0267905011857108" />
+        ixx="0.022082"
+        ixy="3.2369E-07"
+        ixz="6.8653E-05"
+        iyy="0.031986"
+        iyz="2.8565E-07"
+        izz="0.040389" />
     </inertial>
     <visual>
@@ -40,5 +42,5 @@
         name="">
         <color
-          rgba="0.698039215686274 0.698039215686274 0.698039215686274 1" />
+          rgba="0.69804 0.69804 0.69804 1" />
       </material>
     </visual>
@@ -52,20 +54,19 @@
     </collision>
   </link>
-  <xacro:include filename="$(find ayg_description)/urdf/legs.xacro" />
   <link
     name="IMU">
     <inertial>
       <origin
-        xyz="-8.67049396793524E-18 0.02 5.37094698008006E-18"
+        xyz="-1.26817788945405E-05 -3.05893593341006E-06 0.00502425421604302"
         rpy="0 0 0" />
       <mass
-        value="0.08" />
+        value="0.0181381899874512" />
       <inertia
-        ixx="2.13333333333333E-05"
-        ixy="-4.34540023236298E-22"
-        ixz="-1.52363539595465E-21"
-        iyy="2.73333333333333E-05"
-        iyz="-2.43977500178881E-21"
-        izz="2.73333333333333E-05" />
+        ixx="4.80017459218422E-06"
+        ixy="-6.17315963282016E-11"
+        ixz="-1.66852937330168E-09"
+        iyy="3.40477341509462E-06"
+        iyz="-3.279931989329E-11"
+        izz="7.92679226862755E-06" />
     </inertial>
     <visual>
@@ -88,6 +89,6 @@
     type="fixed">
     <origin
-      xyz="0 0 0.006"
-      rpy="-1.5708 0 1.5708" />
+      xyz="-3.79309829856879E-05 0 -0.0172341687059438"
+      rpy="0 0 0" />
     <parent
       link="Base" />
@@ -97,99 +98,7 @@
       xyz="0 0 0" />
   </joint>
-  <link
-    name="Neck">
-    <inertial>
-      <origin
-        xyz="0 0 0"
-        rpy="0 0 0" />
-      <mass
-        value="0" />
-      <inertia
-        ixx="0"
-        ixy="0"
-        ixz="0"
-        iyy="0"
-        iyz="0"
-        izz="0" />
-    </inertial>
-    <visual>
-      <origin
-        xyz="0 0 0"
-        rpy="0 0 0" />
-      <geometry>
-        <mesh
-          filename="package://ayg_description/meshes/Neck.STL" />
-      </geometry>
-      <material
-        name="">
-        <color
-          rgba="1 1 1 1" />
-      </material>
-    </visual>
-  </link>
-  <joint
-    name="Base_2_Neck"
-    type="fixed">
-    <origin
-      xyz="0.2615 0 0.0249999999999999"
-      rpy="1.5707963267949 0 1.5707963267949" />
-    <parent
-      link="Base" />
-    <child
-      link="Neck" />
-    <axis
-      xyz="0 0 0" />
-  </joint>
-  <link
-    name="Camera">
-    <inertial>
-      <origin
-        xyz="7.0525E-18 -2.7756E-17 0.013"
-        rpy="0 0 0" />
-      <mass
-        value="0.16948" />
-      <inertia
-        ixx="2.085E-05"
-        ixy="5.6809E-20"
-        ixz="-7.2863E-20"
-        iyy="0.00020719"
-        iyz="3.3881E-21"
-        izz="0.00020895" />
-    </inertial>
-    <visual>
-      <origin
-        xyz="0 0 0"
-        rpy="0 0 0" />
-      <geometry>
-        <mesh
-          filename="package://ayg_description/meshes/Camera.STL" />
-      </geometry>
-      <material
-        name="">
-        <color
-          rgba="0.25098 0.25098 0.25098 1" />
-      </material>
-    </visual>
-    <collision>
-      <origin
-        xyz="0 -0.0025 0"
-        rpy="-0.288975409992567 0 0" />
-      <geometry>
-        <box size="0.13 0.035 0.05"/>
-      </geometry>
-    </collision>
-  </link>
-  <joint
-    name="Neck_2_Camera"
-    type="fixed">
-    <origin
-      xyz="0 0.0166603444360147 0.0804068913666247"
-      rpy="0.288975409992567 0 0" />
-    <parent
-      link="Neck" />
-    <child
-      link="Camera" />
-    <axis
-      xyz="0 0 0" />
-  </joint>
+  <xacro:include filename="$(find ayg_description)/urdf/legs.xacro" />
+  <xacro:if value="${has_camera}">
+    <xacro:include filename="$(find ayg_description)/urdf/camera.xacro" />
+  </xacro:if>
 </robot>

File: urdf/legs.xacro (robot description, xacro)
@@ -7,21 +7,21 @@
         <xacro:if value="${FH == 'F'}">
           <origin
-            xyz="0.0624625305028617 0.000263588472359728 -0.00241409757946361"
+            xyz="0.063065 -0.0051556 -5.3332E-05"
             rpy="0 0 0" />
         </xacro:if>
         <xacro:unless value="${FH == 'F'}">
           <origin
-            xyz="0.062462530502862 0.000263588472360432 0.0024140975794637"
+            xyz="0.063077 0.0051556 -6.5344E-05"
             rpy="0 0 0" />
         </xacro:unless>
         <mass
-          value="1.00401999005125" />
-        <inertia
-          ixx="0.000584357699669872"
-          ixy="1.71578981310067E-06"
-          ixz="-2.61675027998363E-19"
-          iyy="0.000584539401732687"
-          iyz="-3.57751728713357E-20"
-          izz="0.00102756652010595" />
+          value="1.0709" />
+        <inertia
+          ixx="0.00078713"
+          ixy="-7.2738E-08"
+          ixz="-1.6354E-06"
+          iyy="0.0013471"
+          iyz="-2.2108E-07"
+          izz="0.00073074" />
       </inertial>
       <visual>
@@ -42,5 +42,5 @@
           name="">
           <color
-            rgba="0.698039215686274 0.698039215686274 0.698039215686274 1" />
+            rgba="0.69804 0.69804 0.69804 1" />
         </material>
       </visual>
@@ -48,6 +48,6 @@
         <collision>
           <origin
-            xyz="0.0665 0 ${0.019+0.015}"
-            rpy="0 0 0" />
+            xyz="0.0665 0.034 0"
+            rpy="${PI/2} 0 0" />
           <geometry>
             <cylinder radius="0.05" length="0.13"/>
@@ -58,6 +58,6 @@
         <collision>
           <origin
-            xyz="0.0665 0 ${-0.019-0.015}"
-            rpy="0 0 0" />
+            xyz="0.0665 0.034 0"
+            rpy="${PI/2} 0 0" />
           <geometry>
             <cylinder radius="0.05" length="0.13"/>
@@ -71,11 +71,11 @@
       <xacro:if value="${FH == 'F'}">
         <origin
-          xyz="0.197 0.054 0"
-          rpy="-1.5708 0 0" />
-      </xacro:if>
-      <xacro:unless value="${FH == 'F'}">
-        <origin
-          xyz="-0.197 0.054 0"
-          rpy="-1.5708 0 3.1416" />
+          xyz="0.2021 0.054 0"
+          rpy="0 0 0" />
+      </xacro:if>
+      <xacro:unless value="${FH == 'F'}">
+        <origin
+          xyz="-0.2021 0.054 0"
+          rpy="0 0 3.1416" />
       </xacro:unless>
       <parent
@@ -88,5 +88,5 @@
         <limit
           lower="-0.5236"
-          upper="0.34907"
+          upper="0.43633"
           effort="${effort_lim}"
           velocity="${velocity_lim}" />
@@ -96,6 +96,6 @@
         xyz="-1 0 0" />
         <limit
-          lower="-0.87266"
-          upper="0.5236"
+          lower="-0.5236"
+          upper="0.83776"
           effort="${effort_lim}"
           velocity="${velocity_lim}" />
@@ -106,15 +106,15 @@
       <inertial>
         <origin
-          xyz="-0.00815740476229621 -0.00912689407030123 -0.0420066354122466"
-          rpy="0 0 0" />
-        <mass
-          value="1.15974999242447" />
-        <inertia
-          ixx="0.000911992879302287"
-          ixy="-0.000310524680951164"
-          ixz="-4.3266057977693E-16"
-          iyy="0.00091897366461706"
-          iyz="-1.93894477964206E-06"
-          izz="0.00169326046596367" />
+          xyz="-0.0095261 0.047418 -0.010869"
+          rpy="0 0 0" />
+        <mass
+          value="1.361" />
+        <inertia
+          ixx="0.0012156"
+          ixy="1.025E-06"
+          ixz="-0.00042254"
+          iyy="0.0022368"
+          iyz="-1.3825E-06"
+          izz="0.0012227" />
       </inertial>
       <visual>
@@ -129,11 +129,11 @@
           name="">
           <color
-            rgba="0.698039215686274 0.698039215686274 0.698039215686274 1" />
-        </material>
-      </visual>
-      <collision>
-        <origin
-          xyz="-0.0975 -0.075 -0.07"
-          rpy="0 ${PI/2} ${PI/4}" />
+            rgba="0.69804 0.69804 0.69804 1" />
+        </material>
+      </visual>
+      <collision>
+        <origin
+          xyz="-0.0975 +0.08 -0.07"
+          rpy="${PI/4} 0 ${PI/2}" />
         <geometry>
           <box size="0.025 0.05 0.14"/>
@@ -146,10 +146,10 @@
       <xacro:if value="${FH == 'F'}">
         <origin
-          xyz="0.0665 0 0.019"
-          rpy="3.1416 0 0" />
-      </xacro:if>
-      <xacro:unless value="${FH == 'F'}">
-        <origin
-          xyz="0.0665 0 -0.019"
+          xyz="0.0679 0.01985 0"
+          rpy="0 0 0" />
+      </xacro:if>
+      <xacro:unless value="${FH == 'F'}">
+        <origin
+          xyz="0.0679 0.01985 0"
           rpy="0 0 3.1416" />
       </xacro:unless>
@@ -159,16 +159,16 @@
         link="L${FH}_Thigh" />
       <axis
-        xyz="0 0 1" />
-      <xacro:if value="${FH == 'F'}">
-        <limit
-          lower="-0.87266"
-          upper="2.5307"
-          effort="${effort_lim}"
-          velocity="${velocity_lim}" />
-      </xacro:if>
-      <xacro:unless value="${FH == 'F'}">
-        <limit
-          lower="-2.5307"
-          upper="0.87266"
+        xyz="0 -1 0" />
+      <xacro:if value="${FH == 'F'}">
+        <limit
+          lower="-1.6668"
+          upper="3.2376"
+          effort="${effort_lim}"
+          velocity="${velocity_lim}" />
+      </xacro:if>
+      <xacro:unless value="${FH == 'F'}">
+        <limit
+          lower="-2.4522"
+          upper="2.4522"
           effort="${effort_lim}"
           velocity="${velocity_lim}" />
@@ -179,15 +179,15 @@
       <inertial>
         <origin
-          xyz="0.0630329536265654 -0.047817827674744 -0.0185"
-          rpy="0 0 0" />
-        <mass
-          value="0.102570008997248" />
-        <inertia
-          ixx="0.00029767764878727"
-          ixy="0.000296980915761884"
-          ixz="1.63288326545704E-19"
-          iyy="0.000327832614532812"
-          iyz="-1.54063121876522E-19"
-          izz="0.000624546801244392" />
+          xyz="0.059297 0.0205 -0.044894"
+          rpy="0 0 0" />
+        <mass
+          value="0.19753" />
+        <inertia
+          ixx="0.00059399"
+          ixy="-3.3081E-19"
+          ixz="0.00058611"
+          iyy="0.0012346"
+          iyz="3.1645E-19"
+          izz="0.00065333" />
       </inertial>
       <visual>
@@ -202,11 +202,11 @@
           name="">
           <color
-            rgba="0.698039215686274 0.698039215686274 0.698039215686274 1" />
-        </material>
-      </visual>
-      <collision>
-        <origin
-          xyz="0 0 -0.02"
-          rpy="0 0 0" />
+            rgba="0.69804 0.69804 0.69804 1" />
+        </material>
+      </visual>
+      <collision>
+        <origin
+          xyz="0 0.02 0"
+          rpy="${PI/2} 0 0" />
         <geometry>
           <cylinder radius="0.025" length="0.03"/>
@@ -215,6 +215,6 @@
       <collision>
         <origin
-          xyz="0.08 -0.075 -0.02"
-          rpy="0 0 ${PI/4}" />
+          xyz="0.08 0.02 -0.075"
+          rpy="${PI/2} ${-PI/4} 0" />
         <geometry>
           <box size="0.025 0.165 0.0125"/>
@@ -226,5 +226,5 @@
       type="revolute">
       <origin
-        xyz="-0.14936 -0.16017 -0.052"
+        xyz="-0.14936 0.058 -0.16017"
         rpy="0 0 0" />
       <parent
@@ -233,8 +233,8 @@
         link="L${FH}_Shank" />
       <axis
-        xyz="0 0 1" />
+        xyz="0 -1 0" />
       <limit
-        lower="-0.7854"
-        upper="1.2217"
+        lower="-0.74002"
+        upper="1.1868"
         effort="${effort_lim}"
         velocity="${velocity_lim}" />
@@ -245,19 +245,19 @@
         <origin
           xyz="-2.77555756156289E-17 5.55111512312578E-17 0"
-          rpy="0 ${PI/2} 0" />
-        <mass
-          value="0.088054927521184" />
-        <inertia
-          ixx="4.09565481632907E-05"
-          ixy="-8.61058027358505E-21"
-          ixz="2.27932697045296E-20"
-          iyy="2.47049106026622E-05"
-          iyz="5.04870979341448E-29"
-          izz="2.47049106026622E-05" />
-      </inertial>
-      <visual>
-        <origin
-          xyz="0 0 0"
-          rpy="0 0 0" />
+          rpy="0 0 0" />
+        <mass
+          value="0.0701295110066971" />
+        <inertia
+          ixx="1.91783738418569E-05"
+          ixy="4.42768620674145E-20"
+          ixz="8.0334719824878E-35"
+          iyy="3.14806687325575E-05"
+          iyz="2.23148962310519E-20"
+          izz="1.91783738418569E-05" />
+      </inertial>
+      <visual>
+        <origin
+          xyz="0 0 0"
+          rpy="${PI/2} 0 0" />
         <geometry>
           <cylinder length="0.025" radius="0.030" />
@@ -266,11 +266,11 @@
           name="">
           <color
-            rgba="0.250980392156863 0.250980392156863 0.250980392156863 1" />
-        </material>
-      </visual>
-      <collision>
-        <origin
-          xyz="0 0 0"
-          rpy="0 0 0" />
+            rgba="0.29804 0.29804 0.29804 1" />
+        </material>
+      </visual>
+      <collision>
+        <origin
+          xyz="0 0 0"
+          rpy="${PI/2} 0 0" />
         <geometry>
           <cylinder length="0.025" radius="0.030" />
@@ -282,5 +282,5 @@
       type="fixed">
       <origin
-        xyz="0.165 -0.151 -0.0185"
+        xyz="0.165 0.0205 -0.151"
         rpy="0 0 0" />
       <parent
@@ -298,21 +298,21 @@
         <xacro:if value="${FH == 'F'}">
           <origin
-            xyz="0.062462530502862 0.000263588472360484 0.00241409757946365"
+            xyz="0.063077 0.0051556 -6.5344E-05"
             rpy="0 0 0" />
         </xacro:if>
         <xacro:unless value="${FH == 'F'}">
           <origin
-            xyz="0.0624625305028617 0.000263588472359603 -0.00241409757946362"
+            xyz="-0.063065 0.0051556 -5.3332E-05"
             rpy="0 0 0" />
         </xacro:unless>
         <mass
-          value="1.00401999005125" />
-        <inertia
-          ixx="0.000584357699669871"
-          ixy="1.71578981310067E-06"
-          ixz="-3.08533699148142E-19"
-          iyy="0.000584539401732687"
-          iyz="1.3310433650471E-20"
-          izz="0.00102756652010595" />
+          value="1.071" />
+        <inertia
+          ixx="0.00078713"
+          ixy="7.2742E-08"
+          ixz="-1.6354E-06"
+          iyy="0.0013471"
+          iyz="2.2108E-07"
+          izz="0.00073074" />
       </inertial>
       <visual>
@@ -333,5 +333,5 @@
           name="">
           <color
-            rgba="0.698039215686274 0.698039215686274 0.698039215686274 1" />
+            rgba="0.69804 0.69804 0.69804 1" />
         </material>
       </visual>
@@ -339,6 +339,6 @@
         <collision>
           <origin
-            xyz="0.0665 0 ${-0.019-0.015}"
-            rpy="0 0 0" />
+            xyz="0.0665 -0.034 0"
+            rpy="${PI/2} 0 0" />
           <geometry>
             <cylinder radius="0.05" length="0.13"/>
@@ -349,6 +349,6 @@
         <collision>
           <origin
-            xyz="0.0665 0 ${+0.019+0.015}"
-            rpy="0 0 0" />
+            xyz="0.0665 -0.034 0"
+            rpy="${PI/2} 0 0" />
           <geometry>
             <cylinder radius="0.05" length="0.13"/>
@@ -362,11 +362,11 @@
       <xacro:if value="${FH == 'F'}">
         <origin
-          xyz="0.197 -0.054 0"
-          rpy="-1.5708 0 0" />
-      </xacro:if>
-      <xacro:unless value="${FH == 'F'}">
-        <origin
-          xyz="-0.197 -0.054 0"
-          rpy="-1.5708 0 3.1416" />
+          xyz="0.2021 -0.054 0"
+          rpy="0 0 0" />
+      </xacro:if>
+      <xacro:unless value="${FH == 'F'}">
+        <origin
+          xyz="-0.2021 -0.054 0"
+          rpy="0 0 3.1416" />
       </xacro:unless>
       <parent
@@ -378,5 +378,5 @@
         xyz="1 0 0" />
         <limit
-          lower="-0.34907"
+          lower="-0.43633"
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