Commit message: Bug fix

File: urdf/ayg.urdf (robot description, URDF)
Before this commit: robot ayg, 18 links, 17 joints
Links:
- link LF_Hip: geometry collision cylinder length=0.148 radius=0.05; visual mesh filename=package://ayg_description/meshes/L_Hip.STL
- link LH_Hip: geometry collision cylinder length=0.148 radius=0.05; visual mesh filename=package://ayg_description/meshes/R_Hip.STL
- link RF_Hip: geometry collision cylinder length=0.148 radius=0.05; visual mesh filename=package://ayg_description/meshes/R_Hip.STL
- link RH_Hip: geometry collision cylinder length=0.148 radius=0.05; visual mesh filename=package://ayg_description/meshes/L_Hip.STL
Joints:
- joint LH_HFE: origin xyz=0.0679 0.01985 0 rpy=0 0 3.1416 -> xyz=0.0679 -0.01985 0 rpy=0 0 3.1416
- joint RH_HFE: origin xyz=0.0665 -0.01985 0 rpy=0 0 3.1416 -> xyz=0.0665 0.01985 0 rpy=0 0 3.1416

File: urdf/legs.xacro (robot description, xacro)
@@ -48,8 +48,8 @@
         <collision>
           <origin
-            xyz="0.0665 0.034 0"
+            xyz="0.0665 0.04 0"
             rpy="${PI/2} 0 0" />
           <geometry>
-            <cylinder radius="0.05" length="0.13"/>
+            <cylinder radius="0.05" length="0.148"/>
           </geometry>
         </collision>
@@ -58,8 +58,8 @@
         <collision>
           <origin
-            xyz="0.0665 0.034 0"
+            xyz="0.0665 -0.04 0"
             rpy="${PI/2} 0 0" />
           <geometry>
-            <cylinder radius="0.05" length="0.13"/>
+            <cylinder radius="0.05" length="0.148"/>
           </geometry>
         </collision>
@@ -151,5 +151,5 @@
       <xacro:unless value="${FH == 'F'}">
         <origin
-          xyz="0.0679 0.01985 0"
+          xyz="0.0679 -0.01985 0"
           rpy="0 0 3.1416" />
       </xacro:unless>
@@ -339,8 +339,8 @@
         <collision>
           <origin
-            xyz="0.0665 -0.034 0"
+            xyz="0.0665 -0.04 0"
             rpy="${PI/2} 0 0" />
           <geometry>
-            <cylinder radius="0.05" length="0.13"/>
+            <cylinder radius="0.05" length="0.148"/>
           </geometry>
         </collision>
@@ -349,8 +349,8 @@
         <collision>
           <origin
-            xyz="0.0665 -0.034 0"
+            xyz="0.0665 0.04 0"
             rpy="${PI/2} 0 0" />
           <geometry>
-            <cylinder radius="0.05" length="0.13"/>
+            <cylinder radius="0.05" length="0.148"/>
           </geometry>
         </collision>
@@ -442,5 +442,5 @@
       <xacro:unless value="${FH == 'F'}">
         <origin
-          xyz="0.0665 -0.01985 0"
+          xyz="0.0665 0.01985 0"
           rpy="0 0 3.1416" />
       </xacro:unless>

Commit message: Simplify feet collision geometries into spheres

File: urdf/ayg.urdf (robot description, URDF)
Before this commit: robot ayg, 18 links, 17 joints
Links:
- link LF_Foot: geometry collision sphere radius=0.030; visual cylinder length=0.025 radius=0.030
- link LH_Foot: geometry collision sphere radius=0.030; visual cylinder length=0.025 radius=0.030
- link RF_Foot: geometry collision sphere radius=0.030; visual cylinder length=0.025 radius=0.030
- link RH_Foot: geometry collision sphere radius=0.030; visual cylinder length=0.025 radius=0.030

File: urdf/legs.xacro (robot description, xacro)
@@ -261,5 +261,5 @@
           rpy="${PI/2} 0 0" />
         <geometry>
-          <cylinder length="0.025" radius="0.030" />
+          <sphere radius="0.030"/>
         </geometry>
         <material
@@ -274,5 +274,5 @@
           rpy="${PI/2} 0 0" />
         <geometry>
-          <cylinder length="0.025" radius="0.030" />
+          <sphere radius="0.030"/>
         </geometry>
       </collision>
@@ -552,5 +552,5 @@
           rpy="${PI/2} 0 0" />
         <geometry>
-          <cylinder length="0.025" radius="0.030" />
+          <sphere radius="0.030"/>
         </geometry>
         <material
@@ -565,5 +565,5 @@
           rpy="${PI/2} 0 0" />
         <geometry>
-          <cylinder length="0.025" radius="0.030" />
+          <sphere radius="0.030"/>
         </geometry>
       </collision>

Commit message: #11 issue

File: urdf/ayg.urdf (robot description, URDF)
Before this commit: robot ayg, 18 links, 17 joints
Links:
- added link Battery_Left, mass 1.6; collision box size=0.177 0.079 0.096; visual box size=0.177 0.079 0.096
- added link Battery_Right, mass 1.6; collision box size=0.177 0.079 0.096; visual box size=0.177 0.079 0.096
- link Base: mass 9.1298 -> 9.148
Joints:
- added joint Base_2_Battery_Left: type fixed, parent Base, child Battery_Left, origin xyz=0 0.075 0 rpy=0 0 0, axis 0 0 0
- added joint Base_2_Battery_Right: type fixed, parent Base, child Battery_Right, origin xyz=0 -0.075 0 rpy=0 0 0, axis 0 0 0

File: urdf/ayg.xacro (robot description, xacro)
@@ -39,5 +39,5 @@
         rpy="0 0 0" />
       <mass
-        value="9.1298" />
+        value="9.148" />
       <inertia
         ixx="0.022082"
@@ -115,4 +115,73 @@
       xyz="0 0 0" />
   </joint>
+  <!-- Batteries (2x, side-by-side inside body cavity) -->
+  <link name="Battery_Left">
+    <inertial>
+      <origin xyz="0 0 0" rpy="0 0 0" />
+      <mass value="1.6" />
+      <inertia
+        ixx="0.002061"
+        ixy="0"
+        ixz="0"
+        iyy="0.005406"
+        iyz="0"
+        izz="0.005009" />
+    </inertial>
+    <visual>
+      <origin xyz="0 0 0" rpy="0 0 0" />
+      <geometry>
+        <box size="0.177 0.079 0.096" />
+      </geometry>
+      <material name="battery_color">
+        <color rgba="0.2 0.2 0.3 1" />
+      </material>
+    </visual>
+    <collision>
+      <origin xyz="0 0 0" rpy="0 0 0" />
+      <geometry>
+        <box size="0.177 0.079 0.096" />
+      </geometry>
+    </collision>
+  </link>
+  <joint name="Base_2_Battery_Left" type="fixed">
+    <origin xyz="0 0.075 0" rpy="0 0 0" />
+    <parent link="Base" />
+    <child link="Battery_Left" />
+    <axis xyz="0 0 0" />
+  </joint>
+  <link name="Battery_Right">
+    <inertial>
+      <origin xyz="0 0 0" rpy="0 0 0" />
+      <mass value="1.6" />
+      <inertia
+        ixx="0.002061"
+        ixy="0"
+        ixz="0"
+        iyy="0.005406"
+        iyz="0"
+        izz="0.005009" />
+    </inertial>
+    <visual>
+      <origin xyz="0 0 0" rpy="0 0 0" />
+      <geometry>
+        <box size="0.177 0.079 0.096" />
+      </geometry>
+      <material name="battery_color">
+        <color rgba="0.2 0.2 0.3 1" />
+      </material>
+    </visual>
+    <collision>
+      <origin xyz="0 0 0" rpy="0 0 0" />
+      <geometry>
+        <box size="0.177 0.079 0.096" />
+      </geometry>
+    </collision>
+  </link>
+  <joint name="Base_2_Battery_Right" type="fixed">
+    <origin xyz="0 -0.075 0" rpy="0 0 0" />
+    <parent link="Base" />
+    <child link="Battery_Right" />
+    <axis xyz="0 0 0" />
+  </joint>
   <xacro:include filename="$(find ayg_description)/urdf/legs.xacro" />
   <xacro:if value="${camera}">

Commit message: correct positioned

File: urdf/ayg.urdf (robot description, URDF)
Before this commit: robot ayg, 20 links, 19 joints
Links:
- removed link Battery_Left
- removed link Battery_Right
- added link Battery_Front, mass 1.6; collision box size=0.079 0.177 0.096; visual box size=0.079 0.177 0.096
- added link Battery_Rear, mass 1.6; collision box size=0.079 0.177 0.096; visual box size=0.079 0.177 0.096
Joints:
- removed joint Base_2_Battery_Left
- removed joint Base_2_Battery_Right
- added joint Base_2_Battery_Front: type fixed, parent Base, child Battery_Front, origin xyz=0.10 0 0 rpy=0 0 0, axis 0 0 0
- added joint Base_2_Battery_Rear: type fixed, parent Base, child Battery_Rear, origin xyz=-0.10 0 0 rpy=0 0 0, axis 0 0 0

File: urdf/ayg.xacro (robot description, xacro)
@@ -115,14 +115,14 @@
       xyz="0 0 0" />
   </joint>
-  <!-- Batteries (2x, side-by-side inside body cavity) -->
-  <link name="Battery_Left">
+  <!-- Batteries (2x, front-to-back inside body cavity, under top hatches) -->
+  <link name="Battery_Front">
     <inertial>
       <origin xyz="0 0 0" rpy="0 0 0" />
       <mass value="1.6" />
       <inertia
-        ixx="0.002061"
+        ixx="0.005406"
         ixy="0"
         ixz="0"
-        iyy="0.005406"
+        iyy="0.002061"
         iyz="0"
         izz="0.005009" />
@@ -131,5 +131,5 @@
       <origin xyz="0 0 0" rpy="0 0 0" />
       <geometry>
-        <box size="0.177 0.079 0.096" />
+        <box size="0.079 0.177 0.096" />
       </geometry>
       <material name="battery_color">
@@ -140,23 +140,23 @@
       <origin xyz="0 0 0" rpy="0 0 0" />
       <geometry>
-        <box size="0.177 0.079 0.096" />
+        <box size="0.079 0.177 0.096" />
       </geometry>
     </collision>
   </link>
-  <joint name="Base_2_Battery_Left" type="fixed">
-    <origin xyz="0 0.075 0" rpy="0 0 0" />
+  <joint name="Base_2_Battery_Front" type="fixed">
+    <origin xyz="0.10 0 0" rpy="0 0 0" />
     <parent link="Base" />
-    <child link="Battery_Left" />
+    <child link="Battery_Front" />
     <axis xyz="0 0 0" />
   </joint>
-  <link name="Battery_Right">
+  <link name="Battery_Rear">
     <inertial>
       <origin xyz="0 0 0" rpy="0 0 0" />
       <mass value="1.6" />
       <inertia
-        ixx="0.002061"
+        ixx="0.005406"
         ixy="0"
         ixz="0"
-        iyy="0.005406"
+        iyy="0.002061"
         iyz="0"
         izz="0.005009" />
@@ -165,5 +165,5 @@
       <origin xyz="0 0 0" rpy="0 0 0" />
       <geometry>
-        <box size="0.177 0.079 0.096" />
+        <box size="0.079 0.177 0.096" />
       </geometry>
       <material name="battery_color">
@@ -174,12 +174,12 @@
       <origin xyz="0 0 0" rpy="0 0 0" />
       <geometry>
-        <box size="0.177 0.079 0.096" />
+        <box size="0.079 0.177 0.096" />
       </geometry>
     </collision>
   </link>
-  <joint name="Base_2_Battery_Right" type="fixed">
-    <origin xyz="0 -0.075 0" rpy="0 0 0" />
+  <joint name="Base_2_Battery_Rear" type="fixed">
+    <origin xyz="-0.10 0 0" rpy="0 0 0" />
     <parent link="Base" />
-    <child link="Battery_Right" />
+    <child link="Battery_Rear" />
     <axis xyz="0 0 0" />
   </joint>

Commit message: with correct CAD values

File: urdf/ayg.urdf (robot description, URDF)
Before this commit: robot ayg, 20 links, 19 joints
Joints:
- joint Base_2_Battery_Front: origin xyz=0.10 0 0 rpy=0 0 0 -> xyz=0.10070 0 -0.00900 rpy=0 0 0
- joint Base_2_Battery_Rear: origin xyz=-0.10 0 0 rpy=0 0 0 -> xyz=-0.10070 0 -0.00900 rpy=0 0 0

File: urdf/ayg.xacro (robot description, xacro)
@@ -15,4 +15,26 @@
   <xacro:property name="velocity_lim" value="10.0" />
   <xacro:property name="PI" value="3.1415926535897931" />
+  <!-- Battery inertial properties (CAD export → URDF frame)
+       CAD frame: X=forward, Y=up, Z=left  |  URDF frame: X=forward, Y=left, Z=up
+       Mapping: (URDF_x, URDF_y, URDF_z) = (CAD_x, CAD_z, CAD_y)
+       CAD mass: 1.55217 kg  |  Weighed: 1.6 kg each  |  Housing mass is in Base -->
+  <xacro:property name="battery_cad_mass" value="1.55217" />
+  <xacro:property name="battery_real_mass" value="1.6" />
+  <xacro:property name="battery_inertia_scale" value="${battery_real_mass / battery_cad_mass}" />
+  <!-- CoM in battery link frame (URDF, meters) -->
+  <xacro:property name="battery_com_x" value="-0.00002" />
+  <xacro:property name="battery_com_y" value="-0.00421" />
+  <xacro:property name="battery_com_z" value="0.04143" />
+  <!-- Inertia at CoM, at CAD mass, URDF frame (kg·m²) -->
+  <xacro:property name="battery_cad_ixx" value="0.0043243903" />
+  <xacro:property name="battery_cad_ixy" value="-0.0000040621" />
+  <xacro:property name="battery_cad_ixz" value="-0.0000050483" />
+  <xacro:property name="battery_cad_iyy" value="0.0074475647" />
+  <xacro:property name="battery_cad_iyz" value="-0.0002587481" />
+  <xacro:property name="battery_cad_izz" value="0.0043149743" />
+  <!-- Battery positions relative to Base (URDF, meters) -->
+  <xacro:property name="battery_front_x" value="0.10070" />
+  <xacro:property name="battery_rear_x" value="-0.10070" />
+  <xacro:property name="battery_pos_z" value="-0.00900" />
   <xacro:if value="${sim}">
     <xacro:include filename="$(find ayg_description)/urdf/ayg_sim_ros2_control.xacro" />
@@ -118,13 +140,13 @@
   <link name="Battery_Front">
     <inertial>
-      <origin xyz="0 0 0" rpy="0 0 0" />
-      <mass value="1.6" />
-      <inertia
-        ixx="0.005406"
-        ixy="0"
-        ixz="0"
-        iyy="0.002061"
-        iyz="0"
-        izz="0.005009" />
+      <origin xyz="${battery_com_x} ${battery_com_y} ${battery_com_z}" rpy="0 0 0" />
+      <mass value="${battery_real_mass}" />
+      <inertia
+        ixx="${battery_cad_ixx * battery_inertia_scale}"
+        ixy="${battery_cad_ixy * battery_inertia_scale}"
+        ixz="${battery_cad_ixz * battery_inertia_scale}"
+        iyy="${battery_cad_iyy * battery_inertia_scale}"
+        iyz="${battery_cad_iyz * battery_inertia_scale}"
+        izz="${battery_cad_izz * battery_inertia_scale}" />
     </inertial>
     <visual>
@@ -145,5 +167,5 @@
   </link>
   <joint name="Base_2_Battery_Front" type="fixed">
-    <origin xyz="0.10 0 0" rpy="0 0 0" />
+    <origin xyz="${battery_front_x} 0 ${battery_pos_z}" rpy="0 0 0" />
     <parent link="Base" />
     <child link="Battery_Front" />
@@ -152,13 +174,13 @@
   <link name="Battery_Rear">
     <inertial>
-      <origin xyz="0 0 0" rpy="0 0 0" />
-      <mass value="1.6" />
-      <inertia
-        ixx="0.005406"
-        ixy="0"
-        ixz="0"
-        iyy="0.002061"
-        iyz="0"
-        izz="0.005009" />
+      <origin xyz="${battery_com_x} ${battery_com_y} ${battery_com_z}" rpy="0 0 0" />
+      <mass value="${battery_real_mass}" />
+      <inertia
+        ixx="${battery_cad_ixx * battery_inertia_scale}"
+        ixy="${battery_cad_ixy * battery_inertia_scale}"
+        ixz="${battery_cad_ixz * battery_inertia_scale}"
+        iyy="${battery_cad_iyy * battery_inertia_scale}"
+        iyz="${battery_cad_iyz * battery_inertia_scale}"
+        izz="${battery_cad_izz * battery_inertia_scale}" />
     </inertial>
     <visual>
@@ -179,5 +201,5 @@
   </link>
   <joint name="Base_2_Battery_Rear" type="fixed">
-    <origin xyz="-0.10 0 0" rpy="0 0 0" />
+    <origin xyz="${battery_rear_x} 0 ${battery_pos_z}" rpy="0 0 0" />
     <parent link="Base" />
     <child link="Battery_Rear" />

Commit message: Fix robot weight values in description files (#5)
* #11 issue

* correct positioned

* with correct CAD values

* Remove .vscode/

* Use macro for batteries

---------

Co-authored-by: Hovsepyan Miqayel <hovsepyanmiqyel23@gmail.com>
Co-authored-by: Davide De Benedittis <davide.debenedittis@gmail.com>

File: urdf/ayg.urdf (robot description, URDF)
Before this commit: robot ayg, 18 links, 17 joints
Links:
- added link Battery_Front, mass 1.6; collision box size=0.079 0.177 0.096; visual box size=0.079 0.177 0.096
- added link Battery_Rear, mass 1.6; collision box size=0.079 0.177 0.096; visual box size=0.079 0.177 0.096
- link Base: mass 9.1298 -> 9.148
Joints:
- added joint Base_2_Battery_Front: type fixed, parent Base, child Battery_Front, origin xyz=0.10070 0 -0.00900 rpy=0 0 0, axis 0 0 0
- added joint Base_2_Battery_Rear: type fixed, parent Base, child Battery_Rear, origin xyz=-0.10070 0 -0.00900 rpy=0 0 0, axis 0 0 0

File: urdf/ayg.xacro (robot description, xacro)
@@ -15,4 +15,26 @@
   <xacro:property name="velocity_lim" value="10.0" />
   <xacro:property name="PI" value="3.1415926535897931" />
+  <!-- Battery inertial properties (CAD export → URDF frame)
+       CAD frame: X=forward, Y=up, Z=left  |  URDF frame: X=forward, Y=left, Z=up
+       Mapping: (URDF_x, URDF_y, URDF_z) = (CAD_x, CAD_z, CAD_y)
+       CAD mass: 1.55217 kg  |  Weighed: 1.6 kg each  |  Housing mass is in Base -->
+  <xacro:property name="battery_cad_mass" value="1.55217" />
+  <xacro:property name="battery_real_mass" value="1.6" />
+  <xacro:property name="battery_inertia_scale" value="${battery_real_mass / battery_cad_mass}" />
+  <!-- CoM in battery link frame (URDF, meters) -->
+  <xacro:property name="battery_com_x" value="-0.00002" />
+  <xacro:property name="battery_com_y" value="-0.00421" />
+  <xacro:property name="battery_com_z" value="0.04143" />
+  <!-- Inertia at CoM, at CAD mass, URDF frame (kg·m²) -->
+  <xacro:property name="battery_cad_ixx" value="0.0043243903" />
+  <xacro:property name="battery_cad_ixy" value="-0.0000040621" />
+  <xacro:property name="battery_cad_ixz" value="-0.0000050483" />
+  <xacro:property name="battery_cad_iyy" value="0.0074475647" />
+  <xacro:property name="battery_cad_iyz" value="-0.0002587481" />
+  <xacro:property name="battery_cad_izz" value="0.0043149743" />
+  <!-- Battery positions relative to Base (URDF, meters) -->
+  <xacro:property name="battery_front_x" value="0.10070" />
+  <xacro:property name="battery_rear_x" value="-0.10070" />
+  <xacro:property name="battery_pos_z" value="-0.00900" />
   <xacro:if value="${sim}">
     <xacro:include filename="$(find ayg_description)/urdf/ayg_sim_ros2_control.xacro" />
@@ -38,6 +60,7 @@
         xyz="0.00057686 -0.00018498 0.0026529"
         rpy="0 0 0" />
+      <!-- Measured: 9.148 kg (CAD: 9.1298 kg) -->
       <mass
-        value="9.1298" />
+        value="9.148" />
       <inertia
         ixx="0.022082"
@@ -115,4 +138,43 @@
       xyz="0 0 0" />
   </joint>
+  <!-- Battery macro (2x identical packs, front and rear) -->
+  <xacro:macro name="battery" params="name pos_x">
+    <link name="Battery_${name}">
+      <inertial>
+        <origin xyz="${battery_com_x} ${battery_com_y} ${battery_com_z}" rpy="0 0 0" />
+        <mass value="${battery_real_mass}" />
+        <inertia
+          ixx="${battery_cad_ixx * battery_inertia_scale}"
+          ixy="${battery_cad_ixy * battery_inertia_scale}"
+          ixz="${battery_cad_ixz * battery_inertia_scale}"
+          iyy="${battery_cad_iyy * battery_inertia_scale}"
+          iyz="${battery_cad_iyz * battery_inertia_scale}"
+          izz="${battery_cad_izz * battery_inertia_scale}" />
+      </inertial>
+      <visual>
+        <origin xyz="0 0 0" rpy="0 0 0" />
+        <geometry>
+          <box size="0.079 0.177 0.096" />
+        </geometry>
+        <material name="battery_color">
+          <color rgba="0.2 0.2 0.3 1" />
+        </material>
+      </visual>
+      <collision>
+        <origin xyz="0 0 0" rpy="0 0 0" />
+        <geometry>
+          <box size="0.079 0.177 0.096" />
+        </geometry>
+      </collision>
+    </link>
+    <joint name="Base_2_Battery_${name}" type="fixed">
+      <origin xyz="${pos_x} 0 ${battery_pos_z}" rpy="0 0 0" />
+      <parent link="Base" />
+      <child link="Battery_${name}" />
+      <axis xyz="0 0 0" />
+    </joint>
+  </xacro:macro>
+  <xacro:battery name="Front" pos_x="${battery_front_x}" />
+  <xacro:battery name="Rear"  pos_x="${battery_rear_x}" />
   <xacro:include filename="$(find ayg_description)/urdf/legs.xacro" />
   <xacro:if value="${camera}">
