Commit message: Add Intel RealSense D555 to AYG: URDF frames, Gazebo depth sensor, driver frame alignment (#7)
* #6 Add Intel RealSense D555

* Regenerate urdf/ayg.urdf with D555 camera link tree

Follow-up housekeeping to PR #6 (Add D555 RealSense camera link tree).
That PR intentionally left urdf/ayg.urdf dormant because ROS launches invoke
xacro at runtime. Isaac Lab consumes the static .urdf directly, however
(UrdfFileCfg in cf_lab tasks), so the unregenerated dormant file caused
spawn failures of the depth sensor's parent prim Camera_depth_optical_frame.

This commit refreshes the auto-generated artifact so it matches the xacro
source: 974 lines, 59 Camera_* link references, full RealSense optical
frame chain. Source xacro and Gazebo plugin block are unchanged.

No code or behavior change for ROS launches (they still call xacro). Isaac
Lab now loads the up-to-date URDF without needing per-machine working-tree
regeneration.

* camera: explicit massless inertials on D555 reference frames

Isaac Sim's URDF importer silently assigns mass=1.0 kg to any link
without an <inertial> tag. Across the 14 D555 reference frames
(Camera_body, *_frame, *_optical_frame, imu) this injected +14 kg
of phantom mass rigid-fixed to Base, breaking the AYG locomotion
teacher in Isaac Lab (98% base-contact faceplant after a few
seconds of episode).

Fix:
- Add <xacro:massless_frame> macro in camera.xacro emitting an
  explicit epsilon inertial (mass=1e-6, inertia=1e-9 diagonal).
- Use the macro for every reference-frame link in the D555 tree.
- Patch the static urdf/ayg.urdf artifact the same way (Isaac Lab
  consumes that file directly via cf_lab AYG_CFG.asset_path).
- Physical Camera link (mass 0.3912 kg, visual, collision) is
  untouched.

Real hardware and robot_state_publisher are unaffected — they only
consume TF, never inertia.

Verified by rolling out the Phase 1 teacher checkpoint
(Teacher_baseline/model_9999.pt) in Isaac Lab on Isaac-Velocity-
Rough-Ayg-v0 with 50 envs x 2000 steps:
  before: 98% base_contact, mean ep-len 3.33s, robot mass 37.5 kg
  after:  14% base_contact, mean ep-len 18.80s, robot mass 23.56 kg
matching the pre-camera-tree URDF baseline (5-7%).

* camera: place D555 optical center inside housing, raise Camera link 1 cm

Two changes to the camera transform chain:

- Base_2_Camera xyz z: 0.095 -> 0.105 (raise mount 1 cm to mirror the
  planned hardware bracket revision).
- Camera_body_joint xyz: 0 0 0 -> 0.0527 -0.024 0 (place the D450
  optical-module reference at +5.27 cm fwd and -2.4 cm vertical from
  the Camera link origin in robot body convention, so depth, IR1/IR2,
  color and IMU all sit inside the physical housing instead of at the
  mounting point).

After these changes, the depth optical center in Base is (0.3002, 0,
0.081). The D555 stereo baseline (95 mm) and depth-to-color offset
(47.5 mm) continue to match the datasheet because all downstream sensor
frames inherit from the shifted Camera_body. realsense2_camera per-unit
calibrated TFs continue to supersede these nominal values on the real
robot.

Closes the longstanding 0-vs-real-mount divergence in the camera link
tree: Gazebo, robot_state_publisher and Isaac Lab now all see the same
geometry.

* camera: fix Gazebo depth CameraInfo intrinsics + add RGB color sensor

Add explicit <lens><intrinsics> to the D555 depth sensor so gz-sim Fortress
publishes the configured 640x360/87deg model in CameraInfo (K) instead of its
320x240/60deg default. Without this the reconstructed depth cloud is skewed and
drooping. NOTE gz applies this only to K, not the projection matrix P; the
companion ayg_gazebo fix_depth_camera_info node copies K->P for consumers.

Add an RGB color sensor on Camera_color_frame so /camera/Camera/color/image_raw
has a producer in Gazebo (the image was otherwise black).

* camera: raise MuJoCo camera mount z 0.095 -> 0.105 to match URDF/Isaac

The MuJoCo model still used the pre-bracket-revision camera height
(z=0.095), 1 cm below the URDF Base_2_Camera joint and the Isaac Lab
depth-sensor config, which both place the D555 mount at
(0.2475, 0, 0.105) in Base. Update the Camera_visual geom and the
Camera_color camera so all robot models agree.

---------

Co-authored-by: Hovsepyan Miqayel <hovsepyanmiqyel23@gmail.com>

File: urdf/ayg.urdf (robot description, URDF)
Before this commit: robot ayg, 20 links, 19 joints
Links:
- added link Camera, mass 0.3912; collision mesh filename=package://ayg_description/meshes/Camera.STL; visual mesh filename=package://ayg_description/meshes/Camera.STL
- added link Camera_accel_frame, mass 1e-6
- added link Camera_accel_optical_frame, mass 1e-6
- added link Camera_body, mass 1e-6
- added link Camera_color_frame, mass 1e-6
- added link Camera_color_optical_frame, mass 1e-6
- added link Camera_depth_frame, mass 1e-6
- added link Camera_depth_optical_frame, mass 1e-6
- added link Camera_gyro_frame, mass 1e-6
- added link Camera_gyro_optical_frame, mass 1e-6
- added link Camera_imu_optical_frame, mass 1e-6
- added link Camera_infra1_frame, mass 1e-6
- added link Camera_infra1_optical_frame, mass 1e-6
- added link Camera_infra2_frame, mass 1e-6
- added link Camera_infra2_optical_frame, mass 1e-6
Joints:
- added joint Base_2_Camera: type fixed, parent Base, child Camera, origin xyz=0.2475 0 0.105 rpy=1.5708 0 0, axis 0 0 0
- added joint Camera_accel_joint: type fixed, parent Camera_body, child Camera_accel_frame, origin xyz=0.0114 -0.0195 0.0 rpy=0 0 0
- added joint Camera_accel_optical_joint: type fixed, parent Camera_accel_frame, child Camera_accel_optical_frame, origin xyz=0 0 0 rpy=-1.5707963267948966 0 -1.5707963267948966
- added joint Camera_body_joint: type fixed, parent Camera, child Camera_body, origin xyz=0.0527 -0.024 0 rpy=-1.5707963267948966 0 0
- added joint Camera_color_joint: type fixed, parent Camera_body, child Camera_color_frame, origin xyz=0 -0.0475 0 rpy=0 0 0
- added joint Camera_color_optical_joint: type fixed, parent Camera_color_frame, child Camera_color_optical_frame, origin xyz=0 0 0 rpy=-1.5707963267948966 0 -1.5707963267948966
- added joint Camera_depth_joint: type fixed, parent Camera_body, child Camera_depth_frame, origin xyz=0 0 0 rpy=0 0 0
- added joint Camera_depth_optical_joint: type fixed, parent Camera_depth_frame, child Camera_depth_optical_frame, origin xyz=0 0 0 rpy=-1.5707963267948966 0 -1.5707963267948966
- added joint Camera_gyro_joint: type fixed, parent Camera_body, child Camera_gyro_frame, origin xyz=0.0114 -0.0195 0.0 rpy=0 0 0
- added joint Camera_gyro_optical_joint: type fixed, parent Camera_gyro_frame, child Camera_gyro_optical_frame, origin xyz=0 0 0 rpy=-1.5707963267948966 0 -1.5707963267948966
- added joint Camera_imu_optical_joint: type fixed, parent Camera_gyro_optical_frame, child Camera_imu_optical_frame, origin xyz=0 0 0 rpy=0 0 0
- added joint Camera_infra1_joint: type fixed, parent Camera_body, child Camera_infra1_frame, origin xyz=0 0.0 0 rpy=0 0 0
- added joint Camera_infra1_optical_joint: type fixed, parent Camera_infra1_frame, child Camera_infra1_optical_frame, origin xyz=0 0 0 rpy=-1.5707963267948966 0 -1.5707963267948966
- added joint Camera_infra2_joint: type fixed, parent Camera_body, child Camera_infra2_frame, origin xyz=0 -0.095 0 rpy=0 0 0
- added joint Camera_infra2_optical_joint: type fixed, parent Camera_infra2_frame, child Camera_infra2_optical_frame, origin xyz=0 0 0 rpy=-1.5707963267948966 0 -1.5707963267948966
- joint Base_2_Battery_Front: origin xyz=0.10070 0 -0.00900 rpy=0 0 0 -> xyz=0.1007 0 -0.009 rpy=0 0 0
- joint Base_2_Battery_Rear: origin xyz=-0.10070 0 -0.00900 rpy=0 0 0 -> xyz=-0.1007 0 -0.009 rpy=0 0 0

File: urdf/camera.xacro (robot description, xacro)
@@ -1,56 +1,251 @@
 <?xml version="1.0"?>
 <robot xmlns:xacro="http://www.ros.org/wiki/xacro">
-  <link
-    name="Camera">
+  <!--
+    Intel RealSense D555 (RGB-D + IMU, D450 optical module, PoE).
+    Housing: 167 x 42 x 48 mm, baseline 95 mm, weight 337 g (D555 datasheet v1.1).
+    Sensor-internal extrinsics are nominal D450-module values taken from
+    realsense2_description/urdf/_d585.urdf.xacro (same optical module).
+    realsense2_camera publishes per-unit calibrated TFs at runtime that
+    supersede these nominal values.
+  -->
+  <xacro:property name="M_PI" value="3.1415926535897931"/>
+  <xacro:property name="d555_depth_to_infra1_offset" value="0.0"/>
+  <xacro:property name="d555_depth_to_infra2_offset" value="-0.095"/>
+  <xacro:property name="d555_depth_to_color_offset"  value="-0.0475"/>
+  <xacro:property name="d555_imu_px" value="0.0114"/>
+  <xacro:property name="d555_imu_py" value="-0.0195"/>
+  <xacro:property name="d555_imu_pz" value="0.0"/>
+  <!--
+    Massless reference frame for TF purposes only (depth/color/infra/IMU
+    optical frames). An explicit epsilon-mass inertial is required because
+    physics simulators (Isaac Sim, Gazebo) silently assign a 1.0 kg default
+    to any link without <inertial>. Across 14 D555 reference frames that
+    silently injected +14 kg of phantom mass rigid-fixed to Base — enough
+    to faceplant the AYG locomotion policy in Isaac Lab. Real hardware /
+    robot_state_publisher are unaffected (TF-only consumers ignore inertia).
+  -->
+  <xacro:macro name="massless_frame" params="name">
+    <link name="${name}">
+      <inertial>
+        <origin xyz="0 0 0" rpy="0 0 0"/>
+        <mass value="1e-6"/>
+        <inertia ixx="1e-9" ixy="0" ixz="0" iyy="1e-9" iyz="0" izz="1e-9"/>
+      </inertial>
+    </link>
+  </xacro:macro>
+  <!-- Physical Camera body (mesh + inertials from SolidWorks export). -->
+  <link name="Camera">
     <inertial>
-      <origin
-        xyz="0.027539 -0.0054988 -1.4524E-08"
-        rpy="0 0 0" />
-      <mass
-        value="0.3912" />
-      <inertia
-        ixx="0.00080723"
-        ixy="4.4453E-06"
-        ixz="-1.7833E-09"
-        iyy="0.00082275"
-        iyz="2.4795E-09"
-        izz="0.00010329" />
+      <origin xyz="0.027539 -0.0054988 -1.4524E-08" rpy="0 0 0"/>
+      <mass value="0.3912"/>
+      <inertia ixx="0.00080723" ixy="4.4453E-06" ixz="-1.7833E-09"
+               iyy="0.00082275" iyz="2.4795E-09" izz="0.00010329"/>
     </inertial>
     <visual>
-      <origin
-        xyz="0 0 0"
-        rpy="0 0 0" />
+      <origin xyz="0 0 0" rpy="0 0 0"/>
       <geometry>
-        <mesh
-          filename="package://ayg_description/meshes/Camera.STL" />
+        <mesh filename="package://ayg_description/meshes/Camera.STL"/>
       </geometry>
-      <material
-        name="">
-        <color
-          rgba="0.69804 0.69804 0.69804 1" />
+      <material name="">
+        <color rgba="0.69804 0.69804 0.69804 1"/>
       </material>
     </visual>
     <collision>
-      <origin
-        xyz="0 0 0"
-        rpy="0 0 0" />
+      <origin xyz="0 0 0" rpy="0 0 0"/>
       <geometry>
-        <mesh
-          filename="package://ayg_description/meshes/Camera.STL" />
+        <mesh filename="package://ayg_description/meshes/Camera.STL"/>
       </geometry>
     </collision>
   </link>
-  <joint
-    name="Base_2_Camera"
-    type="fixed">
-    <origin
-      xyz="0.2475 0 0.095"
-      rpy="1.5708 0 0" />
-    <parent
-      link="Base" />
-    <child
-      link="Camera" />
-    <axis
-      xyz="0 0 0" />
-  </joint>
+  <joint name="Base_2_Camera" type="fixed">
+    <origin xyz="0.2475 0 0.105" rpy="1.5708 0 0"/>
+    <parent link="Base"/>
+    <child link="Camera"/>
+    <axis xyz="0 0 0"/>
+  </joint>
+  <!--
+    Camera frame post-Base_2_Camera is (X-fwd, Y-up, Z-right) due to the
+    90 deg roll in the parent joint. Camera_body undoes that roll so the
+    RealSense optical-frame convention (rpy="-pi/2 0 -pi/2" => Z-fwd) works
+    as in realsense2_description.
+    The xyz=(0.0527 -0.024 0) translation here places Camera_body at the
+    D450 optical-module reference point inside the housing: +5.27 cm forward
+    and -2.4 cm vertical (down) from the Camera link origin in robot body
+    convention. Camera link's local Y axis is Base +Z (up) due to the 90 deg
+    roll above, so -0.024 along local Y = 2.4 cm down in body frame; local Z
+    is Base -Y, so 0 leaves the optical module on the body centerline. Depth,
+    color, IR1/IR2 baselines and IMU offsets all inherit from this corrected
+    Camera_body position so the whole D555 sensor stack sits where it
+    physically does on the robot.
+  -->
+  <xacro:massless_frame name="Camera_body"/>
+  <joint name="Camera_body_joint" type="fixed">
+    <origin xyz="0.0527 -0.024 0" rpy="${-M_PI/2} 0 0"/>
+    <parent link="Camera"/>
+    <child link="Camera_body"/>
+  </joint>
+  <!-- Depth (left IR is depth origin in D450 module). -->
+  <xacro:massless_frame name="Camera_depth_frame"/>
+  <joint name="Camera_depth_joint" type="fixed">
+    <origin xyz="0 0 0" rpy="0 0 0"/>
+    <parent link="Camera_body"/>
+    <child link="Camera_depth_frame"/>
+  </joint>
+  <xacro:massless_frame name="Camera_depth_optical_frame"/>
+  <joint name="Camera_depth_optical_joint" type="fixed">
+    <origin xyz="0 0 0" rpy="${-M_PI/2} 0 ${-M_PI/2}"/>
+    <parent link="Camera_depth_frame"/>
+    <child link="Camera_depth_optical_frame"/>
+  </joint>
+  <!-- Left IR imager (coincident with depth origin). -->
+  <xacro:massless_frame name="Camera_infra1_frame"/>
+  <joint name="Camera_infra1_joint" type="fixed">
+    <origin xyz="0 ${d555_depth_to_infra1_offset} 0" rpy="0 0 0"/>
+    <parent link="Camera_body"/>
+    <child link="Camera_infra1_frame"/>
+  </joint>
+  <xacro:massless_frame name="Camera_infra1_optical_frame"/>
+  <joint name="Camera_infra1_optical_joint" type="fixed">
+    <origin xyz="0 0 0" rpy="${-M_PI/2} 0 ${-M_PI/2}"/>
+    <parent link="Camera_infra1_frame"/>
+    <child link="Camera_infra1_optical_frame"/>
+  </joint>
+  <!-- Right IR imager (95 mm baseline; sign per D555 datasheet + D585 xacro). -->
+  <xacro:massless_frame name="Camera_infra2_frame"/>
+  <joint name="Camera_infra2_joint" type="fixed">
+    <origin xyz="0 ${d555_depth_to_infra2_offset} 0" rpy="0 0 0"/>
+    <parent link="Camera_body"/>
+    <child link="Camera_infra2_frame"/>
+  </joint>
+  <xacro:massless_frame name="Camera_infra2_optical_frame"/>
+  <joint name="Camera_infra2_optical_joint" type="fixed">
+    <origin xyz="0 0 0" rpy="${-M_PI/2} 0 ${-M_PI/2}"/>
+    <parent link="Camera_infra2_frame"/>
+    <child link="Camera_infra2_optical_frame"/>
+  </joint>
+  <!-- RGB sensor. -->
+  <xacro:massless_frame name="Camera_color_frame"/>
+  <joint name="Camera_color_joint" type="fixed">
+    <origin xyz="0 ${d555_depth_to_color_offset} 0" rpy="0 0 0"/>
+    <parent link="Camera_body"/>
+    <child link="Camera_color_frame"/>
+  </joint>
+  <xacro:massless_frame name="Camera_color_optical_frame"/>
+  <joint name="Camera_color_optical_joint" type="fixed">
+    <origin xyz="0 0 0" rpy="${-M_PI/2} 0 ${-M_PI/2}"/>
+    <parent link="Camera_color_frame"/>
+    <child link="Camera_color_optical_frame"/>
+  </joint>
+  <!-- IMU (accel + gyro share the same physical position on D450 module). -->
+  <xacro:massless_frame name="Camera_accel_frame"/>
+  <joint name="Camera_accel_joint" type="fixed">
+    <origin xyz="${d555_imu_px} ${d555_imu_py} ${d555_imu_pz}" rpy="0 0 0"/>
+    <parent link="Camera_body"/>
+    <child link="Camera_accel_frame"/>
+  </joint>
+  <xacro:massless_frame name="Camera_accel_optical_frame"/>
+  <joint name="Camera_accel_optical_joint" type="fixed">
+    <origin xyz="0 0 0" rpy="${-M_PI/2} 0 ${-M_PI/2}"/>
+    <parent link="Camera_accel_frame"/>
+    <child link="Camera_accel_optical_frame"/>
+  </joint>
+  <xacro:massless_frame name="Camera_gyro_frame"/>
+  <joint name="Camera_gyro_joint" type="fixed">
+    <origin xyz="${d555_imu_px} ${d555_imu_py} ${d555_imu_pz}" rpy="0 0 0"/>
+    <parent link="Camera_body"/>
+    <child link="Camera_gyro_frame"/>
+  </joint>
+  <xacro:massless_frame name="Camera_gyro_optical_frame"/>
+  <joint name="Camera_gyro_optical_joint" type="fixed">
+    <origin xyz="0 0 0" rpy="${-M_PI/2} 0 ${-M_PI/2}"/>
+    <parent link="Camera_gyro_frame"/>
+    <child link="Camera_gyro_optical_frame"/>
+  </joint>
+  <xacro:massless_frame name="Camera_imu_optical_frame"/>
+  <joint name="Camera_imu_optical_joint" type="fixed">
+    <origin xyz="0 0 0" rpy="0 0 0"/>
+    <parent link="Camera_gyro_optical_frame"/>
+    <child link="Camera_imu_optical_frame"/>
+  </joint>
+  <!--
+    Gazebo Ignition (Fortress) depth sensor.
+    Renders along Camera_depth_frame's +X axis (forward in robot body).
+    Topic and frame_id are chosen to match real-hardware realsense2_camera
+    when launched with camera_name=Camera (see ayg_bringup/launch/ayg.launch.py).
+    Resolution + FoV + clip range mirror D555 datasheet v1.1 depth specs.
+  -->
+  <gazebo reference="Camera_depth_frame">
+    <sensor name="d555_depth" type="depth_camera">
+      <update_rate>30</update_rate>
+      <topic>camera/Camera/depth/image_rect_raw</topic>
+      <gz_frame_id>Camera_depth_optical_frame</gz_frame_id>
+      <camera>
+        <horizontal_fov>1.5184</horizontal_fov>  <!-- 87 deg -->
+        <!--
+          Explicit intrinsics: gz-sim Fortress otherwise populates CameraInfo
+          with its default 320x240/60deg model (fx=277, cx=160, cy=120) instead
+          of the configured 640x360/87deg. NOTE gz applies this only to the K
+          matrix, not P; a small republisher copies K->P (ayg_gazebo
+          fix_depth_camera_info.py + depth_cloud.launch.py) so depth_image_proc
+          and RViz reconstruct an aligned point cloud.
+          fx=fy=(width/2)/tan(hfov/2)=337.2, cx=width/2, cy=height/2.
+        -->
+        <lens>
+          <intrinsics>
+            <fx>337.2</fx>
+            <fy>337.2</fy>
+            <cx>320.0</cx>
+            <cy>180.0</cy>
+            <s>0.0</s>
+          </intrinsics>
+        </lens>
+        <image>
+          <width>640</width>
+          <height>360</height>
+          <format>R_FLOAT32</format>
+        </image>
+        <clip>
+          <near>0.26</near>  <!-- D555 Min-Z at VGA -->
+          <far>9.0</far>     <!-- D555 ideal range upper bound -->
+        </clip>
+      </camera>
+      <always_on>1</always_on>
+      <visualize>false</visualize>
+    </sensor>
+  </gazebo>
+  <!--
+    RGB color sensor. Without this the /camera/Camera/color/image_raw topic
+    has no producer in Gazebo (the image reads black). gz_frame_id +
+    intrinsics chosen to match real-hardware realsense2_camera color stream.
+  -->
+  <gazebo reference="Camera_color_frame">
+    <sensor name="d555_color" type="camera">
+      <update_rate>30</update_rate>
+      <topic>camera/Camera/color/image_raw</topic>
+      <gz_frame_id>Camera_color_optical_frame</gz_frame_id>
+      <camera>
+        <horizontal_fov>1.5184</horizontal_fov>  <!-- 87 deg -->
+        <lens>
+          <intrinsics>
+            <fx>337.2</fx>
+            <fy>337.2</fy>
+            <cx>320.0</cx>
+            <cy>180.0</cy>
+            <s>0.0</s>
+          </intrinsics>
+        </lens>
+        <image>
+          <width>640</width>
+          <height>360</height>
+          <format>R8G8B8</format>
+        </image>
+        <clip>
+          <near>0.1</near>
+          <far>100.0</far>
+        </clip>
+      </camera>
+      <always_on>1</always_on>
+      <visualize>false</visualize>
+    </sensor>
+  </gazebo>
 </robot>
