Commit message: Fix: manually update collision geometries to reasonable geometries

File: urdf/ayg.urdf (robot description, URDF)
Before this commit: robot ayg, 23 links, 22 joints
Links:
- removed link Camera
- removed link Camera_color_frame
- removed link Camera_color_optical_frame
- removed link Camera_depth_frame
- removed link Camera_depth_optical_frame
- link Base: geometry collision box size=0.44 0.239 0.122; visual mesh filename=package://ayg_description/meshes/Base.STL
- link LF_Foot: geometry collision sphere radius=0.032; visual cylinder length=0.031 radius=0.032
- link LF_Hip: geometry collision cylinder length=0.14 radius=0.055; visual mesh filename=package://ayg_description/meshes/L_Hip.STL
- link LF_Shank: geometry collision box size=0.02 0.017 0.18; collision cylinder length=0.031 radius=0.03
- link LF_Thigh: geometry collision box size=0.05 0.014 0.16; visual mesh filename=package://ayg_description/meshes/L_Thigh.STL
- link LH_Foot: geometry collision sphere radius=0.032; visual cylinder length=0.031 radius=0.032
- link LH_Hip: geometry collision cylinder length=0.14 radius=0.055; visual mesh filename=package://ayg_description/meshes/R_Hip.STL
- link LH_Shank: geometry collision box size=0.02 0.017 0.18; collision cylinder length=0.031 radius=0.03
- link LH_Thigh: geometry collision box size=0.05 0.014 0.16; visual mesh filename=package://ayg_description/meshes/L_Thigh.STL
- link RF_Foot: geometry collision sphere radius=0.032; visual cylinder length=0.031 radius=0.032
- link RF_Hip: geometry collision cylinder length=0.14 radius=0.055; visual mesh filename=package://ayg_description/meshes/R_Hip.STL
- link RF_Shank: geometry collision box size=0.02 0.017 0.18; collision cylinder length=0.031 radius=0.03
- link RF_Thigh: geometry collision box size=0.05 0.014 0.16; visual mesh filename=package://ayg_description/meshes/R_Thigh.STL
- link RH_Foot: geometry collision sphere radius=0.032; visual cylinder length=0.031 radius=0.032
- link RH_Hip: geometry collision cylinder length=0.14 radius=0.055; visual mesh filename=package://ayg_description/meshes/L_Hip.STL
- link RH_Shank: geometry collision box size=0.02 0.017 0.18; collision cylinder length=0.031 radius=0.03
- link RH_Thigh: geometry collision box size=0.05 0.014 0.16; visual mesh filename=package://ayg_description/meshes/R_Thigh.STL
Joints:
- removed joint Base_2_Camera
- removed joint Camera_color_joint
- removed joint Camera_color_optical_joint
- removed joint Camera_depth_joint
- removed joint Camera_depth_optical_joint

File: urdf/ayg.xacro (robot description, xacro)
@@ -7,5 +7,5 @@
   <xacro:arg name="gazebo_version" default="fortress" />
   <xacro:property name="gazebo_version" value="$(arg gazebo_version)" />
-  <xacro:arg name="camera" default="True" />
+  <xacro:arg name="camera" default="False" />
   <xacro:property name="camera" default="$(arg camera)" />
   <xacro:arg name="initial_configuration" default="lying_down" />
@@ -68,10 +68,14 @@
       </material>
     </visual>
+    <!-- Trunk collision: axis-aligned box wrapping the Base mesh body (AABB
+         0.444 x 0.239 x 0.187 centred at z=0.0055). Height is kept to the main
+         body (0.14); the narrow top mount rail (z up to 0.099, only +/-0.06
+         wide) is left out so the box does not over-claim empty space beside it. -->
     <collision>
       <origin
-        xyz="0 0 0"
+        xyz="0 0 0.0"
         rpy="0 0 0" />
       <geometry>
-        <box size="0.42 0.23 0.14" />
+        <box size="0.44 0.239 0.122" />
       </geometry>
     </collision>

File: urdf/camera.xacro (robot description, xacro)
@@ -62,7 +62,7 @@
     -->
     <collision>
-      <origin xyz="0.0121 -0.0062 0" rpy="0 0 0"/>
+      <origin xyz="0.025 -0.0025 0" rpy="0 0 -0.25"/>
       <geometry>
-        <box size="0.0942 0.053 0.1669"/>
+        <box size="0.06 0.04 0.13"/>
       </geometry>
     </collision>

File: urdf/legs.xacro (robot description, xacro)
@@ -42,8 +42,16 @@
         </material>
       </visual>
-      <collision>
-        <origin xyz="0.055 0 0" rpy="0 0 0" />
-        <geometry>
-          <box size="0.11 0.07 0.11" />
+      <!-- Hip: cylinder about the Y axis (the HFE motor barrel), wrapping the
+           disc-shaped hip housing. y-offset tracks the HFE side (front vs hind
+           use mirrored hip meshes: F -> L_Hip, H -> R_Hip). -->
+      <collision>
+        <xacro:if value="${FH == 'F'}">
+          <origin xyz="0.065 0.0375 0" rpy="1.5708 0 0" />
+        </xacro:if>
+        <xacro:unless value="${FH == 'F'}">
+          <origin xyz="0.065 -0.0375 0" rpy="1.5708 0 0" />
+        </xacro:unless>
+        <geometry>
+          <cylinder radius="0.055" length="0.14" />
         </geometry>
       </collision>
@@ -83,8 +91,10 @@
         </material>
       </visual>
-      <collision>
-        <origin xyz="-0.0786 0.0285 -0.1004" rpy="0 2.4474 2.7935" />
-        <geometry>
-          <box size="0.06 0.06 0.24" />
+      <!-- Thigh: slim box along the leg, rotated only about the Y swing axis
+           (single pitch, no roll/yaw twist), shortened at both ends for gaps. -->
+      <collision>
+        <origin xyz="-0.105 0.0734 -0.1" rpy="0 -2.4776 0" />
+        <geometry>
+          <box size="0.05 0.014 0.16" />
         </geometry>
       </collision>
@@ -119,8 +129,19 @@
         </material>
       </visual>
-      <collision>
-        <origin xyz="0.0852 0.0078 -0.0948" rpy="0 2.4073 0.0911" />
-        <geometry>
-          <box size="0.05 0.05 0.24" />
+      <!-- Shank: slim box along the leg, rotated only about the Y swing axis
+           (single pitch, no roll/yaw twist), shortened to leave gaps. -->
+      <collision>
+        <origin xyz="0.0867 0.0155 -0.0965" rpy="0 2.4093 0" />
+        <geometry>
+          <box size="0.02 0.017 0.18" />
+        </geometry>
+      </collision>
+      <!-- Knee joint filler: cylinder coaxial with the KFE (y) axis at the
+           joint. Coaxial => invariant under knee bend => bridges the thigh/shank
+           gap for external contacts without ever self-colliding with either. -->
+      <collision>
+        <origin xyz="0 0.0155 0" rpy="1.5708 0 0" />
+        <geometry>
+          <cylinder radius="0.03" length="0.031" />
         </geometry>
       </collision>
@@ -141,7 +162,9 @@
       </inertial>
       <visual>
-        <origin xyz="0 0 0" rpy="0 0 0" />
-        <geometry>
-          <mesh filename="package://ayg_description/meshes/Foot.STL" />
+        <!-- Foot: cylinder about the Y axis, replicating the Foot.STL mesh
+             (radius 0.032, length 0.031 spanning y = ±0.0155). -->
+        <origin xyz="0 0 0" rpy="1.5708 0 0" />
+        <geometry>
+          <cylinder radius="0.032" length="0.031" />
         </geometry>
         <material name="">
@@ -193,8 +216,16 @@
         </material>
       </visual>
-      <collision>
-        <origin xyz="0.055 0 0" rpy="0 0 0" />
-        <geometry>
-          <box size="0.11 0.07 0.11" />
+      <!-- Hip: cylinder about the Y axis (the HFE motor barrel), wrapping the
+           disc-shaped hip housing. y-offset tracks the HFE side (front vs hind
+           use mirrored hip meshes: F -> R_Hip, H -> L_Hip). Mirror of L_Leg. -->
+      <collision>
+        <xacro:if value="${FH == 'F'}">
+          <origin xyz="0.065 -0.0375 0" rpy="1.5708 0 0" />
+        </xacro:if>
+        <xacro:unless value="${FH == 'F'}">
+          <origin xyz="0.065 0.0375 0" rpy="1.5708 0 0" />
+        </xacro:unless>
+        <geometry>
+          <cylinder radius="0.055" length="0.14" />
         </geometry>
       </collision>
@@ -234,8 +265,10 @@
         </material>
       </visual>
-      <collision>
-        <origin xyz="-0.0786 -0.0285 -0.1004" rpy="0 2.4474 -2.7935" />
-        <geometry>
-          <box size="0.06 0.06 0.24" />
+      <!-- Thigh: slim box along the leg, rotated only about the Y swing axis
+           (single pitch, no roll/yaw twist), shortened at both ends for gaps. -->
+      <collision>
+        <origin xyz="-0.105 -0.0734 -0.1" rpy="0 -2.4776 0" />
+        <geometry>
+          <box size="0.05 0.014 0.16" />
         </geometry>
       </collision>
@@ -270,8 +303,19 @@
         </material>
       </visual>
-      <collision>
-        <origin xyz="0.0852 -0.0078 -0.0948" rpy="0 2.4073 -0.0911" />
-        <geometry>
-          <box size="0.05 0.05 0.24" />
+      <!-- Shank: slim box along the leg, rotated only about the Y swing axis
+           (single pitch, no roll/yaw twist), shortened to leave gaps. -->
+      <collision>
+        <origin xyz="0.0867 -0.0155 -0.0965" rpy="0 2.4093 0" />
+        <geometry>
+          <box size="0.02 0.017 0.18" />
+        </geometry>
+      </collision>
+      <!-- Knee joint filler: cylinder coaxial with the KFE (y) axis at the
+           joint. Coaxial => invariant under knee bend => bridges the thigh/shank
+           gap for external contacts without ever self-colliding with either. -->
+      <collision>
+        <origin xyz="0 -0.0155 0" rpy="1.5708 0 0" />
+        <geometry>
+          <cylinder radius="0.03" length="0.031" />
         </geometry>
       </collision>
@@ -292,7 +336,9 @@
       </inertial>
       <visual>
-        <origin xyz="0 0 0" rpy="0 0 0" />
-        <geometry>
-          <mesh filename="package://ayg_description/meshes/Foot.STL" />
+        <!-- Foot: cylinder about the Y axis, replicating the Foot.STL mesh
+             (radius 0.032, length 0.031 spanning y = ±0.0155). -->
+        <origin xyz="0 0 0" rpy="1.5708 0 0" />
+        <geometry>
+          <cylinder radius="0.032" length="0.031" />
         </geometry>
         <material name="">

Commit message: feat: exact-mesh top handle collision (handle_F/R.STL) in URDF + MuJoCo xml
Two small end-arch carry handles extracted from the Base.STL CAD mesh (front x=+0.21,
rear x=-0.21, span the base width, ~3.2 cm tall), added as Base collision geometry in
both sims (PhysX/MuJoCo convex-hull each arch). Recovery-critical: belly-up contact.
Validated harmless for the deployables (MuJoCo multi-init WITH handles: p8_01 100%,
s0175 91.7%); training model for the overnight_hd handle-aware batch (2026-07-14).

Clean-fix TODO: proper change belongs in ayg.xacro (Ayg repo) + URDF regen.

File: urdf/ayg.urdf (robot description, URDF)
Before this commit: robot ayg, 20 links, 19 joints
Links:
- link Base: geometry collision box size=0.4 0.23 0.12; collision mesh filename=package://ayg_description/meshes/handle_F.STL

Commit message: Rebase the 1.3 model onto SolidWorks export CF-AYG-1.3-00-000-URDF-7
URDF-7 fixes the thigh-to-chassis collision at extreme HFE angles (a known
thigh cable cover vs panel overlap remains and is ignored; the cover will
change). Same 19 links and joints as URDF-6; what moved:

* Masses everywhere: 22.948 -> 23.809 kg. Base +0.29, Head +0.09, each hip
  +0.064, each thigh +0.103 (redesigned part), each shank -0.061 (same
  envelope), each foot 0.040 -> 0.05447 (elastic tire; still the same solid
  cylinder r=0.032 L=0.031 inertia model). All CoMs and inertias re-read from
  the export; the thigh inertia is now an exact left/right mirror, so one
  signed block replaces the separate L/R values.
* HAA origins (+/-0.203, +/-0.054) -> (+/-0.201, +/-0.056). The export slid the
  HFE/KFE origins along their (y) axes -- kinematically null -- so the strut
  plane sits at y=0.0731 in the thigh frame and y=0.0156 in the shank frame;
  every leg collision primitive carries that offset, measured on the meshes.
  Foot track in Base changes by 0.5 mm.
* Shank_2_Foot z -0.189639 -> -0.19164: shank 0.2550 -> 0.2565 m, zero-pose
  base height 0.4225 -> 0.4245 m.
* Front HAA limits symmetric at +/-0.5236 (was 0.43633 outward).
* IMU 19 mm lower (Base_2_IMU z -0.00983 -> -0.02883).
* Head/LiDAR mount unchanged; the cage is 5 mm wider each side, which the
  primitives already left out.

Meshes: full URDF-7 set. Thigh dedup still holds (LF/LH agree to 0.07 mm, RF/RH
exactly). The right shank is the LF part translated -0.031164 in y, not a
mirror, so one Shank.STL remains and the right-side visual carries the shift.

Hip cylinder x offset 0.058 -> 0.060 so it stays at Base x=+/-0.261 (unchanged
Base-box and LiDAR clearances); its y/z are deliberately kept, since widening
it inboard would push its rim into the Head handle collider under +/-30 deg HAA.

Verified: the regenerated ayg.urdf matches the export on every link mass, CoM,
inertia, joint origin and limit (axis-flip aware); total 23.8093 kg; MuJoCo
loads mujoco/ayg.xml and a per-leg joint sweep shows the same wrapper
self-contact pairs as the URDF-6 model, with the hip-to-handle clearance at
full HAA up from 0.86 to 1.25 mm.

File: urdf/ayg.urdf (robot description, URDF)
Before this commit: robot ayg, 20 links, 19 joints
Links:
- link Base: mass 10.732 -> 11.02
- link Head: mass 0.72713 -> 0.81801
- link LF_Foot: mass 0.04 -> 0.05447
- link LF_Hip: mass 0.98111 -> 1.0451
- link LF_Shank: mass 0.34563 -> 0.28461
- link LF_Thigh: mass 1.5051 -> 1.6083
- link LH_Foot: mass 0.04 -> 0.05447
- link LH_Hip: mass 0.98111 -> 1.0451
- link LH_Shank: mass 0.34563 -> 0.28461
- link LH_Thigh: mass 1.5051 -> 1.6083
- link RF_Foot: mass 0.04 -> 0.05447
- link RF_Hip: mass 0.98111 -> 1.0451
- link RF_Shank: mass 0.34563 -> 0.28461
- link RF_Thigh: mass 1.5052 -> 1.6083
- link RH_Foot: mass 0.04 -> 0.05447
- link RH_Hip: mass 0.98111 -> 1.0451
- link RH_Shank: mass 0.34563 -> 0.28461
- link RH_Thigh: mass 1.5052 -> 1.6083
Joints:
- joint Base_2_IMU: origin xyz=0 0 -0.00983 rpy=0 0 0 -> xyz=0 0 -0.02883 rpy=0 0 0
- joint LF_HAA: limit lower=-0.5236 upper=0.43633 effort=50.0 velocity=10.0 -> lower=-0.5236 upper=0.5236 effort=50.0 velocity=10.0; origin xyz=0.203 0.054 0 rpy=0 0 0 -> xyz=0.201 0.056 0 rpy=0 0 0
- joint LF_HFE: origin xyz=0.063 0.0996 0 rpy=0 0 0 -> xyz=0.065 0.0215 0 rpy=0 0 0
- joint LF_KFE: origin xyz=-0.15715 -0.0035 -0.20082 rpy=0 0 0 -> xyz=-0.15715 0.057518 -0.20082 rpy=0 0 0
- joint LF_Shank_2_Foot: origin xyz=0.170476 0 -0.189639 rpy=0 0 0 -> xyz=0.17048 0.015582 -0.19164 rpy=0 0 0
- joint LH_HAA: origin xyz=-0.203 0.054 0 rpy=0 0 0 -> xyz=-0.201 0.056 0 rpy=0 0 0
- joint LH_HFE: origin xyz=-0.063 0.0996 0 rpy=0 0 0 -> xyz=-0.065 0.0215 0 rpy=0 0 0
- joint LH_KFE: origin xyz=-0.15715 -0.0035 -0.20082 rpy=0 0 0 -> xyz=-0.15715 0.057518 -0.20082 rpy=0 0 0
- joint LH_Shank_2_Foot: origin xyz=0.170476 0 -0.189639 rpy=0 0 0 -> xyz=0.17048 0.015582 -0.19164 rpy=0 0 0
- joint RF_HAA: limit lower=-0.43633 upper=0.5236 effort=50.0 velocity=10.0 -> lower=-0.5236 upper=0.5236 effort=50.0 velocity=10.0; origin xyz=0.203 -0.054 0 rpy=0 0 0 -> xyz=0.201 -0.056 0 rpy=0 0 0
- joint RF_HFE: origin xyz=0.063 -0.0996 0 rpy=0 0 0 -> xyz=0.065 -0.0215 0 rpy=0 0 0
- joint RF_KFE: origin xyz=-0.15715 0.0035 -0.20082 rpy=0 0 0 -> xyz=-0.15715 -0.057518 -0.20082 rpy=0 0 0
- joint RF_Shank_2_Foot: origin xyz=0.170476 0 -0.189639 rpy=0 0 0 -> xyz=0.17048 -0.015582 -0.19164 rpy=0 0 0
- joint RH_HAA: origin xyz=-0.203 -0.054 0 rpy=0 0 0 -> xyz=-0.201 -0.056 0 rpy=0 0 0
- joint RH_HFE: origin xyz=-0.063 -0.0996 0 rpy=0 0 0 -> xyz=-0.065 -0.0215 0 rpy=0 0 0
- joint RH_KFE: origin xyz=-0.15715 0.0035 -0.20082 rpy=0 0 0 -> xyz=-0.15715 -0.057518 -0.20082 rpy=0 0 0
- joint RH_Shank_2_Foot: origin xyz=0.170476 0 -0.189639 rpy=0 0 0 -> xyz=0.17048 -0.015582 -0.19164 rpy=0 0 0

File: urdf/ayg.xacro (robot description, xacro)
@@ -41,20 +41,22 @@
     name="Base">
     <inertial>
-      <!-- Ayg 1.3 SolidWorks export CF-AYG-1.3-00-000-URDF-6. Batteries are
+      <!-- Ayg 1.3 SolidWorks export CF-AYG-1.3-00-000-URDF-7. Batteries are
            rigidly fixed inside the chassis and are lumped into this Base
            mass/inertia (no separate Battery links), so the trunk is a single
-           rigid body. Whole-robot mass 22.948 kg across 19 links. -->
+           rigid body. Whole-robot mass 23.809 kg across 19 links. The Base
+           mesh envelope is unchanged from URDF-6, so the collision box below
+           still fits. -->
       <origin
-        xyz="-0.00030633 -0.0051482 -0.0019103"
+        xyz="-0.0005817 -1.9934E-05 -0.0020067"
         rpy="0 0 0" />
       <mass
-        value="10.732" />
+        value="11.02" />
       <inertia
-        ixx="0.029884"
-        ixy="4.1808E-07"
-        ixz="0.00015159"
-        iyy="0.038536"
-        iyz="1.5415E-07"
-        izz="0.055747" />
+        ixx="0.035479"
+        ixy="-3.4801E-06"
+        ixz="8.3812E-05"
+        iyy="0.032555"
+        iyz="0.00043953"
+        izz="0.055613" />
     </inertial>
     <visual>
@@ -90,5 +92,6 @@
        Gazebo/real IMU sensor is defined on the Base link (see
        ayg_sim_ros2_control.xacro), not on this link. Mass/inertia are the 1.3
-       CAD-export values (bare module, ~1.35 g); negligible vs the 23 kg total. -->
+       CAD-export values (bare module, ~1.35 g); negligible vs the 24 kg total.
+       URDF-7 moved the module 19 mm down (z -0.00983 -> -0.02883). -->
   <link
     name="IMU">
@@ -101,8 +104,8 @@
       <inertia
         ixx="4.0133E-08"
-        ixy="-6.9855E-14"
+        ixy="-6.9859E-14"
         ixz="8.9554E-12"
         iyy="5.9906E-08"
-        iyz="-1.4564E-14"
+        iyz="-1.4567E-14"
         izz="9.917E-08" />
     </inertial>
@@ -112,5 +115,5 @@
     type="fixed">
     <origin
-      xyz="0 0 -0.00983"
+      xyz="0 0 -0.02883"
       rpy="0 0 0" />
     <parent
@@ -123,5 +126,5 @@
   <xacro:include filename="$(find ayg_description)/urdf/legs.xacro" />
   <!-- Unconditional: unlike the optional D555 it replaces, the 1.3 head is
-       structural chassis (0.72713 kg fixed to Base, reaching 0.425 m forward).
+       structural chassis (0.81801 kg fixed to Base, reaching 0.425 m forward).
        Leaving it out would hand ayg_kindyn/Pinocchio a robot missing that mass
        and its pitch moment. The `lidar` arg inside gates only the sensor frame. -->

File: urdf/ayg_sim_ros2_control.xacro (robot description, xacro)
@@ -58,11 +58,12 @@
         <!--
             standing: the zero pose, feet directly below their HFE origins at a
-            0.4225 m base height. This is the 1.3 nominal stance: it equals the
-            cf_lab training init (every episode resets to all-zero joints), it
-            clears the JT128's 0.35 m near-field threshold (sensor at 0.413 m vs
-            0.330 m at the earlier 0.340 m carry-over), and it holds the lowest
-            static KFE torque of the workable range (9.2 vs 11.4 N*m per leg).
+            0.4245 m base height (URDF-7; 0.4225 on URDF-6). This is the 1.3
+            nominal stance: it equals the cf_lab training init (every episode
+            resets to all-zero joints), it clears the JT128's 0.35 m near-field
+            threshold (sensor at 0.415 m vs 0.330 m at the earlier 0.340 m
+            carry-over), and it holds the lowest static KFE torque of the
+            workable range (9.2 vs 11.4 N*m per leg at the URDF-6 masses).
             The KFE extension stop still leaves 0.565 rad (7.6 cm of base rise)
-            beyond it. Requires spawn_height above 0.4225 (simulate_ayg uses
+            beyond it. Requires spawn_height above 0.4245 (simulate_ayg uses
             0.45).
         -->
