Commit message: Rebase the 1.3 model onto SolidWorks export CF-AYG-1.3-00-000-URDF-7
URDF-7 fixes the thigh-to-chassis collision at extreme HFE angles (a known
thigh cable cover vs panel overlap remains and is ignored; the cover will
change). Same 19 links and joints as URDF-6; what moved:

* Masses everywhere: 22.948 -> 23.809 kg. Base +0.29, Head +0.09, each hip
  +0.064, each thigh +0.103 (redesigned part), each shank -0.061 (same
  envelope), each foot 0.040 -> 0.05447 (elastic tire; still the same solid
  cylinder r=0.032 L=0.031 inertia model). All CoMs and inertias re-read from
  the export; the thigh inertia is now an exact left/right mirror, so one
  signed block replaces the separate L/R values.
* HAA origins (+/-0.203, +/-0.054) -> (+/-0.201, +/-0.056). The export slid the
  HFE/KFE origins along their (y) axes -- kinematically null -- so the strut
  plane sits at y=0.0731 in the thigh frame and y=0.0156 in the shank frame;
  every leg collision primitive carries that offset, measured on the meshes.
  Foot track in Base changes by 0.5 mm.
* Shank_2_Foot z -0.189639 -> -0.19164: shank 0.2550 -> 0.2565 m, zero-pose
  base height 0.4225 -> 0.4245 m.
* Front HAA limits symmetric at +/-0.5236 (was 0.43633 outward).
* IMU 19 mm lower (Base_2_IMU z -0.00983 -> -0.02883).
* Head/LiDAR mount unchanged; the cage is 5 mm wider each side, which the
  primitives already left out.

Meshes: full URDF-7 set. Thigh dedup still holds (LF/LH agree to 0.07 mm, RF/RH
exactly). The right shank is the LF part translated -0.031164 in y, not a
mirror, so one Shank.STL remains and the right-side visual carries the shift.

Hip cylinder x offset 0.058 -> 0.060 so it stays at Base x=+/-0.261 (unchanged
Base-box and LiDAR clearances); its y/z are deliberately kept, since widening
it inboard would push its rim into the Head handle collider under +/-30 deg HAA.

Verified: the regenerated ayg.urdf matches the export on every link mass, CoM,
inertia, joint origin and limit (axis-flip aware); total 23.8093 kg; MuJoCo
loads mujoco/ayg.xml and a per-leg joint sweep shows the same wrapper
self-contact pairs as the URDF-6 model, with the hip-to-handle clearance at
full HAA up from 0.86 to 1.25 mm.

File: urdf/legs.xacro (robot description, xacro)
@@ -2,9 +2,11 @@
 <robot xmlns:xacro="http://www.ros.org/wiki/xacro">
   <!--
-    Legs, Ayg 1.3 (SolidWorks export CF-AYG-1.3-00-000-URDF-6).
+    Legs, Ayg 1.3 (SolidWorks export CF-AYG-1.3-00-000-URDF-7).
     One macro instantiated four times. `sx` = +1 front / -1 hind, `sy` = +1 left /
     -1 right; every joint origin and mirrored inertia term is written as an export
     value times those signs, so the file reads as a direct transcription of the
-    export and can be re-checked against a future one line by line.
+    export and can be re-checked against a future one line by line. Where the
+    export's four instances of a part disagree in the last digits (tessellation
+    noise, at most 4e-5 m / 1.6e-6 kg m^2), the LF value is the one written.
     Frames are the export's own placement, unchanged. Axes are normalized to the
     deployed convention: HAA about +x, HFE/KFE about -y (the export uses +y for
@@ -12,8 +14,15 @@
     negated-and-swapped limits). Because the HFE/KFE axes are parallel to y, the
     export's frame origins sit at an arbitrary point along the rotation axis -
-    sliding them in y is kinematically null, which is why the export's y offsets
-    differ from earlier revisions while the foot positions are identical.
-    Segment lengths: thigh |(-0.15715, -0.20082)| = shank |(0.170476, -0.189639)|
-    = 0.255 m exactly, so the leg extends 0.510 m hip-to-foot (was 0.443 m).
+    sliding them in y is kinematically null. URDF-7 slid the HFE origin 78 mm
+    inboard and the KFE origin 61 mm outboard relative to URDF-6, so the thigh's
+    strut plane now sits at y = 0.0731 (not -0.0035) in the thigh frame and the
+    shank/foot plane at y = 0.0156 (not 0) in the shank frame; the foot track in
+    the Base frame moved by only 0.5 mm. The collision primitives below carry
+    those y offsets.
+    Segment lengths: thigh |(-0.15715, -0.20082)| = 0.2550 m, shank
+    |(0.17048, -0.19164)| = 0.2565 m (URDF-6: 0.2550; the shank envelope is
+    unchanged, the foot centre moved 2 mm down its frame), so the leg extends
+    0.5115 m hip-to-foot and the zero pose puts Base 0.4245 m above ground
+    (0.20082 + 0.19164 + 0.032 foot radius).
   -->
   <xacro:macro name="ayg_leg" params="side FH sx sy">
@@ -24,8 +33,8 @@
     <link name="${side}${FH}_Hip">
       <inertial>
-        <origin xyz="${0.059856*sx} ${0.0023868*sy} ${1.6688E-05*sx*sy}" rpy="0 0 0" />
-        <mass value="0.98111" />
-        <inertia ixx="0.00070791" ixy="${1.6598E-06*sx*sy}" ixz="${9.3501E-07*sy}"
-                 iyy="0.0012845"  iyz="${-2.4177E-07*sx}"   izz="0.00087996" />
+        <origin xyz="${0.06215*sx} ${-0.0031317*sy} -0.00034351" rpy="0 0 0" />
+        <mass value="1.0451" />
+        <inertia ixx="0.00069698" ixy="${-1.5149E-06*sx*sy}" ixz="${1.4486E-05*sx}"
+                 iyy="0.0012902"  iyz="${-1.5206E-06*sy}"    izz="0.00084229" />
       </inertial>
       <visual>
@@ -39,28 +48,34 @@
       </visual>
       <!-- Hip housing AND HFE motor barrel: ONE cylinder about y, spanning the
-           whole HAA-to-HFE assembly (hip mesh y -0.0331..0.0250, barrel y
-           0.0235..0.1116 -> 0.0393 +/- 0.0725). This is the pre-1.3 arrangement:
-           the barrel is coaxial with the HFE axis, so carrying it on the parent
-           link is kinematically identical to carrying it on the thigh, and it
-           keeps one collider per hip instead of two.
-           The housing mesh is symmetric in z (+/-0.0513) but its two sides are
-           not: the top is roofed by the Head deck collider (underside z=+0.0455)
-           and can never touch anything, while the underside faces terrain and is
-           in the base_contact termination list. So the cylinder is r=0.047 with
-           its axis dropped to z=-0.0045 rather than r=0.053 centred: bottom
-           -0.0515 still covers the real underside (-0.0513), top +0.0425 clears
-           the deck by 3 mm. A symmetric shrink to r=0.044 would clear the deck
-           too but leave the exposed underside 7.3 mm short.
+           whole HAA-to-HFE assembly (hip mesh y -0.0376..0.0250, barrel y
+           0.0215..0.1071 in this frame). This is the pre-1.3 arrangement: the
+           barrel is coaxial with the HFE axis, so carrying it on the parent link
+           is kinematically identical to carrying it on the thigh, and it keeps
+           one collider per hip instead of two.
+           The housing mesh is near-symmetric in z (-0.0520..+0.0513) but its two
+           sides are not: the top is roofed by the Head deck collider (underside
+           z=+0.0455) and can never touch anything, while the underside faces
+           terrain and is in the base_contact termination list. So the cylinder
+           is r=0.047 with its axis dropped to z=-0.0045 rather than r=0.053
+           centred: bottom -0.0515 covers the real underside to within 0.5 mm,
+           top +0.0425 clears the deck by 3 mm. A symmetric shrink to r=0.044
+           would clear the deck too but leave the exposed underside 7.3 mm short.
+           The y span is deliberately NOT widened to the hip mesh's new inboard
+           end (-0.0376): under +/-30 deg HAA the inboard rim of this cylinder
+           rises to z=+0.0534, 0.5 mm under the Head handle collider, and every
+           mm added inboard pushes it into that box. The uncovered 4.4 mm sliver
+           sits inside the Base collision box anyway.
            The last few mm of each x end stay uncovered, which is where the HAA
            flange and the HFE interface sit - both shielded by the neighbouring
            link.
-           x=0.058 rather than the mesh centre 0.0591 or the HFE axis 0.063: the
-           Base box is not centred (front face +0.2105, rear face -0.2125), so
-           0.058 is the smallest offset that clears the box at BOTH ends (front
-           3.5 mm, hind 1.5 mm) while still stopping short of the Head pod
-           collider at x=0.312 (4.0 mm). The Base overlap it removes is filtered
-           anyway (parent-child); this only keeps the wrappers visually honest. -->
-      <collision>
-        <origin xyz="${0.058*sx} ${0.0393*sy} -0.0045" rpy="${PI/2} 0 0" />
+           x=0.060 puts the cylinder at Base x=+/-0.261, exactly where URDF-6 had
+           it (0.203 + 0.058): the HAA moved 2 mm inboard in x and the offset
+           follows, so the clearances to the Base box (front 3.5 mm, hind 1.5 mm;
+           the box is not centred, faces +0.2105/-0.2125) and to the LiDAR
+           collider ahead of it are unchanged. The Base overlap it removes is
+           filtered anyway (parent-child); this only keeps the wrappers visually
+           honest. -->
+      <collision>
+        <origin xyz="${0.060*sx} ${0.0393*sy} -0.0045" rpy="${PI/2} 0 0" />
         <geometry>
           <cylinder radius="0.047" length="0.145" />
@@ -69,39 +84,36 @@
     </link>
     <joint name="${side}${FH}_HAA" type="revolute">
-      <origin xyz="${0.203*sx} ${0.054*sy} 0" rpy="0 0 0" />
+      <origin xyz="${0.201*sx} ${0.056*sy} 0" rpy="0 0 0" />
       <parent link="Base" />
       <child link="${side}${FH}_Hip" />
       <axis xyz="1 0 0" />
-      <!-- Export HAA limits carry over verbatim (axis unchanged). The outward
-           travel differs front vs hind: 0.43633 front, 0.8203 hind. -->
+      <!-- Export HAA limits carry over verbatim (axis unchanged). URDF-7 made
+           the front hips symmetric (+/-0.5236; URDF-6 allowed only 0.43633
+           outward); the hind outward travel stays 0.8203. -->
       <xacro:if value="${side == 'L'}">
-        <limit lower="-0.5236" upper="${0.43633 if FH == 'F' else 0.8203}"
+        <limit lower="-0.5236" upper="${0.5236 if FH == 'F' else 0.8203}"
                effort="${effort_lim}" velocity="${velocity_lim}" />
       </xacro:if>
       <xacro:unless value="${side == 'L'}">
-        <limit lower="${-0.43633 if FH == 'F' else -0.8203}" upper="0.5236"
+        <limit lower="${-0.5236 if FH == 'F' else -0.8203}" upper="0.5236"
                effort="${effort_lim}" velocity="${velocity_lim}" />
       </xacro:unless>
     </joint>
     <!-- ============================= Thigh ============================= -->
-    <!-- Front and hind share one mesh per side (LF_Thigh and LH_Thigh are
-         geometrically identical in the export, likewise RF/RH), so only L_/R_
-         are shipped.
+    <!-- Front and hind share one mesh per side (LF_Thigh and LH_Thigh agree to
+         0.07 mm in the export, RF/RH exactly), so only L_/R_ are shipped. Left
+         and right are NOT mirror images (5 mm apart), hence two files.
+         URDF-7 redesigned this part (the collision with the chassis at extreme
+         HFE is gone; the barrel's rear face pulled in 1.7 mm) and its inertia is
+         now an exact left/right mirror, so one signed block replaces URDF-6's
+         separate L/R values.
          The HFE motor barrel lives on the hip link (one cylinder for the whole
          HAA-to-HFE assembly), so the thigh carries only the slim leg member. -->
     <link name="${side}${FH}_Thigh">
       <inertial>
-        <xacro:if value="${side == 'L'}">
-          <origin xyz="-0.028374 -0.02602 -0.029622" rpy="0 0 0" />
-          <mass value="1.5051" />
-          <inertia ixx="0.0043448" ixy="0.00034914" ixz="-0.0029698"
-                   iyy="0.0075708" iyz="0.00034106" izz="0.0039222" />
-        </xacro:if>
-        <xacro:unless value="${side == 'L'}">
-          <origin xyz="-0.02838 0.025988 -0.029631" rpy="0 0 0" />
-          <mass value="1.5052" />
-          <inertia ixx="0.0043476" ixy="-0.00034935" ixz="-0.0029719"
-                   iyy="0.0075751" iyz="-0.00034134" izz="0.0039239" />
-        </xacro:unless>
+        <origin xyz="-0.024065 ${0.049498*sy} -0.02468" rpy="0 0 0" />
+        <mass value="1.6083" />
+        <inertia ixx="0.004797"  ixy="${0.00038562*sy}" ixz="-0.0032535"
+                 iyy="0.0083583" iyz="${0.00037881*sy}" izz="0.0043329" />
       </inertial>
       <visual>
@@ -116,7 +128,10 @@
       <!-- Slim leg member: box pitched about y onto the HFE->KFE line
            (atan2(-0.15715, -0.20082) = -2.4776 rad), shortened at the knee end
-           where the shank's coaxial knee cylinder takes over. -->
-      <collision>
-        <origin xyz="-0.1121 ${-0.0035*sy} -0.1091" rpy="0 -2.4776 0" />
+           where the shank's coaxial knee cylinder takes over. y is the strut's
+           centre plane, measured on the mesh (mid-strut y 0.0661..0.0801, 14 mm
+           wide) = the KFE origin's 0.057518 plus the shank frame's 0.015582
+           foot offset. -->
+      <collision>
+        <origin xyz="-0.1121 ${0.0731*sy} -0.1091" rpy="0 -2.4776 0" />
         <geometry>
           <box size="0.052 0.016 0.170" />
@@ -125,5 +140,5 @@
     </link>
     <joint name="${side}${FH}_HFE" type="revolute">
-      <origin xyz="${0.063*sx} ${0.0996*sy} 0" rpy="0 0 0" />
+      <origin xyz="${0.065*sx} ${0.0215*sy} 0" rpy="0 0 0" />
       <parent link="${side}${FH}_Hip" />
       <child link="${side}${FH}_Thigh" />
@@ -140,17 +155,20 @@
     </joint>
     <!-- ============================= Shank ============================= -->
-    <!-- All four shank meshes are geometrically identical in the export, so one
-         Shank.STL serves every leg. The part is unchanged from the previous
-         revision; only its frame slid 15.6 mm along y (the foot now sits at y=0
-         in this frame). -->
+    <!-- The same physical part on all four legs: LF and LH agree to 0.07 mm,
+         and RF/RH are LF translated by -0.031164 in y (0.02 mm) - a plain copy,
+         not a mirror image (the strut is not symmetric about its own plane). So
+         one Shank.STL serves every leg, placed at the export's y = +0.015582
+         (left) / -0.015582 (right); the visual origin below carries the
+         -0.031164 shift on the right side.
+         URDF-7 reworked the part inside the same envelope (0.346 -> 0.285 kg). -->
     <link name="${side}${FH}_Shank">
       <inertial>
-        <origin xyz="0.081442 -1.3138E-05 -0.079562" rpy="0 0 0" />
-        <mass value="0.34563" />
-        <inertia ixx="0.0016882" ixy="-5.8149E-12" ixz="0.0015751"
-                 iyy="0.0032906" iyz="-3.2788E-12" izz="0.0016244" />
-      </inertial>
-      <visual>
-        <origin xyz="0 0 0" rpy="0 0 0" />
+        <origin xyz="0.079065 ${0.015593*sy} -0.077092" rpy="0 0 0" />
+        <mass value="0.28461" />
+        <inertia ixx="0.0013467" ixy="3.9114E-12" ixz="0.0012546"
+                 iyy="0.0026227" iyz="-1.247E-11" izz="0.0012937" />
+      </inertial>
+      <visual>
+        <origin xyz="0 ${0.015582*(sy-1)} 0" rpy="0 0 0" />
         <geometry>
           <mesh filename="package://ayg_description/meshes/Shank.STL" />
@@ -161,9 +179,10 @@
       </visual>
       <!-- Slim leg member: box pitched onto the KFE->foot line
-           (atan2(0.170476, -0.189639) = +2.4094 rad). Widened to 0.040 in the
-           box's x from the 0.020 used for the previous revision: the strut is
-           curved, and 0.020 left the outer ~25 mm of its sweep uncovered. -->
-      <collision>
-        <origin xyz="0.0897 0 -0.0938" rpy="0 2.4094 0" />
+           (atan2(0.17048, -0.19164) = +2.4146 rad; URDF-6: 2.4094), 0.040 wide
+           in the box's x because the strut is curved and 0.020 left the outer
+           ~25 mm of its sweep uncovered. Centred on the foot plane y=0.015582
+           (strut mesh y 0.0001..0.0311). -->
+      <collision>
+        <origin xyz="0.0897 ${0.015582*sy} -0.0938" rpy="0 2.4146 0" />
         <geometry>
           <box size="0.040 0.017 0.180" />
@@ -172,8 +191,8 @@
       <!-- Knee filler: cylinder coaxial with the KFE axis, so it is invariant
            under knee bend and bridges the thigh/shank gap for external contacts
-           without ever self-colliding with either. Length follows the new knee
-           width (0.018 measured) rather than the old 0.031. -->
-      <collision>
-        <origin xyz="0 0 0" rpy="${PI/2} 0 0" />
+           without ever self-colliding with either. Centred on the knee's own
+           y (mesh 0.0071..0.0241 at the joint, 17 mm wide). -->
+      <collision>
+        <origin xyz="0 ${0.015582*sy} 0" rpy="${PI/2} 0 0" />
         <geometry>
           <cylinder radius="0.030" length="0.019" />
@@ -182,5 +201,5 @@
     </link>
     <joint name="${side}${FH}_KFE" type="revolute">
-      <origin xyz="-0.15715 ${-0.0035*sy} -0.20082" rpy="0 0 0" />
+      <origin xyz="-0.15715 ${0.057518*sy} -0.20082" rpy="0 0 0" />
       <parent link="${side}${FH}_Thigh" />
       <child link="${side}${FH}_Shank" />
@@ -192,12 +211,14 @@
     <!-- Modelled as primitives rather than the export's Foot mesh: the export's
          own inertia is exactly that of a solid cylinder r=0.032, L=0.031 about y
-         (iyy = m r^2 / 2 = 2.048E-05, ixx = izz = m r^2 / 4 + m L^2 / 12 =
-         1.3443E-05), so the primitive is the mass model, not an approximation. -->
+         (iyy = m r^2 / 2 = 2.7889E-05, ixx = izz = m r^2 / 4 + m L^2 / 12 =
+         1.8306E-05), so the primitive is the mass model, not an approximation.
+         URDF-7 keeps that cylinder and raises its mass 0.040 -> 0.05447 kg (the
+         elastic-tire foot); the compliance itself is not modelled here. -->
     <link name="${side}${FH}_Foot">
       <inertial>
         <origin xyz="0 0 0" rpy="0 0 0" />
-        <mass value="0.04" />
-        <inertia ixx="1.3443E-05" ixy="0" ixz="0"
-                 iyy="2.048E-05"  iyz="0" izz="1.3443E-05" />
+        <mass value="0.05447" />
+        <inertia ixx="1.8306E-05" ixy="0" ixz="0"
+                 iyy="2.7889E-05" iyz="0" izz="1.8306E-05" />
       </inertial>
       <visual>
@@ -218,5 +239,5 @@
     </link>
     <joint name="${side}${FH}_Shank_2_Foot" type="fixed">
-      <origin xyz="0.170476 0 -0.189639" rpy="0 0 0" />
+      <origin xyz="0.17048 ${0.015582*sy} -0.19164" rpy="0 0 0" />
       <parent link="${side}${FH}_Shank" />
       <child link="${side}${FH}_Foot" />

File: urdf/lidar.xacro (robot description, xacro)
@@ -7,6 +7,8 @@
     stamps clouds in `lidar_link`.
     The `Head` link is the mount, taken verbatim from the SolidWorks export
-    CF-AYG-1.3-00-000-URDF-6. Its 0.72713 kg ALREADY INCLUDES the LiDAR body
-    (confirmed with the mechanical engineer) - do not add sensor mass on top.
+    CF-AYG-1.3-00-000-URDF-7. Its 0.81801 kg ALREADY INCLUDES the LiDAR body
+    (confirmed with the mechanical engineer for URDF-6's 0.72713 kg; URDF-7 adds
+    91 g and moves the CoM 15 mm back and 13 mm up) - do not add sensor mass on
+    top. The mount geometry (axis, face distance, Base_2_Head) is unchanged.
     The link is named `Head` (the export's name), not `Camera` as the D555 era
     used. Anything that referenced the old body name must follow - notably
@@ -87,8 +89,8 @@
   <link name="Head">
     <inertial>
-      <origin xyz="0.14526 0.0015227 -0.038347" rpy="0 0 0"/>
-      <mass value="0.72713"/>
-      <inertia ixx="0.00048304" ixy="5.642E-09" ixz="2.7327E-05"
-               iyy="0.0012008"  iyz="4.3319E-09" izz="0.001352"/>
+      <origin xyz="0.13017 -9.7488E-06 -0.025308" rpy="0 0 0"/>
+      <mass value="0.81801"/>
+      <inertia ixx="0.00052732" ixy="-3.3579E-08" ixz="-3.8961E-05"
+               iyy="0.0012906"  iyz="-4.1369E-08" izz="0.0015175"/>
     </inertial>
     <visual>
@@ -104,18 +106,19 @@
       Collision as two primitives, each shaped like the thing it stands for: a
       box for the carry handle on top, a cylinder for the LiDAR below it. The
-      head mesh fills only 10.4% of its 0.226 x 0.134 x 0.116 bounding box (it
-      is an open bracket cage), so a single wrapping box would claim a great
-      deal of empty space on a part that protrudes 0.21 m ahead of the chassis.
-      Since this is the body that strikes obstacles, and near-field obstacle
-      response is the open problem, shape faithfulness is worth the extra
-      primitive.
-      Measured sub-regions, in the Head frame:
+      head mesh fills only ~10% of its 0.226 x 0.144 x 0.116 bounding box (it
+      is an open bracket cage; 10.4% measured on URDF-6), so a single wrapping
+      box would claim a great deal of empty space on a part that protrudes
+      0.21 m ahead of the chassis. Since this is the body that strikes
+      obstacles, and near-field obstacle response is the open problem, shape
+      faithfulness is worth the extra primitive.
+      Measured sub-regions, in the Head frame (URDF-7; only the cage width
+      changed from URDF-6, +/-0.067 -> +/-0.072):
         handle x 0.000..0.226  y +/-0.045  z  0.000..0.008
-        cage   x 0.113..0.152  y +/-0.067  z -0.092..-0.006
+        cage   x 0.113..0.152  y +/-0.072  z -0.092..-0.006
         shroud x 0.165..0.230  y +/-0.032  z -0.093..-0.029  (coaxial with the
                spin axis; its 64.4 mm width is the CAD aperture, 64.3 mm)
       The thin strut below the handle (x 0.008..0.113, y +/-0.010) is left out:
       it is tucked under the handle box and is not a plausible contact point.
-      The cage's side walls (|y| 0.033..0.067) are left out too: they are thin
+      The cage's side walls (|y| 0.033..0.072) are left out too: they are thin
       sheet either side of the sensor, and wrapping them cost a 611 cm3 box.
       The top box is the CARRY HANDLE above the LiDAR, sized to the part rather
