Commit message: Regenerate urdf/ayg.urdf with D555 camera link tree
Follow-up housekeeping to PR #6 (Add D555 RealSense camera link tree).
That PR intentionally left urdf/ayg.urdf dormant because ROS launches invoke
xacro at runtime. Isaac Lab consumes the static .urdf directly, however
(UrdfFileCfg in cf_lab tasks), so the unregenerated dormant file caused
spawn failures of the depth sensor's parent prim Camera_depth_optical_frame.

This commit refreshes the auto-generated artifact so it matches the xacro
source: 974 lines, 59 Camera_* link references, full RealSense optical
frame chain. Source xacro and Gazebo plugin block are unchanged.

No code or behavior change for ROS launches (they still call xacro). Isaac
Lab now loads the up-to-date URDF without needing per-machine working-tree
regeneration.

Co-Authored-By: Claude Opus 4.7 (1M context) <noreply@anthropic.com>

File: urdf/ayg.urdf (robot description, URDF)
Before this commit: robot ayg, 20 links, 19 joints
Links:
- added link Camera, mass 0.3912; collision mesh filename=package://ayg_description/meshes/Camera.STL; visual mesh filename=package://ayg_description/meshes/Camera.STL
- added link Camera_accel_frame
- added link Camera_accel_optical_frame
- added link Camera_body
- added link Camera_color_frame
- added link Camera_color_optical_frame
- added link Camera_depth_frame
- added link Camera_depth_optical_frame
- added link Camera_gyro_frame
- added link Camera_gyro_optical_frame
- added link Camera_imu_optical_frame
- added link Camera_infra1_frame
- added link Camera_infra1_optical_frame
- added link Camera_infra2_frame
- added link Camera_infra2_optical_frame
Joints:
- added joint Base_2_Camera: type fixed, parent Base, child Camera, origin xyz=0.2475 0 0.095 rpy=1.5708 0 0, axis 0 0 0
- added joint Camera_accel_joint: type fixed, parent Camera_body, child Camera_accel_frame, origin xyz=0.0114 -0.0195 0.0 rpy=0 0 0
- added joint Camera_accel_optical_joint: type fixed, parent Camera_accel_frame, child Camera_accel_optical_frame, origin xyz=0 0 0 rpy=-1.5707963267948966 0 -1.5707963267948966
- added joint Camera_body_joint: type fixed, parent Camera, child Camera_body, origin xyz=0 0 0 rpy=-1.5707963267948966 0 0
- added joint Camera_color_joint: type fixed, parent Camera_body, child Camera_color_frame, origin xyz=0 -0.0475 0 rpy=0 0 0
- added joint Camera_color_optical_joint: type fixed, parent Camera_color_frame, child Camera_color_optical_frame, origin xyz=0 0 0 rpy=-1.5707963267948966 0 -1.5707963267948966
- added joint Camera_depth_joint: type fixed, parent Camera_body, child Camera_depth_frame, origin xyz=0 0 0 rpy=0 0 0
- added joint Camera_depth_optical_joint: type fixed, parent Camera_depth_frame, child Camera_depth_optical_frame, origin xyz=0 0 0 rpy=-1.5707963267948966 0 -1.5707963267948966
- added joint Camera_gyro_joint: type fixed, parent Camera_body, child Camera_gyro_frame, origin xyz=0.0114 -0.0195 0.0 rpy=0 0 0
- added joint Camera_gyro_optical_joint: type fixed, parent Camera_gyro_frame, child Camera_gyro_optical_frame, origin xyz=0 0 0 rpy=-1.5707963267948966 0 -1.5707963267948966
- added joint Camera_imu_optical_joint: type fixed, parent Camera_gyro_optical_frame, child Camera_imu_optical_frame, origin xyz=0 0 0 rpy=0 0 0
- added joint Camera_infra1_joint: type fixed, parent Camera_body, child Camera_infra1_frame, origin xyz=0 0.0 0 rpy=0 0 0
- added joint Camera_infra1_optical_joint: type fixed, parent Camera_infra1_frame, child Camera_infra1_optical_frame, origin xyz=0 0 0 rpy=-1.5707963267948966 0 -1.5707963267948966
- added joint Camera_infra2_joint: type fixed, parent Camera_body, child Camera_infra2_frame, origin xyz=0 -0.095 0 rpy=0 0 0
- added joint Camera_infra2_optical_joint: type fixed, parent Camera_infra2_frame, child Camera_infra2_optical_frame, origin xyz=0 0 0 rpy=-1.5707963267948966 0 -1.5707963267948966
- joint Base_2_Battery_Front: origin xyz=0.10070 0 -0.00900 rpy=0 0 0 -> xyz=0.1007 0 -0.009 rpy=0 0 0
- joint Base_2_Battery_Rear: origin xyz=-0.10070 0 -0.00900 rpy=0 0 0 -> xyz=-0.1007 0 -0.009 rpy=0 0 0

Commit message: camera: explicit massless inertials on D555 reference frames
Isaac Sim's URDF importer silently assigns mass=1.0 kg to any link
without an <inertial> tag. Across the 14 D555 reference frames
(Camera_body, *_frame, *_optical_frame, imu) this injected +14 kg
of phantom mass rigid-fixed to Base, breaking the AYG locomotion
teacher in Isaac Lab (98% base-contact faceplant after a few
seconds of episode).

Fix:
- Add <xacro:massless_frame> macro in camera.xacro emitting an
  explicit epsilon inertial (mass=1e-6, inertia=1e-9 diagonal).
- Use the macro for every reference-frame link in the D555 tree.
- Patch the static urdf/ayg.urdf artifact the same way (Isaac Lab
  consumes that file directly via cf_lab AYG_CFG.asset_path).
- Physical Camera link (mass 0.3912 kg, visual, collision) is
  untouched.

Real hardware and robot_state_publisher are unaffected — they only
consume TF, never inertia.

Verified by rolling out the Phase 1 teacher checkpoint
(Teacher_baseline/model_9999.pt) in Isaac Lab on Isaac-Velocity-
Rough-Ayg-v0 with 50 envs x 2000 steps:
  before: 98% base_contact, mean ep-len 3.33s, robot mass 37.5 kg
  after:  14% base_contact, mean ep-len 18.80s, robot mass 23.56 kg
matching the pre-camera-tree URDF baseline (5-7%).

Co-Authored-By: Claude Opus 4.7 (1M context) <noreply@anthropic.com>

File: urdf/ayg.urdf (robot description, URDF)
Before this commit: robot ayg, 35 links, 34 joints
Links:
- link Camera_accel_frame: mass None -> 1e-6
- link Camera_accel_optical_frame: mass None -> 1e-6
- link Camera_body: mass None -> 1e-6
- link Camera_color_frame: mass None -> 1e-6
- link Camera_color_optical_frame: mass None -> 1e-6
- link Camera_depth_frame: mass None -> 1e-6
- link Camera_depth_optical_frame: mass None -> 1e-6
- link Camera_gyro_frame: mass None -> 1e-6
- link Camera_gyro_optical_frame: mass None -> 1e-6
- link Camera_imu_optical_frame: mass None -> 1e-6
- link Camera_infra1_frame: mass None -> 1e-6
- link Camera_infra1_optical_frame: mass None -> 1e-6
- link Camera_infra2_frame: mass None -> 1e-6
- link Camera_infra2_optical_frame: mass None -> 1e-6

File: urdf/camera.xacro (robot description, xacro)
@@ -16,4 +16,22 @@
   <xacro:property name="d555_imu_py" value="-0.0195"/>
   <xacro:property name="d555_imu_pz" value="0.0"/>
+  <!--
+    Massless reference frame for TF purposes only (depth/color/infra/IMU
+    optical frames). An explicit epsilon-mass inertial is required because
+    physics simulators (Isaac Sim, Gazebo) silently assign a 1.0 kg default
+    to any link without <inertial>. Across 14 D555 reference frames that
+    silently injected +14 kg of phantom mass rigid-fixed to Base — enough
+    to faceplant the AYG locomotion policy in Isaac Lab. Real hardware /
+    robot_state_publisher are unaffected (TF-only consumers ignore inertia).
+  -->
+  <xacro:macro name="massless_frame" params="name">
+    <link name="${name}">
+      <inertial>
+        <origin xyz="0 0 0" rpy="0 0 0"/>
+        <mass value="1e-6"/>
+        <inertia ixx="1e-9" ixy="0" ixz="0" iyy="1e-9" iyz="0" izz="1e-9"/>
+      </inertial>
+    </link>
+  </xacro:macro>
   <!-- Physical Camera body (mesh + inertials from SolidWorks export). -->
   <link name="Camera">
@@ -52,5 +70,5 @@
     as in realsense2_description.
   -->
-  <link name="Camera_body"/>
+  <xacro:massless_frame name="Camera_body"/>
   <joint name="Camera_body_joint" type="fixed">
     <origin xyz="0 0 0" rpy="${-M_PI/2} 0 0"/>
@@ -59,5 +77,5 @@
   </joint>
   <!-- Depth (left IR is depth origin in D450 module). -->
-  <link name="Camera_depth_frame"/>
+  <xacro:massless_frame name="Camera_depth_frame"/>
   <joint name="Camera_depth_joint" type="fixed">
     <origin xyz="0 0 0" rpy="0 0 0"/>
@@ -65,5 +83,5 @@
     <child link="Camera_depth_frame"/>
   </joint>
-  <link name="Camera_depth_optical_frame"/>
+  <xacro:massless_frame name="Camera_depth_optical_frame"/>
   <joint name="Camera_depth_optical_joint" type="fixed">
     <origin xyz="0 0 0" rpy="${-M_PI/2} 0 ${-M_PI/2}"/>
@@ -72,5 +90,5 @@
   </joint>
   <!-- Left IR imager (coincident with depth origin). -->
-  <link name="Camera_infra1_frame"/>
+  <xacro:massless_frame name="Camera_infra1_frame"/>
   <joint name="Camera_infra1_joint" type="fixed">
     <origin xyz="0 ${d555_depth_to_infra1_offset} 0" rpy="0 0 0"/>
@@ -78,5 +96,5 @@
     <child link="Camera_infra1_frame"/>
   </joint>
-  <link name="Camera_infra1_optical_frame"/>
+  <xacro:massless_frame name="Camera_infra1_optical_frame"/>
   <joint name="Camera_infra1_optical_joint" type="fixed">
     <origin xyz="0 0 0" rpy="${-M_PI/2} 0 ${-M_PI/2}"/>
@@ -85,5 +103,5 @@
   </joint>
   <!-- Right IR imager (95 mm baseline; sign per D555 datasheet + D585 xacro). -->
-  <link name="Camera_infra2_frame"/>
+  <xacro:massless_frame name="Camera_infra2_frame"/>
   <joint name="Camera_infra2_joint" type="fixed">
     <origin xyz="0 ${d555_depth_to_infra2_offset} 0" rpy="0 0 0"/>
@@ -91,5 +109,5 @@
     <child link="Camera_infra2_frame"/>
   </joint>
-  <link name="Camera_infra2_optical_frame"/>
+  <xacro:massless_frame name="Camera_infra2_optical_frame"/>
   <joint name="Camera_infra2_optical_joint" type="fixed">
     <origin xyz="0 0 0" rpy="${-M_PI/2} 0 ${-M_PI/2}"/>
@@ -98,5 +116,5 @@
   </joint>
   <!-- RGB sensor. -->
-  <link name="Camera_color_frame"/>
+  <xacro:massless_frame name="Camera_color_frame"/>
   <joint name="Camera_color_joint" type="fixed">
     <origin xyz="0 ${d555_depth_to_color_offset} 0" rpy="0 0 0"/>
@@ -104,5 +122,5 @@
     <child link="Camera_color_frame"/>
   </joint>
-  <link name="Camera_color_optical_frame"/>
+  <xacro:massless_frame name="Camera_color_optical_frame"/>
   <joint name="Camera_color_optical_joint" type="fixed">
     <origin xyz="0 0 0" rpy="${-M_PI/2} 0 ${-M_PI/2}"/>
@@ -111,5 +129,5 @@
   </joint>
   <!-- IMU (accel + gyro share the same physical position on D450 module). -->
-  <link name="Camera_accel_frame"/>
+  <xacro:massless_frame name="Camera_accel_frame"/>
   <joint name="Camera_accel_joint" type="fixed">
     <origin xyz="${d555_imu_px} ${d555_imu_py} ${d555_imu_pz}" rpy="0 0 0"/>
@@ -117,5 +135,5 @@
     <child link="Camera_accel_frame"/>
   </joint>
-  <link name="Camera_accel_optical_frame"/>
+  <xacro:massless_frame name="Camera_accel_optical_frame"/>
   <joint name="Camera_accel_optical_joint" type="fixed">
     <origin xyz="0 0 0" rpy="${-M_PI/2} 0 ${-M_PI/2}"/>
@@ -123,5 +141,5 @@
     <child link="Camera_accel_optical_frame"/>
   </joint>
-  <link name="Camera_gyro_frame"/>
+  <xacro:massless_frame name="Camera_gyro_frame"/>
   <joint name="Camera_gyro_joint" type="fixed">
     <origin xyz="${d555_imu_px} ${d555_imu_py} ${d555_imu_pz}" rpy="0 0 0"/>
@@ -129,5 +147,5 @@
     <child link="Camera_gyro_frame"/>
   </joint>
-  <link name="Camera_gyro_optical_frame"/>
+  <xacro:massless_frame name="Camera_gyro_optical_frame"/>
   <joint name="Camera_gyro_optical_joint" type="fixed">
     <origin xyz="0 0 0" rpy="${-M_PI/2} 0 ${-M_PI/2}"/>
@@ -135,5 +153,5 @@
     <child link="Camera_gyro_optical_frame"/>
   </joint>
-  <link name="Camera_imu_optical_frame"/>
+  <xacro:massless_frame name="Camera_imu_optical_frame"/>
   <joint name="Camera_imu_optical_joint" type="fixed">
     <origin xyz="0 0 0" rpy="0 0 0"/>

Commit message: camera: place D555 optical center inside housing, raise Camera link 1 cm
Two changes to the camera transform chain:

- Base_2_Camera xyz z: 0.095 -> 0.105 (raise mount 1 cm to mirror the
  planned hardware bracket revision).
- Camera_body_joint xyz: 0 0 0 -> 0.0527 -0.024 0 (place the D450
  optical-module reference at +5.27 cm fwd and -2.4 cm vertical from
  the Camera link origin in robot body convention, so depth, IR1/IR2,
  color and IMU all sit inside the physical housing instead of at the
  mounting point).

After these changes, the depth optical center in Base is (0.3002, 0,
0.081). The D555 stereo baseline (95 mm) and depth-to-color offset
(47.5 mm) continue to match the datasheet because all downstream sensor
frames inherit from the shifted Camera_body. realsense2_camera per-unit
calibrated TFs continue to supersede these nominal values on the real
robot.

Closes the longstanding 0-vs-real-mount divergence in the camera link
tree: Gazebo, robot_state_publisher and Isaac Lab now all see the same
geometry.

Co-Authored-By: Claude Opus 4.7 (1M context) <noreply@anthropic.com>

File: urdf/ayg.urdf (robot description, URDF)
Before this commit: robot ayg, 35 links, 34 joints
Joints:
- joint Base_2_Camera: origin xyz=0.2475 0 0.095 rpy=1.5708 0 0 -> xyz=0.2475 0 0.105 rpy=1.5708 0 0
- joint Camera_body_joint: origin xyz=0 0 0 rpy=-1.5707963267948966 0 0 -> xyz=0.0527 -0.024 0 rpy=-1.5707963267948966 0 0

File: urdf/camera.xacro (robot description, xacro)
@@ -59,5 +59,5 @@
   </link>
   <joint name="Base_2_Camera" type="fixed">
-    <origin xyz="0.2475 0 0.095" rpy="1.5708 0 0"/>
+    <origin xyz="0.2475 0 0.105" rpy="1.5708 0 0"/>
     <parent link="Base"/>
     <child link="Camera"/>
@@ -69,8 +69,17 @@
     RealSense optical-frame convention (rpy="-pi/2 0 -pi/2" => Z-fwd) works
     as in realsense2_description.
+    The xyz=(0.0527 -0.024 0) translation here places Camera_body at the
+    D450 optical-module reference point inside the housing: +5.27 cm forward
+    and -2.4 cm vertical (down) from the Camera link origin in robot body
+    convention. Camera link's local Y axis is Base +Z (up) due to the 90 deg
+    roll above, so -0.024 along local Y = 2.4 cm down in body frame; local Z
+    is Base -Y, so 0 leaves the optical module on the body centerline. Depth,
+    color, IR1/IR2 baselines and IMU offsets all inherit from this corrected
+    Camera_body position so the whole D555 sensor stack sits where it
+    physically does on the robot.
   -->
   <xacro:massless_frame name="Camera_body"/>
   <joint name="Camera_body_joint" type="fixed">
-    <origin xyz="0 0 0" rpy="${-M_PI/2} 0 0"/>
+    <origin xyz="0.0527 -0.024 0" rpy="${-M_PI/2} 0 0"/>
     <parent link="Camera"/>
     <child link="Camera_body"/>
