Commit message: Update URDF to Ayg 1.3 (#9)
Fold the new 1.3 leg design into the description, preserving the hand-normalized
joint convention (hind pi-yaw; HAA limits direct, HFE+KFE flipped) that the
deployment and training stack depend on.

- legs.xacro: 1.3 geometry, inertials and mechanical limits mapped into the
  deployed convention; front/hind reuse the L_/R_ segment meshes; collision
  primitives approximate the members; foot uses the export mesh (visual) + a
  sphere (collision).
- meshes: dedup front/hind to L_/R_, drop the invisible IMU mesh + old
  Camera/Neck, add Head + Foot. Base kept full-res (visual-only).
- ayg.xacro: base uses the export lumped mass/inertia (batteries dissolved,
  no separate Battery links), resized collision box; IMU visual dropped, mass
  set to export. Total robot mass ~23 kg.
- camera.xacro: keep the "Camera" link + D555 optical-frame tree + Gazebo
  sensors; visual -> Head.STL (roll-compensated); mount at the 1.3 head position
  (0.257 0 0.095) with the 15 deg pitch-down bracket baked into Base_2_Camera
  (single source of truth for the tilt -> Gazebo, Isaac, RViz and real HW agree).
- regenerate flattened ayg.urdf; update the MuJoCo twin to match.

Verified: FK cross-check vs raw export = 0.004 mm; mass 23.07 kg; camera boresight
15.0 deg pitch-down (no image roll); Isaac joint order unchanged; stands in sim.

Co-Authored-By: Claude Opus 4.8 (1M context) <noreply@anthropic.com>

File: urdf/ayg.urdf (robot description, URDF)
Before this commit: robot ayg, 25 links, 24 joints
Links:
- removed link Battery_Front
- removed link Battery_Rear
- link Base: mass 9.148 -> 11.049; geometry collision box size=0.42 0.23 0.14; visual mesh filename=package://ayg_description/meshes/Base.STL
- link Camera: mass 0.3912 -> 0.38664; geometry collision box size=0.0942 0.053 0.1669; visual mesh filename=package://ayg_description/meshes/Head.STL
- link IMU: mass 0.0181381899874512 -> 0.0013495; geometry 
- link LF_Foot: mass 0.0701295110066971 -> 0.04; geometry collision sphere radius=0.032; visual mesh filename=package://ayg_description/meshes/Foot.STL
- link LF_Hip: mass 1.0709 -> 1.017; geometry collision box size=0.11 0.07 0.11; visual mesh filename=package://ayg_description/meshes/L_Hip.STL
- link LF_Shank: mass 0.19753 -> 0.34563; geometry collision box size=0.05 0.05 0.24; visual mesh filename=package://ayg_description/meshes/L_Shank.STL
- link LF_Thigh: mass 1.361 -> 1.505; geometry collision box size=0.06 0.06 0.24; visual mesh filename=package://ayg_description/meshes/L_Thigh.STL
- link LH_Foot: mass 0.0701295110066971 -> 0.04; geometry collision sphere radius=0.032; visual mesh filename=package://ayg_description/meshes/Foot.STL
- link LH_Hip: mass 1.0709 -> 1.017; geometry collision box size=0.11 0.07 0.11; visual mesh filename=package://ayg_description/meshes/R_Hip.STL
- link LH_Shank: mass 0.19753 -> 0.34563; geometry collision box size=0.05 0.05 0.24; visual mesh filename=package://ayg_description/meshes/L_Shank.STL
- link LH_Thigh: mass 1.361 -> 1.505; geometry collision box size=0.06 0.06 0.24; visual mesh filename=package://ayg_description/meshes/L_Thigh.STL
- link RF_Foot: mass 0.07013 -> 0.04; geometry collision sphere radius=0.032; visual mesh filename=package://ayg_description/meshes/Foot.STL
- link RF_Hip: mass 1.071 -> 1.017; geometry collision box size=0.11 0.07 0.11; visual mesh filename=package://ayg_description/meshes/R_Hip.STL
- link RF_Shank: mass 0.19753 -> 0.34563; geometry collision box size=0.05 0.05 0.24; visual mesh filename=package://ayg_description/meshes/R_Shank.STL
- link RF_Thigh: mass 1.361 -> 1.5051; geometry collision box size=0.06 0.06 0.24; visual mesh filename=package://ayg_description/meshes/R_Thigh.STL
- link RH_Foot: mass 0.07013 -> 0.04; geometry collision sphere radius=0.032; visual mesh filename=package://ayg_description/meshes/Foot.STL
- link RH_Hip: mass 1.071 -> 1.017; geometry collision box size=0.11 0.07 0.11; visual mesh filename=package://ayg_description/meshes/L_Hip.STL
- link RH_Shank: mass 0.19753 -> 0.34563; geometry collision box size=0.05 0.05 0.24; visual mesh filename=package://ayg_description/meshes/R_Shank.STL
- link RH_Thigh: mass 1.361 -> 1.5051; geometry collision box size=0.06 0.06 0.24; visual mesh filename=package://ayg_description/meshes/R_Thigh.STL
Joints:
- removed joint Base_2_Battery_Front
- removed joint Base_2_Battery_Rear
- joint Base_2_Camera: origin xyz=0.2475 0 0.095 rpy=1.5708 0 0 -> xyz=0.257 0 0.095 rpy=1.5708 0.2618 0
- joint Base_2_IMU: origin xyz=-3.79309829856879E-05 0 -0.0172341687059438 rpy=0 0 0 -> xyz=0 0 -0.00983 rpy=0 0 0
- joint LF_HAA: origin xyz=0.2021 0.054 0 rpy=0 0 0 -> xyz=0.2105 0.054 0 rpy=0 0 0
- joint LF_HFE: limit lower=-1.6668 upper=3.2376 effort=50.0 velocity=10.0 -> lower=-1.2625 upper=3.0761 effort=50.0 velocity=10.0; origin xyz=0.0679 0.01985 0 rpy=0 0 0 -> xyz=0.065 0.0235 0 rpy=0 0 0
- joint LF_KFE: limit lower=-0.74002 upper=1.1868 effort=50.0 velocity=10.0 -> lower=-0.56374 upper=1.4015 effort=50.0 velocity=10.0; origin xyz=-0.14936 0.058 -0.16017 rpy=0 0 0 -> xyz=-0.15715 0.057018 -0.20082 rpy=0 0 0
- joint LF_Shank_2_Foot: origin xyz=0.165 0.0205 -0.151 rpy=0 0 0 -> xyz=0.17048 0.015582 -0.18964 rpy=0 0 0
- joint LH_HAA: limit lower=-0.5236 upper=0.83776 effort=50.0 velocity=10.0 -> lower=-0.5236 upper=0.8203 effort=50.0 velocity=10.0; origin xyz=-0.2021 0.054 0 rpy=0 0 3.1416 -> xyz=-0.2105 0.054 0 rpy=0 0 3.141592653589793
- joint LH_HFE: limit lower=-2.4522 upper=2.4522 effort=50.0 velocity=10.0 -> lower=-2.2907 upper=2.0479 effort=50.0 velocity=10.0; origin xyz=0.0679 -0.01985 0 rpy=0 0 3.1416 -> xyz=0.065 -0.0235 0 rpy=0 0 3.141592653589793
- joint LH_KFE: limit lower=-0.74002 upper=1.1868 effort=50.0 velocity=10.0 -> lower=-0.56374 upper=1.4015 effort=50.0 velocity=10.0; origin xyz=-0.14936 0.058 -0.16017 rpy=0 0 0 -> xyz=-0.15715 0.057018 -0.20082 rpy=0 0 0
- joint LH_Shank_2_Foot: origin xyz=0.165 0.0205 -0.151 rpy=0 0 0 -> xyz=0.17048 0.015582 -0.18964 rpy=0 0 0
- joint RF_HAA: origin xyz=0.2021 -0.054 0 rpy=0 0 0 -> xyz=0.2105 -0.054 0 rpy=0 0 0
- joint RF_HFE: limit lower=-1.6668 upper=3.2376 effort=50.0 velocity=10.0 -> lower=-1.2625 upper=3.0761 effort=50.0 velocity=10.0; origin xyz=0.0679 -0.01985 0 rpy=0 0 0 -> xyz=0.065 -0.0235 0 rpy=0 0 0
- joint RF_KFE: limit lower=-0.74002 upper=1.1868 effort=50.0 velocity=10.0 -> lower=-0.56374 upper=1.4015 effort=50.0 velocity=10.0; origin xyz=-0.14936 -0.058 -0.16017 rpy=0 0 0 -> xyz=-0.15715 -0.057037 -0.20082 rpy=0 0 0
- joint RF_Shank_2_Foot: origin xyz=0.165 -0.0205 -0.151 rpy=0 0 0 -> xyz=0.170476 -0.0155635 -0.189639 rpy=0 0 0
- joint RH_HAA: limit lower=-0.83776 upper=0.5236 effort=50.0 velocity=10.0 -> lower=-0.8203 upper=0.5236 effort=50.0 velocity=10.0; origin xyz=-0.2021 -0.054 0 rpy=0 0 3.1416 -> xyz=-0.2105 -0.054 0 rpy=0 0 3.141592653589793
- joint RH_HFE: limit lower=-2.4522 upper=2.4522 effort=50.0 velocity=10.0 -> lower=-2.2907 upper=2.0479 effort=50.0 velocity=10.0; origin xyz=0.0665 0.01985 0 rpy=0 0 3.1416 -> xyz=0.065 0.0235 0 rpy=0 0 3.141592653589793
- joint RH_KFE: limit lower=-0.74002 upper=1.1868 effort=50.0 velocity=10.0 -> lower=-0.56374 upper=1.4015 effort=50.0 velocity=10.0; origin xyz=-0.14936 -0.058 -0.16017 rpy=0 0 0 -> xyz=-0.15715 -0.057037 -0.20082 rpy=0 0 0
- joint RH_Shank_2_Foot: origin xyz=0.165 -0.0205 -0.151 rpy=0 0 0 -> xyz=0.170476 -0.0155635 -0.189639 rpy=0 0 0

File: urdf/ayg.xacro (robot description, xacro)
@@ -17,26 +17,4 @@
   <xacro:property name="velocity_lim" value="10.0" />
   <xacro:property name="PI" value="3.1415926535897931" />
-  <!-- Battery inertial properties (CAD export → URDF frame)
-       CAD frame: X=forward, Y=up, Z=left  |  URDF frame: X=forward, Y=left, Z=up
-       Mapping: (URDF_x, URDF_y, URDF_z) = (CAD_x, CAD_z, CAD_y)
-       CAD mass: 1.55217 kg  |  Weighed: 1.6 kg each  |  Housing mass is in Base -->
-  <xacro:property name="battery_cad_mass" value="1.55217" />
-  <xacro:property name="battery_real_mass" value="1.6" />
-  <xacro:property name="battery_inertia_scale" value="${battery_real_mass / battery_cad_mass}" />
-  <!-- CoM in battery link frame (URDF, meters) -->
-  <xacro:property name="battery_com_x" value="-0.00002" />
-  <xacro:property name="battery_com_y" value="-0.00421" />
-  <xacro:property name="battery_com_z" value="0.04143" />
-  <!-- Inertia at CoM, at CAD mass, URDF frame (kg·m²) -->
-  <xacro:property name="battery_cad_ixx" value="0.0043243903" />
-  <xacro:property name="battery_cad_ixy" value="-0.0000040621" />
-  <xacro:property name="battery_cad_ixz" value="-0.0000050483" />
-  <xacro:property name="battery_cad_iyy" value="0.0074475647" />
-  <xacro:property name="battery_cad_iyz" value="-0.0002587481" />
-  <xacro:property name="battery_cad_izz" value="0.0043149743" />
-  <!-- Battery positions relative to Base (URDF, meters) -->
-  <xacro:property name="battery_front_x" value="0.10070" />
-  <xacro:property name="battery_rear_x" value="-0.10070" />
-  <xacro:property name="battery_pos_z" value="-0.00900" />
   <xacro:if value="${sim}">
     <xacro:include filename="$(find ayg_description)/urdf/ayg_sim_ros2_control.xacro" />
@@ -59,17 +37,20 @@
     name="Base">
     <inertial>
+      <!-- Ayg 1.3 SolidWorks export. Batteries are rigidly fixed inside the
+           chassis and are lumped into this Base mass/inertia (no separate
+           Battery links), so the trunk is a single rigid body. Total robot
+           mass ~23 kg. -->
       <origin
-        xyz="0.00057686 -0.00018498 0.0026529"
+        xyz="-0.0030682 -4.5608E-05 -0.0023186"
         rpy="0 0 0" />
-      <!-- Measured: 9.148 kg (CAD: 9.1298 kg) -->
       <mass
-        value="9.148" />
+        value="11.049" />
       <inertia
-        ixx="0.022082"
-        ixy="3.2369E-07"
-        ixz="6.8653E-05"
-        iyy="0.031986"
-        iyz="2.8565E-07"
-        izz="0.040389" />
+        ixx="0.032662"
+        ixy="-2.5713E-06"
+        ixz="6.2419E-05"
+        iyy="0.034773"
+        iyz="-2.217E-06"
+        izz="0.054917" />
     </inertial>
     <visual>
@@ -92,38 +73,29 @@
         rpy="0 0 0" />
       <geometry>
-        <box size="0.4 0.23 0.12" />
+        <box size="0.42 0.23 0.14" />
       </geometry>
     </collision>
   </link>
+  <!-- IMU is a massless-ish reference frame only: it is rigidly fixed to Base,
+       its mesh is inside the chassis (not visible) so no <visual>, and the
+       Gazebo/real IMU sensor is defined on the Base link (see
+       ayg_sim_ros2_control.xacro), not on this link. Mass/inertia are the 1.3
+       CAD-export values (bare module, ~1.35 g); negligible vs the 23 kg total. -->
   <link
     name="IMU">
     <inertial>
       <origin
-        xyz="-1.26817788945405E-05 -3.05893593341006E-06 0.00502425421604302"
+        xyz="-0.00099712 0.00015501 -0.00052021"
         rpy="0 0 0" />
       <mass
-        value="0.0181381899874512" />
+        value="0.0013495" />
       <inertia
-        ixx="4.80017459218422E-06"
-        ixy="-6.17315963282016E-11"
-        ixz="-1.66852937330168E-09"
-        iyy="3.40477341509462E-06"
-        iyz="-3.279931989329E-11"
-        izz="7.92679226862755E-06" />
+        ixx="4.0133E-08"
+        ixy="-6.9859E-14"
+        ixz="8.9554E-12"
+        iyy="5.9906E-08"
+        iyz="-1.4567E-14"
+        izz="9.917E-08" />
     </inertial>
-    <visual>
-      <origin
-        xyz="0 0 0"
-        rpy="0 0 0" />
-      <geometry>
-        <mesh
-          filename="package://ayg_description/meshes/IMU.STL" />
-      </geometry>
-      <material
-        name="">
-        <color
-          rgba="0.792156862745098 0.819607843137255 0.933333333333333 1" />
-      </material>
-    </visual>
   </link>
   <joint
@@ -131,5 +103,5 @@
     type="fixed">
     <origin
-      xyz="-3.79309829856879E-05 0 -0.0172341687059438"
+      xyz="0 0 -0.00983"
       rpy="0 0 0" />
     <parent
@@ -140,43 +112,4 @@
       xyz="0 0 0" />
   </joint>
-  <!-- Battery macro (2x identical packs, front and rear) -->
-  <xacro:macro name="battery" params="name pos_x">
-    <link name="Battery_${name}">
-      <inertial>
-        <origin xyz="${battery_com_x} ${battery_com_y} ${battery_com_z}" rpy="0 0 0" />
-        <mass value="${battery_real_mass}" />
-        <inertia
-          ixx="${battery_cad_ixx * battery_inertia_scale}"
-          ixy="${battery_cad_ixy * battery_inertia_scale}"
-          ixz="${battery_cad_ixz * battery_inertia_scale}"
-          iyy="${battery_cad_iyy * battery_inertia_scale}"
-          iyz="${battery_cad_iyz * battery_inertia_scale}"
-          izz="${battery_cad_izz * battery_inertia_scale}" />
-      </inertial>
-      <visual>
-        <origin xyz="0 0 0" rpy="0 0 0" />
-        <geometry>
-          <box size="0.079 0.177 0.096" />
-        </geometry>
-        <material name="battery_color">
-          <color rgba="0.2 0.2 0.3 1" />
-        </material>
-      </visual>
-      <collision>
-        <origin xyz="0 0 0" rpy="0 0 0" />
-        <geometry>
-          <box size="0.079 0.177 0.096" />
-        </geometry>
-      </collision>
-    </link>
-    <joint name="Base_2_Battery_${name}" type="fixed">
-      <origin xyz="${pos_x} 0 ${battery_pos_z}" rpy="0 0 0" />
-      <parent link="Base" />
-      <child link="Battery_${name}" />
-      <axis xyz="0 0 0" />
-    </joint>
-  </xacro:macro>
-  <xacro:battery name="Front" pos_x="${battery_front_x}" />
-  <xacro:battery name="Rear"  pos_x="${battery_rear_x}" />
   <xacro:include filename="$(find ayg_description)/urdf/legs.xacro" />
   <xacro:if value="${camera}">

File: urdf/camera.xacro (robot description, xacro)
@@ -29,16 +29,24 @@
     </link>
   </xacro:macro>
-  <!-- Physical Camera body (mesh + inertials from SolidWorks export). -->
+  <!--
+    Physical front head body (Ayg 1.3 "Head" mesh + inertials from the SolidWorks
+    export). The link keeps the name "Camera" so the D555 optical-frame tree,
+    Gazebo sensors, realsense2_camera camera_name and all /camera/Camera/* topics
+    are unchanged. The Head mesh is exported base-aligned; because Base_2_Camera
+    carries a +90 deg roll (needed by the optical frames below), the visual and
+    inertial are expressed with a compensating -90 deg roll so the head renders
+    upright. Mass/CoM/inertia are the export Head values rolled into this frame.
+  -->
   <link name="Camera">
     <inertial>
-      <origin xyz="0.027539 -0.0054988 -1.4524E-08" rpy="0 0 0"/>
-      <mass value="0.3912"/>
-      <inertia ixx="0.00080723" ixy="4.4453E-06" ixz="-1.7833E-09"
-               iyy="0.00082275" iyz="2.4795E-09" izz="0.00010329"/>
+      <origin xyz="0.026077 -0.0052539 0" rpy="0 0 0"/>
+      <mass value="0.38664"/>
+      <inertia ixx="0.00083292" ixy="3.6679E-06" ixz="-5.259E-09"
+               iyy="0.00084639" iyz="-2.8688E-09" izz="0.00011429"/>
     </inertial>
     <visual>
-      <origin xyz="0 0 0" rpy="0 0 0"/>
+      <origin xyz="0 0 0" rpy="${-M_PI/2} 0 0"/>
       <geometry>
-        <mesh filename="package://ayg_description/meshes/Camera.STL"/>
+        <mesh filename="package://ayg_description/meshes/Head.STL"/>
       </geometry>
       <material name="">
@@ -47,19 +55,25 @@
     </visual>
     <!--
-      Collision simplified from the full Camera.STL to a primitive box sized
-      to the bare D555 housing (mesh housing extent 0.0571 x 0.0443 x 0.1670 m,
-      centered at 0.0286 -0.0070 0 in the Camera link frame). The thin rear
-      mounting tab (-0.035 m in X) is intentionally excluded. A box is far
-      cheaper for the physics broadphase/narrowphase than a 1978-triangle mesh.
+      Collision simplified to a primitive box wrapping the 1.3 Head mesh
+      (extent 0.0942 x 0.053 x 0.1669 m in this link frame, centered at
+      0.0121 -0.0062 0). A box is far cheaper for the physics broadphase than
+      the full head mesh, and is what cf_lab's camera-contact termination
+      (body_names="Camera") detects.
     -->
     <collision>
-      <origin xyz="0.0286 -0.007 0" rpy="0 0 0"/>
+      <origin xyz="0.0121 -0.0062 0" rpy="0 0 0"/>
       <geometry>
-        <box size="0.0571 0.0443 0.167"/>
+        <box size="0.0942 0.053 0.1669"/>
       </geometry>
     </collision>
   </link>
+  <!-- Ayg 1.3 head mount (export Base_2_Head at 0.257 0 0.095). rpy = +90 deg roll
+       (for the optical-frame subtree below) + 15 deg pitch-down = the physical D555
+       bracket, so the depth/color frames look 15 deg below horizontal. This is the
+       single source of truth for the tilt: Gazebo, Isaac, RViz TF and the real
+       robot all agree (the cf_lab depth-camera prim offset is identity). z=0.095 is
+       the CAD-confirmed camera height. -->
   <joint name="Base_2_Camera" type="fixed">
-    <origin xyz="0.2475 0 0.095" rpy="1.5708 0 0"/>
+    <origin xyz="0.257 0 0.095" rpy="1.5708 0.2618 0"/>
     <parent link="Base"/>
     <child link="Camera"/>
@@ -74,6 +88,6 @@
     The xyz=(0.0527 -0.024 0) translation places the depth origin at the
     optical-module reference inside the housing: +5.27 cm forward and -2.4 cm
-    vertical (down) from the Camera link origin in robot body convention (CAD
-    values for the 30 deg mount tilt). Camera link's local Y axis is Base +Z
+    vertical (down) from the Camera link origin in robot body convention (nominal
+    D555 optical-module offset inside the housing). Camera link's local Y axis is Base +Z
     (up) due to the 90 deg roll above, so -0.024 along local Y = 2.4 cm down
     in body frame; local Z is Base -Y, so 0 leaves the optical module on the
