Commit message: Update URDF to Ayg 1.3 (#9)
Fold the new 1.3 leg design into the description, preserving the hand-normalized
joint convention (hind pi-yaw; HAA limits direct, HFE+KFE flipped) that the
deployment and training stack depend on.

- legs.xacro: 1.3 geometry, inertials and mechanical limits mapped into the
  deployed convention; front/hind reuse the L_/R_ segment meshes; collision
  primitives approximate the members; foot uses the export mesh (visual) + a
  sphere (collision).
- meshes: dedup front/hind to L_/R_, drop the invisible IMU mesh + old
  Camera/Neck, add Head + Foot. Base kept full-res (visual-only).
- ayg.xacro: base uses the export lumped mass/inertia (batteries dissolved,
  no separate Battery links), resized collision box; IMU visual dropped, mass
  set to export. Total robot mass ~23 kg.
- camera.xacro: keep the "Camera" link + D555 optical-frame tree + Gazebo
  sensors; visual -> Head.STL (roll-compensated); mount at the 1.3 head position
  (0.257 0 0.095) with the 15 deg pitch-down bracket baked into Base_2_Camera
  (single source of truth for the tilt -> Gazebo, Isaac, RViz and real HW agree).
- regenerate flattened ayg.urdf; update the MuJoCo twin to match.

Verified: FK cross-check vs raw export = 0.004 mm; mass 23.07 kg; camera boresight
15.0 deg pitch-down (no image roll); Isaac joint order unchanged; stands in sim.

Co-Authored-By: Claude Opus 4.8 (1M context) <noreply@anthropic.com>

File: urdf/legs.xacro (robot description, xacro)
@@ -1,584 +1,315 @@
 <?xml version="1.0"?>
 <robot xmlns:xacro="http://www.ros.org/wiki/xacro">
+  <!--
+    Parameterized legs (Ayg 1.3). Two macros, L_Leg / R_Leg, each instantiated
+    for front (FH="F") and hind (FH="H"). Hind legs carry a pi yaw on the HAA and
+    HFE joint origins so that identical joint values mirror the front leg (the net
+    rotation on the thigh/shank frames is 2*pi = identity; the hip frame keeps one
+    pi flip). Joint axes are normalized (HAA about +x world, HFE/KFE about -y
+    world) to match the deployed convention (robstride_ros2_control / calibration /
+    policy). Front and hind reuse the same L_/R_ segment meshes.
+    Inertials/limits are the SolidWorks 1.3 export values mapped into this
+    convention; collision primitives approximate the members (refined in sim).
+  -->
   <xacro:macro name="L_Leg" params="FH">
-    <link
-      name="L${FH}_Hip">
+    <link name="L${FH}_Hip">
       <inertial>
         <xacro:if value="${FH == 'F'}">
-          <origin
-            xyz="0.063065 -0.0051556 -5.3332E-05"
-            rpy="0 0 0" />
+          <origin xyz="0.062976 -0.0014435 9.395E-06" rpy="0 0 0" />
+          <mass value="1.017" />
+          <inertia ixx="0.00088413" ixy="1.6599E-05" ixz="5.521E-07"
+                   iyy="0.0014074" iyz="-1.7604E-07" izz="0.00099675" />
         </xacro:if>
         <xacro:unless value="${FH == 'F'}">
-          <origin
-            xyz="0.063077 0.0051556 -6.5344E-05"
-            rpy="0 0 0" />
+          <origin xyz="0.062976 0.0014435 -9.395E-06" rpy="0 0 0" />
+          <mass value="1.017" />
+          <inertia ixx="0.00088413" ixy="-1.6599E-05" ixz="-5.521E-07"
+                   iyy="0.0014074" iyz="-1.7604E-07" izz="0.00099675" />
         </xacro:unless>
-        <mass
-          value="1.0709" />
-        <inertia
-          ixx="0.00078713"
-          ixy="-7.2738E-08"
-          ixz="-1.6354E-06"
-          iyy="0.0013471"
-          iyz="-2.2108E-07"
-          izz="0.00073074" />
-      </inertial>
-      <visual>
-        <origin
-          xyz="0 0 0"
-          rpy="0 0 0" />
+      </inertial>
+      <visual>
+        <origin xyz="0 0 0" rpy="0 0 0" />
         <geometry>
           <xacro:if value="${FH == 'F'}">
-            <mesh
-              filename="package://ayg_description/meshes/L_Hip.STL" />
+            <mesh filename="package://ayg_description/meshes/L_Hip.STL" />
           </xacro:if>
           <xacro:unless value="${FH == 'F'}">
-            <mesh
-              filename="package://ayg_description/meshes/R_Hip.STL" />
+            <mesh filename="package://ayg_description/meshes/R_Hip.STL" />
           </xacro:unless>
         </geometry>
-        <material
-          name="">
-          <color
-            rgba="0.69804 0.69804 0.69804 1" />
-        </material>
-      </visual>
-      <xacro:if value="${FH == 'F'}">
-        <collision>
-          <origin
-            xyz="0.0665 0.04 0"
-            rpy="${PI/2} 0 0" />
-          <geometry>
-            <cylinder radius="0.05" length="0.148"/>
-          </geometry>
-        </collision>
-      </xacro:if>
-      <xacro:unless value="${FH == 'F'}">
-        <collision>
-          <origin
-            xyz="0.0665 -0.04 0"
-            rpy="${PI/2} 0 0" />
-          <geometry>
-            <cylinder radius="0.05" length="0.148"/>
-          </geometry>
-        </collision>
-      </xacro:unless>
-    </link>
-    <joint
-      name="L${FH}_HAA"
-      type="revolute">
-      <xacro:if value="${FH == 'F'}">
-        <origin
-          xyz="0.2021 0.054 0"
-          rpy="0 0 0" />
-      </xacro:if>
-      <xacro:unless value="${FH == 'F'}">
-        <origin
-          xyz="-0.2021 0.054 0"
-          rpy="0 0 3.1416" />
-      </xacro:unless>
-      <parent
-        link="Base" />
-      <child
-        link="L${FH}_Hip" />
-      <xacro:if value="${FH == 'F'}">
-        <axis
-        xyz="1 0 0" />
-        <limit
-          lower="-0.5236"
-          upper="0.43633"
-          effort="${effort_lim}"
-          velocity="${velocity_lim}" />
-      </xacro:if>
-      <xacro:unless value="${FH == 'F'}">
-        <axis
-        xyz="-1 0 0" />
-        <limit
-          lower="-0.5236"
-          upper="0.83776"
-          effort="${effort_lim}"
-          velocity="${velocity_lim}" />
-      </xacro:unless>
-    </joint>
-    <link
-      name="L${FH}_Thigh">
-      <inertial>
-        <origin
-          xyz="-0.0095261 0.047418 -0.010869"
-          rpy="0 0 0" />
-        <mass
-          value="1.361" />
-        <inertia
-          ixx="0.0012156"
-          ixy="1.025E-06"
-          ixz="-0.00042254"
-          iyy="0.0022368"
-          iyz="-1.3825E-06"
-          izz="0.0012227" />
-      </inertial>
-      <visual>
-        <origin
-          xyz="0 0 0"
-          rpy="0 0 0" />
-        <geometry>
-          <mesh
-            filename="package://ayg_description/meshes/L_Thigh.STL" />
-        </geometry>
-        <material
-          name="">
-          <color
-            rgba="0.69804 0.69804 0.69804 1" />
-        </material>
-      </visual>
-      <collision>
-        <origin
-          xyz="-0.0975 +0.08 -0.07"
-          rpy="${PI/4} 0 ${PI/2}" />
-        <geometry>
-          <box size="0.025 0.05 0.14"/>
-        </geometry>
-      </collision>
-    </link>
-    <joint
-      name="L${FH}_HFE"
-      type="revolute">
-      <xacro:if value="${FH == 'F'}">
-        <origin
-          xyz="0.0679 0.01985 0"
-          rpy="0 0 0" />
-      </xacro:if>
-      <xacro:unless value="${FH == 'F'}">
-        <origin
-          xyz="0.0679 -0.01985 0"
-          rpy="0 0 3.1416" />
-      </xacro:unless>
-      <parent
-        link="L${FH}_Hip" />
-      <child
-        link="L${FH}_Thigh" />
-      <axis
-        xyz="0 -1 0" />
-      <xacro:if value="${FH == 'F'}">
-        <limit
-          lower="-1.6668"
-          upper="3.2376"
-          effort="${effort_lim}"
-          velocity="${velocity_lim}" />
-      </xacro:if>
-      <xacro:unless value="${FH == 'F'}">
-        <limit
-          lower="-2.4522"
-          upper="2.4522"
-          effort="${effort_lim}"
-          velocity="${velocity_lim}" />
-      </xacro:unless>
-    </joint>
-    <link
-      name="L${FH}_Shank">
-      <inertial>
-        <origin
-          xyz="0.059297 0.0205 -0.044894"
-          rpy="0 0 0" />
-        <mass
-          value="0.19753" />
-        <inertia
-          ixx="0.00059399"
-          ixy="-3.3081E-19"
-          ixz="0.00058611"
-          iyy="0.0012346"
-          iyz="3.1645E-19"
-          izz="0.00065333" />
-      </inertial>
-      <visual>
-        <origin
-          xyz="0 0 0"
-          rpy="0 0 0" />
-        <geometry>
-          <mesh
-            filename="package://ayg_description/meshes/L_Shank.STL" />
-        </geometry>
-        <material
-          name="">
-          <color
-            rgba="0.69804 0.69804 0.69804 1" />
-        </material>
-      </visual>
-      <collision>
-        <origin
-          xyz="0 0.02 0"
-          rpy="${PI/2} 0 0" />
-        <geometry>
-          <cylinder radius="0.025" length="0.03"/>
-        </geometry>
-      </collision>
-      <collision>
-        <origin
-          xyz="0.08 0.02 -0.075"
-          rpy="${PI/2} ${-PI/4} 0" />
-        <geometry>
-          <box size="0.025 0.165 0.0125"/>
-        </geometry>
-      </collision>
-    </link>
-    <joint
-      name="L${FH}_KFE"
-      type="revolute">
-      <origin
-        xyz="-0.14936 0.058 -0.16017"
-        rpy="0 0 0" />
-      <parent
-        link="L${FH}_Thigh" />
-      <child
-        link="L${FH}_Shank" />
-      <axis
-        xyz="0 -1 0" />
-      <limit
-        lower="-0.74002"
-        upper="1.1868"
-        effort="${effort_lim}"
-        velocity="${velocity_lim}" />
-    </joint>
-    <link
-      name="L${FH}_Foot">
-      <inertial>
-        <origin
-          xyz="-2.77555756156289E-17 5.55111512312578E-17 0"
-          rpy="0 0 0" />
-        <mass
-          value="0.0701295110066971" />
-        <inertia
-          ixx="1.91783738418569E-05"
-          ixy="4.42768620674145E-20"
-          ixz="8.0334719824878E-35"
-          iyy="3.14806687325575E-05"
-          iyz="2.23148962310519E-20"
-          izz="1.91783738418569E-05" />
-      </inertial>
-      <visual>
-        <origin
-          xyz="0 0 0"
-          rpy="${PI/2} 0 0" />
-        <geometry>
-          <cylinder length="0.025" radius="0.030"/>
-        </geometry>
-        <material
-          name="">
-          <color
-            rgba="0.29804 0.29804 0.29804 1" />
-        </material>
-      </visual>
-      <collision>
-        <origin
-          xyz="0 0 0"
-          rpy="${PI/2} 0 0" />
-        <geometry>
-          <sphere radius="0.030"/>
-        </geometry>
-      </collision>
-    </link>
-    <joint
-      name="L${FH}_Shank_2_Foot"
-      type="fixed">
-      <origin
-        xyz="0.165 0.0205 -0.151"
-        rpy="0 0 0" />
-      <parent
-        link="L${FH}_Shank" />
-      <child
-        link="L${FH}_Foot" />
-      <axis
-        xyz="0 0 0" />
+        <material name="">
+          <color rgba="0.69804 0.69804 0.69804 1" />
+        </material>
+      </visual>
+      <collision>
+        <origin xyz="0.055 0 0" rpy="0 0 0" />
+        <geometry>
+          <box size="0.11 0.07 0.11" />
+        </geometry>
+      </collision>
+    </link>
+    <joint name="L${FH}_HAA" type="revolute">
+      <xacro:if value="${FH == 'F'}">
+        <origin xyz="0.2105 0.054 0" rpy="0 0 0" />
+      </xacro:if>
+      <xacro:unless value="${FH == 'F'}">
+        <origin xyz="-0.2105 0.054 0" rpy="0 0 ${PI}" />
+      </xacro:unless>
+      <parent link="Base" />
+      <child link="L${FH}_Hip" />
+      <xacro:if value="${FH == 'F'}">
+        <axis xyz="1 0 0" />
+        <limit lower="-0.5236" upper="0.43633" effort="${effort_lim}" velocity="${velocity_lim}" />
+      </xacro:if>
+      <xacro:unless value="${FH == 'F'}">
+        <axis xyz="-1 0 0" />
+        <limit lower="-0.5236" upper="0.8203" effort="${effort_lim}" velocity="${velocity_lim}" />
+      </xacro:unless>
+    </joint>
+    <link name="L${FH}_Thigh">
+      <inertial>
+        <origin xyz="-0.023305 0.049402 -0.024328" rpy="0 0 0" />
+        <mass value="1.505" />
+        <inertia ixx="0.0030493" ixy="-3.2033E-06" ixz="-0.0016346"
+                 iyy="0.0052191" iyz="-1.6215E-06" izz="0.0026578" />
+      </inertial>
+      <visual>
+        <origin xyz="0 0 0" rpy="0 0 0" />
+        <geometry>
+          <mesh filename="package://ayg_description/meshes/L_Thigh.STL" />
+        </geometry>
+        <material name="">
+          <color rgba="0.69804 0.69804 0.69804 1" />
+        </material>
+      </visual>
+      <collision>
+        <origin xyz="-0.0786 0.0285 -0.1004" rpy="0 2.4474 2.7935" />
+        <geometry>
+          <box size="0.06 0.06 0.24" />
+        </geometry>
+      </collision>
+    </link>
+    <joint name="L${FH}_HFE" type="revolute">
+      <xacro:if value="${FH == 'F'}">
+        <origin xyz="0.065 0.0235 0" rpy="0 0 0" />
+        <limit lower="-1.2625" upper="3.0761" effort="${effort_lim}" velocity="${velocity_lim}" />
+      </xacro:if>
+      <xacro:unless value="${FH == 'F'}">
+        <origin xyz="0.065 -0.0235 0" rpy="0 0 ${PI}" />
+        <limit lower="-2.2907" upper="2.0479" effort="${effort_lim}" velocity="${velocity_lim}" />
+      </xacro:unless>
+      <parent link="L${FH}_Hip" />
+      <child link="L${FH}_Thigh" />
+      <axis xyz="0 -1 0" />
+    </joint>
+    <link name="L${FH}_Shank">
+      <inertial>
+        <origin xyz="0.081442 0.015569 -0.079562" rpy="0 0 0" />
+        <mass value="0.34563" />
+        <inertia ixx="0.0016882" ixy="-5.8149E-12" ixz="0.0015751"
+                 iyy="0.0032906" iyz="-3.2788E-12" izz="0.0016244" />
+      </inertial>
+      <visual>
+        <origin xyz="0 0 0" rpy="0 0 0" />
+        <geometry>
+          <mesh filename="package://ayg_description/meshes/L_Shank.STL" />
+        </geometry>
+        <material name="">
+          <color rgba="0.69804 0.69804 0.69804 1" />
+        </material>
+      </visual>
+      <collision>
+        <origin xyz="0.0852 0.0078 -0.0948" rpy="0 2.4073 0.0911" />
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