Commit message: Rebase the 1.3 model onto SolidWorks export CF-AYG-1.3-00-000-URDF-6
The existing 1.3 commits were built from a 2026-07-04 export; this adopts the
2026-07-16 one, which supersedes it on Base, hips, thighs, the HAA offset,
joint limits and the whole head. Segment lengths are unchanged (thigh = shank =
0.255 m exactly, 0.510 m hip-to-foot), so the leg work carries over - this is a
parts revision, not a new kinematic chain.

legs.xacro is rewritten as one macro instantiated four times with sx/sy sign
parameters, so it reads as a direct transcription of the export and can be
re-checked line by line against a future one. The export's own frame placement
is adopted; the hind pi-yaw is dropped, having existed only so front and hind
could share a hip mesh (the export ships four, differently tessellated). That
removal is behaviour-neutral: HFE/KFE axes are parallel to y, so sliding a
frame along its own rotation axis is kinematically null.

camera.xacro (RealSense D555) becomes lidar.xacro. The head is now
unconditional - it is structural chassis, not an optional payload - so
ayg_kindyn/Pinocchio finally sees its 0.727 kg and forward pitch moment; the
previous flat urdf shipped 18 links with no head at all. That 0.727 kg already
includes the JT128 body (confirmed with the mechanical engineer), so no sensor
mass is added on top. Only lidar_link and the Gazebo gpu_lidar are gated.

Collision primitives were refit by measuring the new meshes rather than scaled:
the HFE motor barrel moved from the hip into the thigh (hip y extent 0.148 ->
0.058), and the head is three boxes because its mesh fills only 10.4% of its
bounding box while protruding 0.21 m ahead of the chassis. The MuJoCo model is
brought along, fixing two faults: it declared a Foot.STL that never existed in
meshes/ (so it could not load) and carried the head as a massless visual geom.

Verified against the export: 22.94804 kg over 19 links, exact; foot positions
agree to 4e-06 m over 200 random in-limit configurations (that residual is the
export rounding one leg's foot offset differently from its own other three);
all 24 joint limits exact; check_urdf clean; and d(foot)/d(q) signs match
main -> 1.3 -> here on all four legs with Jacobian magnitudes identical, which
is what the deployed calibration and policy encode.

TODO(lidar-origin): the mount translation is a flagged placeholder - the export
declares no LiDAR frame and the pod is not a body of revolution, so it is not
recoverable here. Needs the CAD cloud-origin datum.

Co-Authored-By: Claude Opus 5 (1M context) <noreply@anthropic.com>

File: urdf/ayg.urdf (robot description, URDF)
Before this commit: robot ayg, 18 links, 17 joints
Links:
- added link Head, mass 0.72713; collision box size=0.052 0.064 0.064; collision box size=0.053 0.134 0.086
- link Base: mass 11.049 -> 10.732; geometry collision box size=0.423 0.239 0.150; visual mesh filename=package://ayg_description/meshes/Base.STL
- link LF_Hip: mass 1.017 -> 0.98111; geometry collision cylinder length=0.058 radius=0.053; visual mesh filename=package://ayg_description/meshes/LF_Hip.STL
- link LF_Shank: geometry collision box size=0.040 0.017 0.180; collision cylinder length=0.019 radius=0.030
- link LF_Thigh: mass 1.505 -> 1.5051; geometry collision box size=0.052 0.016 0.170; collision cylinder length=0.088 radius=0.055
- link LH_Hip: mass 1.017 -> 0.98111; geometry collision cylinder length=0.058 radius=0.053; visual mesh filename=package://ayg_description/meshes/LH_Hip.STL
- link LH_Shank: geometry collision box size=0.040 0.017 0.180; collision cylinder length=0.019 radius=0.030
- link LH_Thigh: mass 1.505 -> 1.5051; geometry collision box size=0.052 0.016 0.170; collision cylinder length=0.088 radius=0.055
- link RF_Hip: mass 1.017 -> 0.98111; geometry collision cylinder length=0.058 radius=0.053; visual mesh filename=package://ayg_description/meshes/RF_Hip.STL
- link RF_Shank: geometry collision box size=0.040 0.017 0.180; collision cylinder length=0.019 radius=0.030
- link RF_Thigh: mass 1.5051 -> 1.5052; geometry collision box size=0.052 0.016 0.170; collision cylinder length=0.088 radius=0.055
- link RH_Hip: mass 1.017 -> 0.98111; geometry collision cylinder length=0.058 radius=0.053; visual mesh filename=package://ayg_description/meshes/RH_Hip.STL
- link RH_Shank: geometry collision box size=0.040 0.017 0.180; collision cylinder length=0.019 radius=0.030
- link RH_Thigh: mass 1.5051 -> 1.5052; geometry collision box size=0.052 0.016 0.170; collision cylinder length=0.088 radius=0.055
Joints:
- added joint Base_2_Head: type fixed, parent Base, child Head, origin xyz=0.199 0 0.05 rpy=0 0 0, axis 0 0 0
- joint LF_HAA: origin xyz=0.2105 0.054 0 rpy=0 0 0 -> xyz=0.203 0.054 0 rpy=0 0 0
- joint LF_HFE: limit lower=-1.2625 upper=3.0761 effort=50.0 velocity=10.0 -> lower=-2.0412 upper=3.3693 effort=50.0 velocity=10.0; origin xyz=0.065 0.0235 0 rpy=0 0 0 -> xyz=0.063 0.0996 0 rpy=0 0 0
- joint LF_KFE: limit lower=-0.56374 upper=1.4015 effort=50.0 velocity=10.0 -> lower=-0.56374 upper=1.4085 effort=50.0 velocity=10.0; origin xyz=-0.15715 0.057018 -0.20082 rpy=0 0 0 -> xyz=-0.15715 -0.0035 -0.20082 rpy=0 0 0
- joint LF_Shank_2_Foot: origin xyz=0.17048 0.015582 -0.18964 rpy=0 0 0 -> xyz=0.170476 0 -0.189639 rpy=0 0 0
- joint LH_HAA: axis -1 0 0 -> 1 0 0; origin xyz=-0.2105 0.054 0 rpy=0 0 3.141592653589793 -> xyz=-0.203 0.054 0 rpy=0 0 0
- joint LH_HFE: limit lower=-2.2907 upper=2.0479 effort=50.0 velocity=10.0 -> lower=-2.8266 upper=2.5839 effort=50.0 velocity=10.0; origin xyz=0.065 -0.0235 0 rpy=0 0 3.141592653589793 -> xyz=-0.063 0.0996 0 rpy=0 0 0
- joint LH_KFE: limit lower=-0.56374 upper=1.4015 effort=50.0 velocity=10.0 -> lower=-0.56374 upper=1.4085 effort=50.0 velocity=10.0; origin xyz=-0.15715 0.057018 -0.20082 rpy=0 0 0 -> xyz=-0.15715 -0.0035 -0.20082 rpy=0 0 0
- joint LH_Shank_2_Foot: origin xyz=0.17048 0.015582 -0.18964 rpy=0 0 0 -> xyz=0.170476 0 -0.189639 rpy=0 0 0
- joint RF_HAA: origin xyz=0.2105 -0.054 0 rpy=0 0 0 -> xyz=0.203 -0.054 0 rpy=0 0 0
- joint RF_HFE: limit lower=-1.2625 upper=3.0761 effort=50.0 velocity=10.0 -> lower=-2.0412 upper=3.3693 effort=50.0 velocity=10.0; origin xyz=0.065 -0.0235 0 rpy=0 0 0 -> xyz=0.063 -0.0996 0 rpy=0 0 0
- joint RF_KFE: limit lower=-0.56374 upper=1.4015 effort=50.0 velocity=10.0 -> lower=-0.56374 upper=1.4085 effort=50.0 velocity=10.0; origin xyz=-0.15715 -0.057037 -0.20082 rpy=0 0 0 -> xyz=-0.15715 0.0035 -0.20082 rpy=0 0 0
- joint RF_Shank_2_Foot: origin xyz=0.170476 -0.0155635 -0.189639 rpy=0 0 0 -> xyz=0.170476 0 -0.189639 rpy=0 0 0
- joint RH_HAA: axis -1 0 0 -> 1 0 0; origin xyz=-0.2105 -0.054 0 rpy=0 0 3.141592653589793 -> xyz=-0.203 -0.054 0 rpy=0 0 0
- joint RH_HFE: limit lower=-2.2907 upper=2.0479 effort=50.0 velocity=10.0 -> lower=-2.8266 upper=2.5839 effort=50.0 velocity=10.0; origin xyz=0.065 0.0235 0 rpy=0 0 3.141592653589793 -> xyz=-0.063 -0.0996 0 rpy=0 0 0
- joint RH_KFE: limit lower=-0.56374 upper=1.4015 effort=50.0 velocity=10.0 -> lower=-0.56374 upper=1.4085 effort=50.0 velocity=10.0; origin xyz=-0.15715 -0.057037 -0.20082 rpy=0 0 0 -> xyz=-0.15715 0.0035 -0.20082 rpy=0 0 0
- joint RH_Shank_2_Foot: origin xyz=0.170476 -0.0155635 -0.189639 rpy=0 0 0 -> xyz=0.170476 0 -0.189639 rpy=0 0 0

File: urdf/ayg.xacro (robot description, xacro)
@@ -7,6 +7,8 @@
   <xacro:arg name="gazebo_version" default="fortress" />
   <xacro:property name="gazebo_version" value="$(arg gazebo_version)" />
-  <xacro:arg name="camera" default="False" />
-  <xacro:property name="camera" default="$(arg camera)" />
+  <!-- Ayg 1.3 replaced the D555 depth camera with a LiDAR on a new front mount;
+       the argument follows the hardware. -->
+  <xacro:arg name="lidar" default="False" />
+  <xacro:property name="lidar" default="$(arg lidar)" />
   <xacro:arg name="initial_configuration" default="lying_down" />
   <xacro:property name="initial_configuration" value="$(arg initial_configuration)" />
@@ -37,20 +39,20 @@
     name="Base">
     <inertial>
-      <!-- Ayg 1.3 SolidWorks export. Batteries are rigidly fixed inside the
-           chassis and are lumped into this Base mass/inertia (no separate
-           Battery links), so the trunk is a single rigid body. Total robot
-           mass ~23 kg. -->
+      <!-- Ayg 1.3 SolidWorks export CF-AYG-1.3-00-000-URDF-6. Batteries are
+           rigidly fixed inside the chassis and are lumped into this Base
+           mass/inertia (no separate Battery links), so the trunk is a single
+           rigid body. Whole-robot mass 22.948 kg across 19 links. -->
       <origin
-        xyz="-0.0030682 -4.5608E-05 -0.0023186"
+        xyz="-0.00030633 -0.0051482 -0.0019103"
         rpy="0 0 0" />
       <mass
-        value="11.049" />
+        value="10.732" />
       <inertia
-        ixx="0.032662"
-        ixy="-2.5713E-06"
-        ixz="6.2419E-05"
-        iyy="0.034773"
-        iyz="-2.217E-06"
-        izz="0.054917" />
+        ixx="0.029884"
+        ixy="4.1808E-07"
+        ixz="0.00015159"
+        iyy="0.038536"
+        iyz="1.5415E-07"
+        izz="0.055747" />
     </inertial>
     <visual>
@@ -68,14 +70,15 @@
       </material>
     </visual>
-    <!-- Trunk collision: axis-aligned box wrapping the Base mesh body (AABB
-         0.444 x 0.239 x 0.187 centred at z=0.0055). Height is kept to the main
-         body (0.14); the narrow top mount rail (z up to 0.099, only +/-0.06
-         wide) is left out so the box does not over-claim empty space beside it. -->
+    <!-- Trunk collision: axis-aligned box wrapping the Base mesh body. Measured
+         AABB is 0.423 x 0.239 x 0.180 (x -0.2125..0.2105, y +/-0.1195,
+         z -0.088..0.092), but everything above z=0.062 is a single 8 mm rear tab
+         at x~-0.208, so the box stops there (z -0.088..0.062, centred -0.013)
+         rather than over-claiming the empty space beside the tab. -->
     <collision>
       <origin
-        xyz="0 0 0.0"
+        xyz="-0.001 0 -0.013"
         rpy="0 0 0" />
       <geometry>
-        <box size="0.44 0.239 0.122" />
+        <box size="0.423 0.239 0.150" />
       </geometry>
     </collision>
@@ -96,8 +99,8 @@
       <inertia
         ixx="4.0133E-08"
-        ixy="-6.9859E-14"
+        ixy="-6.9855E-14"
         ixz="8.9554E-12"
         iyy="5.9906E-08"
-        iyz="-1.4567E-14"
+        iyz="-1.4564E-14"
         izz="9.917E-08" />
     </inertial>
@@ -117,6 +120,8 @@
   </joint>
   <xacro:include filename="$(find ayg_description)/urdf/legs.xacro" />
-  <xacro:if value="${camera}">
-    <xacro:include filename="$(find ayg_description)/urdf/camera.xacro" />
-  </xacro:if>
+  <!-- Unconditional: unlike the optional D555 it replaces, the 1.3 head is
+       structural chassis (0.72713 kg fixed to Base, reaching 0.425 m forward).
+       Leaving it out would hand ayg_kindyn/Pinocchio a robot missing that mass
+       and its pitch moment. The `lidar` arg inside gates only the sensor frame. -->
+  <xacro:include filename="$(find ayg_description)/urdf/lidar.xacro" />
 </robot>

File: urdf/ayg_sim_ros2_control.xacro (robot description, xacro)
@@ -30,31 +30,55 @@
             </xacro:if>
         </hardware>
+        <!--
+            Ayg 1.3 poses. Both were re-solved for the 0.510 m leg (was 0.443 m);
+            the 1.2 values no longer produce the pose they are named after. In this
+            convention front and hind take the SAME joint values to reach the same
+            leg pose in the Base frame (both thigh frames are Base-aligned), so the
+            legs no longer need front/hind-specific numbers.
+            lying_down: knee near its 1.4085 limit, hip folded so the foot sits
+            under the HFE (foot 3 mm ahead of it). Base 0.1196 m, i.e. 32 mm of
+            belly clearance under the trunk collision box - folded as far as the
+            knee limit allows. The 1.2 values (-0.36/1.09) now leave the base at
+            0.192 m, standing on part-folded legs rather than lying down.
+        -->
         <xacro:if value="${initial_configuration == 'lying_down'}">
-            <xacro:ros2_control_joint joint_name="LF_HAA" effort_lim="${effort_lim}" initial_value="-0.00"/>
-            <xacro:ros2_control_joint joint_name="LF_HFE" effort_lim="${effort_lim}" initial_value="-0.36"/>
-            <xacro:ros2_control_joint joint_name="LF_KFE" effort_lim="${effort_lim}" initial_value=" 1.09"/>
+            <xacro:ros2_control_joint joint_name="LF_HAA" effort_lim="${effort_lim}" initial_value=" 0.00"/>
+            <xacro:ros2_control_joint joint_name="LF_HFE" effort_lim="${effort_lim}" initial_value="-0.70"/>
+            <xacro:ros2_control_joint joint_name="LF_KFE" effort_lim="${effort_lim}" initial_value=" 1.40"/>
             <xacro:ros2_control_joint joint_name="RF_HAA" effort_lim="${effort_lim}" initial_value=" 0.00"/>
-            <xacro:ros2_control_joint joint_name="RF_HFE" effort_lim="${effort_lim}" initial_value="-0.36"/>
-            <xacro:ros2_control_joint joint_name="RF_KFE" effort_lim="${effort_lim}" initial_value=" 1.09"/>
+            <xacro:ros2_control_joint joint_name="RF_HFE" effort_lim="${effort_lim}" initial_value="-0.70"/>
+            <xacro:ros2_control_joint joint_name="RF_KFE" effort_lim="${effort_lim}" initial_value=" 1.40"/>
             <xacro:ros2_control_joint joint_name="LH_HAA" effort_lim="${effort_lim}" initial_value=" 0.00"/>
-            <xacro:ros2_control_joint joint_name="LH_HFE" effort_lim="${effort_lim}" initial_value="-0.48"/>
-            <xacro:ros2_control_joint joint_name="LH_KFE" effort_lim="${effort_lim}" initial_value=" 1.20"/>
+            <xacro:ros2_control_joint joint_name="LH_HFE" effort_lim="${effort_lim}" initial_value="-0.70"/>
+            <xacro:ros2_control_joint joint_name="LH_KFE" effort_lim="${effort_lim}" initial_value=" 1.40"/>
             <xacro:ros2_control_joint joint_name="RH_HAA" effort_lim="${effort_lim}" initial_value=" 0.00"/>
-            <xacro:ros2_control_joint joint_name="RH_HFE" effort_lim="${effort_lim}" initial_value="-0.48"/>
-            <xacro:ros2_control_joint joint_name="RH_KFE" effort_lim="${effort_lim}" initial_value=" 1.20"/>
-        </xacro:if>
+            <xacro:ros2_control_joint joint_name="RH_HFE" effort_lim="${effort_lim}" initial_value="-0.70"/>
+            <xacro:ros2_control_joint joint_name="RH_KFE" effort_lim="${effort_lim}" initial_value=" 1.40"/>
+        </xacro:if>
+        <!--
+            standing: feet directly below their HFE origins at a 0.340 m base
+            height. Solved, not hand-picked: 0.340 is 67% leg extension, the same
+            fraction the 1.2 nominal (0.30 m on a 0.443 m leg) used, so the crouch
+            carries over rather than the number.
+            This replaces the 1.2 all-zeros pose. All-zeros is NOT a standing pose
+            on 1.3: the export's zero configuration now puts the base at 0.4225 m
+            (83% extension, knees near locked) instead of 0.341 m, which is below
+            the 0.3 m Gazebo spawn_height and would drive the feet underground at
+            spawn. The nominal stance height is ultimately a policy/cf_lab
+            decision - treat 0.340 as the geometric carry-over, not a mandate.
+        -->
         <xacro:if value="${initial_configuration == 'standing'}">
-            <xacro:ros2_control_joint joint_name="LF_HAA" effort_lim="${effort_lim}" initial_value="-0.00"/>
-            <xacro:ros2_control_joint joint_name="LF_HFE" effort_lim="${effort_lim}" initial_value="-0.00"/>
-            <xacro:ros2_control_joint joint_name="LF_KFE" effort_lim="${effort_lim}" initial_value=" 0.00"/>
+            <xacro:ros2_control_joint joint_name="LF_HAA" effort_lim="${effort_lim}" initial_value=" 0.00"/>
+            <xacro:ros2_control_joint joint_name="LF_HFE" effort_lim="${effort_lim}" initial_value="-0.2584"/>
+            <xacro:ros2_control_joint joint_name="LF_KFE" effort_lim="${effort_lim}" initial_value=" 0.4485"/>
             <xacro:ros2_control_joint joint_name="RF_HAA" effort_lim="${effort_lim}" initial_value=" 0.00"/>
-            <xacro:ros2_control_joint joint_name="RF_HFE" effort_lim="${effort_lim}" initial_value="-0.00"/>
-            <xacro:ros2_control_joint joint_name="RF_KFE" effort_lim="${effort_lim}" initial_value=" 0.00"/>
+            <xacro:ros2_control_joint joint_name="RF_HFE" effort_lim="${effort_lim}" initial_value="-0.2584"/>
+            <xacro:ros2_control_joint joint_name="RF_KFE" effort_lim="${effort_lim}" initial_value=" 0.4485"/>
             <xacro:ros2_control_joint joint_name="LH_HAA" effort_lim="${effort_lim}" initial_value=" 0.00"/>
-            <xacro:ros2_control_joint joint_name="LH_HFE" effort_lim="${effort_lim}" initial_value="-0.00"/>
-            <xacro:ros2_control_joint joint_name="LH_KFE" effort_lim="${effort_lim}" initial_value=" 0.00"/>
+            <xacro:ros2_control_joint joint_name="LH_HFE" effort_lim="${effort_lim}" initial_value="-0.2584"/>
+            <xacro:ros2_control_joint joint_name="LH_KFE" effort_lim="${effort_lim}" initial_value=" 0.4485"/>
             <xacro:ros2_control_joint joint_name="RH_HAA" effort_lim="${effort_lim}" initial_value=" 0.00"/>
-            <xacro:ros2_control_joint joint_name="RH_HFE" effort_lim="${effort_lim}" initial_value="-0.00"/>
-            <xacro:ros2_control_joint joint_name="RH_KFE" effort_lim="${effort_lim}" initial_value=" 0.00"/>
+            <xacro:ros2_control_joint joint_name="RH_HFE" effort_lim="${effort_lim}" initial_value="-0.2584"/>
+            <xacro:ros2_control_joint joint_name="RH_KFE" effort_lim="${effort_lim}" initial_value=" 0.4485"/>
         </xacro:if>
         <sensor name="imu_sensor">
