Commit message: Rebase the 1.3 model onto SolidWorks export CF-AYG-1.3-00-000-URDF-6
The existing 1.3 commits were built from a 2026-07-04 export; this adopts the
2026-07-16 one, which supersedes it on Base, hips, thighs, the HAA offset,
joint limits and the whole head. Segment lengths are unchanged (thigh = shank =
0.255 m exactly, 0.510 m hip-to-foot), so the leg work carries over - this is a
parts revision, not a new kinematic chain.

legs.xacro is rewritten as one macro instantiated four times with sx/sy sign
parameters, so it reads as a direct transcription of the export and can be
re-checked line by line against a future one. The export's own frame placement
is adopted; the hind pi-yaw is dropped, having existed only so front and hind
could share a hip mesh (the export ships four, differently tessellated). That
removal is behaviour-neutral: HFE/KFE axes are parallel to y, so sliding a
frame along its own rotation axis is kinematically null.

camera.xacro (RealSense D555) becomes lidar.xacro. The head is now
unconditional - it is structural chassis, not an optional payload - so
ayg_kindyn/Pinocchio finally sees its 0.727 kg and forward pitch moment; the
previous flat urdf shipped 18 links with no head at all. That 0.727 kg already
includes the JT128 body (confirmed with the mechanical engineer), so no sensor
mass is added on top. Only lidar_link and the Gazebo gpu_lidar are gated.

Collision primitives were refit by measuring the new meshes rather than scaled:
the HFE motor barrel moved from the hip into the thigh (hip y extent 0.148 ->
0.058), and the head is three boxes because its mesh fills only 10.4% of its
bounding box while protruding 0.21 m ahead of the chassis. The MuJoCo model is
brought along, fixing two faults: it declared a Foot.STL that never existed in
meshes/ (so it could not load) and carried the head as a massless visual geom.

Verified against the export: 22.94804 kg over 19 links, exact; foot positions
agree to 4e-06 m over 200 random in-limit configurations (that residual is the
export rounding one leg's foot offset differently from its own other three);
all 24 joint limits exact; check_urdf clean; and d(foot)/d(q) signs match
main -> 1.3 -> here on all four legs with Jacobian magnitudes identical, which
is what the deployed calibration and policy encode.

TODO(lidar-origin): the mount translation is a flagged placeholder - the export
declares no LiDAR frame and the pod is not a body of revolution, so it is not
recoverable here. Needs the CAD cloud-origin datum.

Co-Authored-By: Claude Opus 5 (1M context) <noreply@anthropic.com>

File: urdf/legs.xacro (robot description, xacro)
@@ -2,28 +2,85 @@
 <robot xmlns:xacro="http://www.ros.org/wiki/xacro">
   <!--
-    Parameterized legs (Ayg 1.3). Two macros, L_Leg / R_Leg, each instantiated
-    for front (FH="F") and hind (FH="H"). Hind legs carry a pi yaw on the HAA and
-    HFE joint origins so that identical joint values mirror the front leg (the net
-    rotation on the thigh/shank frames is 2*pi = identity; the hip frame keeps one
-    pi flip). Joint axes are normalized (HAA about +x world, HFE/KFE about -y
-    world) to match the deployed convention (robstride_ros2_control / calibration /
-    policy). Front and hind reuse the same L_/R_ segment meshes.
-    Inertials/limits are the SolidWorks 1.3 export values mapped into this
-    convention; collision primitives approximate the members (refined in sim).
+    Legs, Ayg 1.3 (SolidWorks export CF-AYG-1.3-00-000-URDF-6).
+    One macro instantiated four times. `sx` = +1 front / -1 hind, `sy` = +1 left /
+    -1 right; every joint origin and mirrored inertia term is written as an export
+    value times those signs, so the file reads as a direct transcription of the
+    export and can be re-checked against a future one line by line.
+    Frames are the export's own placement, unchanged. Axes are normalized to the
+    deployed convention: HAA about +x, HFE/KFE about -y (the export uses +y for
+    HFE/KFE, so those two joints carry a negated axis and correspondingly
+    negated-and-swapped limits). Because the HFE/KFE axes are parallel to y, the
+    export's frame origins sit at an arbitrary point along the rotation axis -
+    sliding them in y is kinematically null, which is why the export's y offsets
+    differ from earlier revisions while the foot positions are identical.
+    Segment lengths: thigh |(-0.15715, -0.20082)| = shank |(0.170476, -0.189639)|
+    = 0.255 m exactly, so the leg extends 0.510 m hip-to-foot (was 0.443 m).
   -->
-  <xacro:macro name="L_Leg" params="FH">
-    <link name="L${FH}_Hip">
-      <inertial>
-        <xacro:if value="${FH == 'F'}">
-          <origin xyz="0.062976 -0.0014435 9.395E-06" rpy="0 0 0" />
-          <mass value="1.017" />
-          <inertia ixx="0.00088413" ixy="1.6599E-05" ixz="5.521E-07"
-                   iyy="0.0014074" iyz="-1.7604E-07" izz="0.00099675" />
+  <xacro:macro name="ayg_leg" params="side FH sx sy">
+    <!-- ============================== Hip ============================== -->
+    <!-- Four distinct hip meshes: front/hind are x-mirrored and left/right are
+         Rx(pi) of each other, and the export tessellates each separately, so no
+         single pair can be reused by rotating a joint frame. -->
+    <link name="${side}${FH}_Hip">
+      <inertial>
+        <origin xyz="${0.059856*sx} ${0.0023868*sy} ${1.6688E-05*sx*sy}" rpy="0 0 0" />
+        <mass value="0.98111" />
+        <inertia ixx="0.00070791" ixy="${1.6598E-06*sx*sy}" ixz="${9.3501E-07*sy}"
+                 iyy="0.0012845"  iyz="${-2.4177E-07*sx}"   izz="0.00087996" />
+      </inertial>
+      <visual>
+        <origin xyz="0 0 0" rpy="0 0 0" />
+        <geometry>
+          <mesh filename="package://ayg_description/meshes/${side}${FH}_Hip.STL" />
+        </geometry>
+        <material name="">
+          <color rgba="0.69804 0.69804 0.69804 1" />
+        </material>
+      </visual>
+      <!-- Rounded hip housing: one cylinder about y. Mesh AABB is
+           0.116 (x) x 0.058 (y) x 0.103 (z); r=0.053 wraps z exactly and leaves
+           the last ~5 mm of each x end uncovered, which is where the HAA flange
+           and the HFE interface sit - both shielded by the neighbouring link. -->
+      <collision>
+        <origin xyz="${0.056*sx} ${-0.004*sy} 0" rpy="${PI/2} 0 0" />
+        <geometry>
+          <cylinder radius="0.053" length="0.058" />
+        </geometry>
+      </collision>
+    </link>
+    <joint name="${side}${FH}_HAA" type="revolute">
+      <origin xyz="${0.203*sx} ${0.054*sy} 0" rpy="0 0 0" />
+      <parent link="Base" />
+      <child link="${side}${FH}_Hip" />
+      <axis xyz="1 0 0" />
+      <!-- Export HAA limits carry over verbatim (axis unchanged). The outward
+           travel differs front vs hind: 0.43633 front, 0.8203 hind. -->
+      <xacro:if value="${side == 'L'}">
+        <limit lower="-0.5236" upper="${0.43633 if FH == 'F' else 0.8203}"
+               effort="${effort_lim}" velocity="${velocity_lim}" />
+      </xacro:if>
+      <xacro:unless value="${side == 'L'}">
+        <limit lower="${-0.43633 if FH == 'F' else -0.8203}" upper="0.5236"
+               effort="${effort_lim}" velocity="${velocity_lim}" />
+      </xacro:unless>
+    </joint>
+    <!-- ============================= Thigh ============================= -->
+    <!-- Front and hind share one mesh per side (LF_Thigh and LH_Thigh are
+         byte-identical in the export, likewise RF/RH), so only L_/R_ are shipped.
+         The thigh now carries the HFE motor barrel: the hip's y extent dropped
+         from 0.148 to 0.058 between revisions and the barrel moved to this link. -->
+    <link name="${side}${FH}_Thigh">
+      <inertial>
+        <xacro:if value="${side == 'L'}">
+          <origin xyz="-0.028374 -0.02602 -0.029622" rpy="0 0 0" />
+          <mass value="1.5051" />
+          <inertia ixx="0.0043448" ixy="0.00034914" ixz="-0.0029698"
+                   iyy="0.0075708" iyz="0.00034106" izz="0.0039222" />
         </xacro:if>
-        <xacro:unless value="${FH == 'F'}">
-          <origin xyz="0.062976 0.0014435 -9.395E-06" rpy="0 0 0" />
-          <mass value="1.017" />
-          <inertia ixx="0.00088413" ixy="-1.6599E-05" ixz="-5.521E-07"
-                   iyy="0.0014074" iyz="-1.7604E-07" izz="0.00099675" />
+        <xacro:unless value="${side == 'L'}">
+          <origin xyz="-0.02838 0.025988 -0.029631" rpy="0 0 0" />
+          <mass value="1.5052" />
+          <inertia ixx="0.0043476" ixy="-0.00034935" ixz="-0.0029719"
+                   iyy="0.0075751" iyz="-0.00034134" izz="0.0039239" />
         </xacro:unless>
       </inertial>
@@ -31,10 +88,5 @@
         <origin xyz="0 0 0" rpy="0 0 0" />
         <geometry>
-          <xacro:if value="${FH == 'F'}">
-            <mesh filename="package://ayg_description/meshes/L_Hip.STL" />
-          </xacro:if>
-          <xacro:unless value="${FH == 'F'}">
-            <mesh filename="package://ayg_description/meshes/R_Hip.STL" />
-          </xacro:unless>
+          <mesh filename="package://ayg_description/meshes/${side}_Thigh.STL" />
         </geometry>
         <material name="">
@@ -42,78 +94,44 @@
         </material>
       </visual>
-      <!-- Hip: cylinder about the Y axis (the HFE motor barrel), wrapping the
-           disc-shaped hip housing. y-offset tracks the HFE side (front vs hind
-           use mirrored hip meshes: F -> L_Hip, H -> R_Hip). -->
-      <collision>
-        <xacro:if value="${FH == 'F'}">
-          <origin xyz="0.065 0.0375 0" rpy="1.5708 0 0" />
-        </xacro:if>
-        <xacro:unless value="${FH == 'F'}">
-          <origin xyz="0.065 -0.0375 0" rpy="1.5708 0 0" />
-        </xacro:unless>
-        <geometry>
-          <cylinder radius="0.055" length="0.14" />
-        </geometry>
-      </collision>
-    </link>
-    <joint name="L${FH}_HAA" type="revolute">
+      <!-- HFE motor barrel: cylinder coaxial with the HFE axis, so it is
+           invariant under hip-flexion and can never self-collide with the hip. -->
+      <collision>
+        <origin xyz="0 ${-0.03205*sy} 0" rpy="${PI/2} 0 0" />
+        <geometry>
+          <cylinder radius="0.055" length="0.088" />
+        </geometry>
+      </collision>
+      <!-- Slim leg member: box pitched about y onto the HFE->KFE line
+           (atan2(-0.15715, -0.20082) = -2.4776 rad), shortened at the knee end
+           where the shank's coaxial knee cylinder takes over. -->
+      <collision>
+        <origin xyz="-0.1121 ${-0.0035*sy} -0.1091" rpy="0 -2.4776 0" />
+        <geometry>
+          <box size="0.052 0.016 0.170" />
+        </geometry>
+      </collision>
+    </link>
+    <joint name="${side}${FH}_HFE" type="revolute">
+      <origin xyz="${0.063*sx} ${0.0996*sy} 0" rpy="0 0 0" />
+      <parent link="${side}${FH}_Hip" />
+      <child link="${side}${FH}_Thigh" />
+      <axis xyz="0 -1 0" />
+      <!-- Export limits negated and swapped for the -y axis:
+           front  (-3.3693, 2.0412) -> (-2.0412, 3.3693)
+           hind   (-2.5839, 2.8266) -> (-2.8266, 2.5839) -->
       <xacro:if value="${FH == 'F'}">
-        <origin xyz="0.2105 0.054 0" rpy="0 0 0" />
+        <limit lower="-2.0412" upper="3.3693" effort="${effort_lim}" velocity="${velocity_lim}" />
       </xacro:if>
       <xacro:unless value="${FH == 'F'}">
-        <origin xyz="-0.2105 0.054 0" rpy="0 0 ${PI}" />
+        <limit lower="-2.8266" upper="2.5839" effort="${effort_lim}" velocity="${velocity_lim}" />
       </xacro:unless>
-      <parent link="Base" />
-      <child link="L${FH}_Hip" />
-      <xacro:if value="${FH == 'F'}">
-        <axis xyz="1 0 0" />
-        <limit lower="-0.5236" upper="0.43633" effort="${effort_lim}" velocity="${velocity_lim}" />
-      </xacro:if>
-      <xacro:unless value="${FH == 'F'}">
-        <axis xyz="-1 0 0" />
-        <limit lower="-0.5236" upper="0.8203" effort="${effort_lim}" velocity="${velocity_lim}" />
-      </xacro:unless>
-    </joint>
-    <link name="L${FH}_Thigh">
-      <inertial>
-        <origin xyz="-0.023305 0.049402 -0.024328" rpy="0 0 0" />
-        <mass value="1.505" />
-        <inertia ixx="0.0030493" ixy="-3.2033E-06" ixz="-0.0016346"
-                 iyy="0.0052191" iyz="-1.6215E-06" izz="0.0026578" />
-      </inertial>
-      <visual>
-        <origin xyz="0 0 0" rpy="0 0 0" />
-        <geometry>
-          <mesh filename="package://ayg_description/meshes/L_Thigh.STL" />
-        </geometry>
-        <material name="">
-          <color rgba="0.69804 0.69804 0.69804 1" />
-        </material>
-      </visual>
-      <!-- Thigh: slim box along the leg, rotated only about the Y swing axis
-           (single pitch, no roll/yaw twist), shortened at both ends for gaps. -->
-      <collision>
-        <origin xyz="-0.105 0.0734 -0.1" rpy="0 -2.4776 0" />
-        <geometry>
-          <box size="0.05 0.014 0.16" />
-        </geometry>
-      </collision>
-    </link>
-    <joint name="L${FH}_HFE" type="revolute">
-      <xacro:if value="${FH == 'F'}">
-        <origin xyz="0.065 0.0235 0" rpy="0 0 0" />
-        <limit lower="-1.2625" upper="3.0761" effort="${effort_lim}" velocity="${velocity_lim}" />
-      </xacro:if>
-      <xacro:unless value="${FH == 'F'}">
-        <origin xyz="0.065 -0.0235 0" rpy="0 0 ${PI}" />
-        <limit lower="-2.2907" upper="2.0479" effort="${effort_lim}" velocity="${velocity_lim}" />
-      </xacro:unless>
-      <parent link="L${FH}_Hip" />
-      <child link="L${FH}_Thigh" />
-      <axis xyz="0 -1 0" />
-    </joint>
-    <link name="L${FH}_Shank">
-      <inertial>
-        <origin xyz="0.081442 0.015569 -0.079562" rpy="0 0 0" />
+    </joint>
+    <!-- ============================= Shank ============================= -->
+    <!-- All four shank meshes are byte-identical in the export, so one Shank.STL
+         serves every leg. The part is unchanged from the previous revision; only
+         its frame slid 15.6 mm along y (the foot now sits at y=0 in this frame). -->
+    <link name="${side}${FH}_Shank">
+      <inertial>
+        <origin xyz="0.081442 -1.3138E-05 -0.079562" rpy="0 0 0" />
         <mass value="0.34563" />
         <inertia ixx="0.0016882" ixy="-5.8149E-12" ixz="0.0015751"
@@ -123,5 +141,5 @@
         <origin xyz="0 0 0" rpy="0 0 0" />
         <geometry>
-          <mesh filename="package://ayg_description/meshes/L_Shank.STL" />
+          <mesh filename="package://ayg_description/meshes/Shank.STL" />
         </geometry>
         <material name="">
@@ -129,40 +147,47 @@
         </material>
       </visual>
-      <!-- Shank: slim box along the leg, rotated only about the Y swing axis
-           (single pitch, no roll/yaw twist), shortened to leave gaps. -->
-      <collision>
-        <origin xyz="0.0867 0.0155 -0.0965" rpy="0 2.4093 0" />
-        <geometry>
-          <box size="0.02 0.017 0.18" />
-        </geometry>
-      </collision>
-      <!-- Knee joint filler: cylinder coaxial with the KFE (y) axis at the
-           joint. Coaxial => invariant under knee bend => bridges the thigh/shank
-           gap for external contacts without ever self-colliding with either. -->
-      <collision>
-        <origin xyz="0 0.0155 0" rpy="1.5708 0 0" />
-        <geometry>
-          <cylinder radius="0.03" length="0.031" />
-        </geometry>
-      </collision>
-    </link>
-    <joint name="L${FH}_KFE" type="revolute">
-      <origin xyz="-0.15715 0.057018 -0.20082" rpy="0 0 0" />
-      <parent link="L${FH}_Thigh" />
-      <child link="L${FH}_Shank" />
+      <!-- Slim leg member: box pitched onto the KFE->foot line
+           (atan2(0.170476, -0.189639) = +2.4094 rad). Widened to 0.040 in the
+           box's x from the 0.020 used for the previous revision: the strut is
+           curved, and 0.020 left the outer ~25 mm of its sweep uncovered. -->
+      <collision>
+        <origin xyz="0.0897 0 -0.0938" rpy="0 2.4094 0" />
+        <geometry>
+          <box size="0.040 0.017 0.180" />
+        </geometry>
+      </collision>
+      <!-- Knee filler: cylinder coaxial with the KFE axis, so it is invariant
+           under knee bend and bridges the thigh/shank gap for external contacts
+           without ever self-colliding with either. Length follows the new knee
+           width (0.018 measured) rather than the old 0.031. -->
+      <collision>
+        <origin xyz="0 0 0" rpy="${PI/2} 0 0" />
+        <geometry>
+          <cylinder radius="0.030" length="0.019" />
+        </geometry>
+      </collision>
+    </link>
+    <joint name="${side}${FH}_KFE" type="revolute">
+      <origin xyz="-0.15715 ${-0.0035*sy} -0.20082" rpy="0 0 0" />
+      <parent link="${side}${FH}_Thigh" />
+      <child link="${side}${FH}_Shank" />
       <axis xyz="0 -1 0" />
-      <limit lower="-0.56374" upper="1.4015" effort="${effort_lim}" velocity="${velocity_lim}" />
-    </joint>
-    <link name="L${FH}_Foot">
+      <!-- Export (-1.4085, 0.56374) negated and swapped for the -y axis. -->
+      <limit lower="-0.56374" upper="1.4085" effort="${effort_lim}" velocity="${velocity_lim}" />
+    </joint>
+    <!-- ============================== Foot ============================= -->
+    <!-- Modelled as primitives rather than the export's Foot mesh: the export's
+         own inertia is exactly that of a solid cylinder r=0.032, L=0.031 about y
+         (iyy = m r^2 / 2 = 2.048E-05, ixx = izz = m r^2 / 4 + m L^2 / 12 =
+         1.3443E-05), so the primitive is the mass model, not an approximation. -->
+    <link name="${side}${FH}_Foot">
       <inertial>
         <origin xyz="0 0 0" rpy="0 0 0" />
         <mass value="0.04" />
         <inertia ixx="1.3443E-05" ixy="0" ixz="0"
-                 iyy="2.048E-05" iyz="0" izz="1.3443E-05" />
-      </inertial>
-      <visual>
-        <!-- Foot: cylinder about the Y axis, replicating the Foot.STL mesh
-             (radius 0.032, length 0.031 spanning y = ±0.0155). -->
-        <origin xyz="0 0 0" rpy="1.5708 0 0" />
+                 iyy="2.048E-05"  iyz="0" izz="1.3443E-05" />
+      </inertial>
+      <visual>
+        <origin xyz="0 0 0" rpy="${PI/2} 0 0" />
         <geometry>
           <cylinder radius="0.032" length="0.031" />
@@ -179,188 +204,14 @@
       </collision>
     </link>
-    <joint name="L${FH}_Shank_2_Foot" type="fixed">
-      <origin xyz="0.17048 0.015582 -0.18964" rpy="0 0 0" />
-      <parent link="L${FH}_Shank" />
-      <child link="L${FH}_Foot" />
+    <joint name="${side}${FH}_Shank_2_Foot" type="fixed">
+      <origin xyz="0.170476 0 -0.189639" rpy="0 0 0" />
+      <parent link="${side}${FH}_Shank" />
+      <child link="${side}${FH}_Foot" />
       <axis xyz="0 0 0" />
     </joint>
   </xacro:macro>
-  <xacro:macro name="R_Leg" params="FH">
-    <link name="R${FH}_Hip">
-      <inertial>
-        <xacro:if value="${FH == 'F'}">
-          <origin xyz="0.062976 0.0014435 -9.395E-06" rpy="0 0 0" />
-          <mass value="1.017" />
-          <inertia ixx="0.00088413" ixy="-1.6599E-05" ixz="-5.521E-07"
-                   iyy="0.0014074" iyz="-1.7604E-07" izz="0.00099675" />
-        </xacro:if>
-        <xacro:unless value="${FH == 'F'}">
-          <origin xyz="0.062976 -0.0014435 9.395E-06" rpy="0 0 0" />
-          <mass value="1.017" />
-          <inertia ixx="0.00088413" ixy="1.6599E-05" ixz="5.521E-07"
-                   iyy="0.0014074" iyz="-1.7604E-07" izz="0.00099675" />
-        </xacro:unless>
-      </inertial>
-      <visual>
-        <origin xyz="0 0 0" rpy="0 0 0" />
-        <geometry>
-          <xacro:if value="${FH == 'F'}">
-            <mesh filename="package://ayg_description/meshes/R_Hip.STL" />
-          </xacro:if>
-          <xacro:unless value="${FH == 'F'}">
-            <mesh filename="package://ayg_description/meshes/L_Hip.STL" />
-          </xacro:unless>
-        </geometry>
-        <material name="">
-          <color rgba="0.69804 0.69804 0.69804 1" />
-        </material>
-      </visual>
-      <!-- Hip: cylinder about the Y axis (the HFE motor barrel), wrapping the
-           disc-shaped hip housing. y-offset tracks the HFE side (front vs hind
-           use mirrored hip meshes: F -> R_Hip, H -> L_Hip). Mirror of L_Leg. -->
-      <collision>
-        <xacro:if value="${FH == 'F'}">
-          <origin xyz="0.065 -0.0375 0" rpy="1.5708 0 0" />
-        </xacro:if>
-        <xacro:unless value="${FH == 'F'}">
-          <origin xyz="0.065 0.0375 0" rpy="1.5708 0 0" />
-        </xacro:unless>
-        <geometry>
-          <cylinder radius="0.055" length="0.14" />
-        </geometry>
-      </collision>
-    </link>
-    <joint name="R${FH}_HAA" type="revolute">
-      <xacro:if value="${FH == 'F'}">
-        <origin xyz="0.2105 -0.054 0" rpy="0 0 0" />
-      </xacro:if>
-      <xacro:unless value="${FH == 'F'}">
-        <origin xyz="-0.2105 -0.054 0" rpy="0 0 ${PI}" />
-      </xacro:unless>
-      <parent link="Base" />
-      <child link="R${FH}_Hip" />
-      <xacro:if value="${FH == 'F'}">
-        <axis xyz="1 0 0" />
-        <limit lower="-0.43633" upper="0.5236" effort="${effort_lim}" velocity="${velocity_lim}" />
-      </xacro:if>
-      <xacro:unless value="${FH == 'F'}">
-        <axis xyz="-1 0 0" />
-        <limit lower="-0.8203" upper="0.5236" effort="${effort_lim}" velocity="${velocity_lim}" />
-      </xacro:unless>
-    </joint>
-    <link name="R${FH}_Thigh">
-      <inertial>
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