Commit message: Match main's sensor-inclusion defaults
main declared the camera arg default True and its committed ayg.urdf therefore
contained the Camera link and its four optical frames. The lidar arg was
defaulting False, so the flat urdf shipped without lidar_link - a structural
difference from main beyond the robot's specification. Default is now True and
ayg.urdf is regenerated with the README's plain command, as main's was.

Also trims process narrative from lidar.xacro, keeping the mount derivation.

Co-Authored-By: Claude Opus 5 (1M context) <noreply@anthropic.com>

File: urdf/ayg.urdf (robot description, URDF)
Before this commit: robot ayg, 19 links, 18 joints
Links:
- added link lidar_link, mass 1e-6
Joints:
- added joint Head_2_lidar: type fixed, parent Head, child lidar_link, origin xyz=0.1438523076923077 0.0 -0.05993846153846154 rpy=-1.965587446494658 0 -1.5707963267948966, axis 0 0 0

File: urdf/ayg.xacro (robot description, xacro)
@@ -8,6 +8,6 @@
   <xacro:property name="gazebo_version" value="$(arg gazebo_version)" />
   <!-- Ayg 1.3 replaced the D555 depth camera with a LiDAR on a new front mount;
-       the argument follows the hardware. -->
-  <xacro:arg name="lidar" default="False" />
+       the argument follows the hardware. Default True, as `camera` was. -->
+  <xacro:arg name="lidar" default="True" />
   <xacro:property name="lidar" default="$(arg lidar)" />
   <xacro:arg name="initial_configuration" default="lying_down" />

File: urdf/lidar.xacro (robot description, xacro)
@@ -8,11 +8,5 @@
     The `Head` link is the mount, taken verbatim from the SolidWorks export
     CF-AYG-1.3-00-000-URDF-6. Its 0.72713 kg ALREADY INCLUDES the LiDAR body
-    (confirmed with the mechanical engineer, 2026-08-03) - do not add sensor mass
-    on top. Corroborating evidence, if this is ever revisited: the export's
-    inertia convention is provably uniform-density-solid-at-CoM (the Foot's
-    inertia is exactly that of a cylinder r=0.032 L=0.031), yet Head's reported
-    inertia is only 0.42-0.70x the uniform solid of its own mesh while its CoM
-    matches that mesh's centroid to 0.13 mm - i.e. a multi-material assembly with
-    the mass packed into the forward pod, which is where the sensor sits.
+    (confirmed with the mechanical engineer) - do not add sensor mass on top.
     The link is named `Head` (the export's name), not `Camera` as the D555 era
     used. Anything that referenced the old body name must follow - notably
@@ -30,11 +24,8 @@
        47.84 mm -> further to the point-cloud origin               (manual Fig 5)
       155.84 mm -> total, Head origin to the cloud origin
-    Cross-check against the head geometry, which was measured before any of these
-    numbers were known: the sensor is 73 mm tall, so its dome tip lands at
-    x = 0.1671 in the Head frame, and the head's nose aperture starts at
-    x = 0.1660 and is 64.3 mm wide against the 62.5 mm dome. The nose is the
-    line-of-sight opening in front of the dome, with ~0.9 mm clearance per side.
-    An independent planar-patch search of Head.STL also found a face normal at
-    22.44 deg, matching the 22.62 deg above.
+    Consistency check: the sensor is 73 mm tall, so its dome tip lands at
+    x = 0.1671 in the Head frame, where the head's nose aperture starts
+    (x = 0.1660) and is 64.3 mm wide against the 62.5 mm dome - the nose is the
+    line-of-sight opening in front of the dome.
   -->
   <xacro:property name="lidar_pitch" value="${atan2(5.0, 12.0)}"/>
@@ -53,9 +44,8 @@
       X_s = Y_s x Z_s                         = ( 0,        -1,  0       )
     which is rpy = (-(pi/2 + pitch), 0, -pi/2) exactly.
-    NOTE this supersedes an earlier guess that azimuth 0 was robot-forward (a
-    bare -pi/2 yaw). It is not: azimuth 0 points DOWN-and-slightly-rearward, so
-    the roll term is required. Getting this wrong rotates the whole cloud about
-    the sensor's own axis. Do NOT negate azimuths to compensate for anything -
-    that mirrors the cloud (see ros/src/ayg_lidar/README.md).
+    Azimuth 0 points down-and-slightly-rearward, not robot-forward, so the roll
+    term is required: a bare -pi/2 yaw would rotate the whole cloud about the
+    sensor axis. Do NOT negate azimuths to compensate - that mirrors the cloud
+    (see ros/src/ayg_lidar/README.md).
   -->
   <xacro:property name="lidar_roll" value="${-(M_PI/2 + lidar_pitch)}"/>

Commit message: collision: one cylinder per hip, one for the LiDAR, smaller handle box
Fixes the AYG 1.3 self-collisions that terminated every training episode at
step 1 (base_contact and head_contact both 1.0000):

  Base <-> hind thigh   1.50 mm interpenetration at the zero pose
  Head <-> front hip    7.50 mm, in every pose

Both were wrapper artifacts. The real meshes clear by 10.4 mm and 2.0 mm
respectively at every joint configuration, so nothing here is a hardware
constraint.

  hip     merged the L=0.058 hip cylinder and the thigh's L=0.088 HFE barrel
          into one cylinder per hip (the pre-1.3 arrangement; combined span
          0.145 against 1.2's 0.148). r 0.053 -> 0.047 with the axis dropped
          4.5 mm, so the terrain-facing underside stays covered and only the
          shielded top gives way. x 0.056 -> 0.058 clears the Base box at both
          ends (the box is not centred: +0.2105 front, -0.2125 rear).
  thigh   keeps only the slim leg member.
  handle  8 mm thick x 90 mm wide, the measured plate, instead of 12.5 x 110.
          Seated 4 mm up so its top face is flush with the Base box top
          surface: under HAA the hip cylinder's inboard end swings to z=+0.0534,
          inside the plate's true 0.0500..0.0580 band, so thinning alone cannot
          clear it.
  LiDAR   pod + nose boxes -> one cylinder on the CAD spin axis (12/13, 0,
          -5/13), r 0.033 covering the O62.5 mm dome and the 64.3 mm aperture,
          spanning 0.132..0.235 along the axis. 823 -> 352 cm3. It starts at
          0.132 rather than the 0.108 mount face because a cylinder reaching
          the mount face overlaps the front hips at every HAA angle.

28 -> 23 collision primitives. Verified clean at the zero pose, across every
single-joint limit, and across the full HAA range on both front legs; the only
remaining contacts are legitimate extreme folds (Base<->Thigh at HAA limits,
Base<->Foot and Foot<->Hip at full knee fold).

mujoco/ayg.xml kept in step; ayg.urdf regenerated from xacro in the container.

Co-Authored-By: Claude Opus 5 (1M context) <noreply@anthropic.com>

File: urdf/ayg.urdf (robot description, URDF)
Before this commit: robot ayg, 20 links, 19 joints
Links:
- link Head: geometry collision box size=0.226 0.090 0.008; collision cylinder length=0.10299999999999998 radius=0.033
- link LF_Hip: geometry collision cylinder length=0.145 radius=0.047; visual mesh filename=package://ayg_description/meshes/LF_Hip.STL
- link LF_Thigh: geometry collision box size=0.052 0.016 0.170; visual mesh filename=package://ayg_description/meshes/L_Thigh.STL
- link LH_Hip: geometry collision cylinder length=0.145 radius=0.047; visual mesh filename=package://ayg_description/meshes/LH_Hip.STL
- link LH_Thigh: geometry collision box size=0.052 0.016 0.170; visual mesh filename=package://ayg_description/meshes/L_Thigh.STL
- link RF_Hip: geometry collision cylinder length=0.145 radius=0.047; visual mesh filename=package://ayg_description/meshes/RF_Hip.STL
- link RF_Thigh: geometry collision box size=0.052 0.016 0.170; visual mesh filename=package://ayg_description/meshes/R_Thigh.STL
- link RH_Hip: geometry collision cylinder length=0.145 radius=0.047; visual mesh filename=package://ayg_description/meshes/RH_Hip.STL
- link RH_Thigh: geometry collision box size=0.052 0.016 0.170; visual mesh filename=package://ayg_description/meshes/R_Thigh.STL

File: urdf/legs.xacro (robot description, xacro)
@@ -38,12 +38,31 @@
         </material>
       </visual>
-      <!-- Rounded hip housing: one cylinder about y. Mesh AABB is
-           0.116 (x) x 0.058 (y) x 0.103 (z); r=0.053 wraps z exactly and leaves
-           the last ~5 mm of each x end uncovered, which is where the HAA flange
-           and the HFE interface sit - both shielded by the neighbouring link. -->
-      <collision>
-        <origin xyz="${0.056*sx} ${-0.004*sy} 0" rpy="${PI/2} 0 0" />
-        <geometry>
-          <cylinder radius="0.053" length="0.058" />
+      <!-- Hip housing AND HFE motor barrel: ONE cylinder about y, spanning the
+           whole HAA-to-HFE assembly (hip mesh y -0.0331..0.0250, barrel y
+           0.0235..0.1116 -> 0.0393 +/- 0.0725). This is the pre-1.3 arrangement:
+           the barrel is coaxial with the HFE axis, so carrying it on the parent
+           link is kinematically identical to carrying it on the thigh, and it
+           keeps one collider per hip instead of two.
+           The housing mesh is symmetric in z (+/-0.0513) but its two sides are
+           not: the top is roofed by the Head deck collider (underside z=+0.0455)
+           and can never touch anything, while the underside faces terrain and is
+           in the base_contact termination list. So the cylinder is r=0.047 with
+           its axis dropped to z=-0.0045 rather than r=0.053 centred: bottom
+           -0.0515 still covers the real underside (-0.0513), top +0.0425 clears
+           the deck by 3 mm. A symmetric shrink to r=0.044 would clear the deck
+           too but leave the exposed underside 7.3 mm short.
+           The last few mm of each x end stay uncovered, which is where the HAA
+           flange and the HFE interface sit - both shielded by the neighbouring
+           link.
+           x=0.058 rather than the mesh centre 0.0591 or the HFE axis 0.063: the
+           Base box is not centred (front face +0.2105, rear face -0.2125), so
+           0.058 is the smallest offset that clears the box at BOTH ends (front
+           3.5 mm, hind 1.5 mm) while still stopping short of the Head pod
+           collider at x=0.312 (4.0 mm). The Base overlap it removes is filtered
+           anyway (parent-child); this only keeps the wrappers visually honest. -->
+      <collision>
+        <origin xyz="${0.058*sx} ${0.0393*sy} -0.0045" rpy="${PI/2} 0 0" />
+        <geometry>
+          <cylinder radius="0.047" length="0.145" />
         </geometry>
       </collision>
@@ -69,6 +88,6 @@
          geometrically identical in the export, likewise RF/RH), so only L_/R_
          are shipped.
-         The thigh now carries the HFE motor barrel: the hip's y extent dropped
-         from 0.148 to 0.058 between revisions and the barrel moved to this link. -->
+         The HFE motor barrel lives on the hip link (one cylinder for the whole
+         HAA-to-HFE assembly), so the thigh carries only the slim leg member. -->
     <link name="${side}${FH}_Thigh">
       <inertial>
@@ -95,12 +114,4 @@
         </material>
       </visual>
-      <!-- HFE motor barrel: cylinder coaxial with the HFE axis, so it is
-           invariant under hip-flexion and can never self-collide with the hip. -->
-      <collision>
-        <origin xyz="0 ${-0.03205*sy} 0" rpy="${PI/2} 0 0" />
-        <geometry>
-          <cylinder radius="0.055" length="0.088" />
-        </geometry>
-      </collision>
       <!-- Slim leg member: box pitched about y onto the HFE->KFE line
            (atan2(-0.15715, -0.20082) = -2.4776 rad), shortened at the knee end

File: urdf/lidar.xacro (robot description, xacro)
@@ -51,4 +51,20 @@
   <xacro:property name="lidar_roll" value="${-(M_PI/2 + lidar_pitch)}"/>
   <xacro:property name="lidar_yaw" value="${-M_PI/2}"/>
+  <!--
+    Collision cylinder for the sensor + its aperture shroud, coaxial with the
+    spin axis (see the Head link below). Distances are along that axis from the
+    Head origin, same convention as the mount geometry above.
+      0.132 -> where the bracket's near-axis material starts (measured); the
+               CAD mount face at 0.108 is further in, shrouded by the cage and
+               close enough to the front hips that a cylinder reaching it
+               overlaps them at every HAA angle
+      0.235 -> front of the aperture shroud
+      0.033 -> covers the O62.5 mm dome (r 0.03125) and the 64.3 mm aperture
+               (r 0.03215)
+  -->
+  <xacro:property name="lidar_col_s0" value="0.132"/>
+  <xacro:property name="lidar_col_s1" value="0.235"/>
+  <xacro:property name="lidar_col_r" value="0.033"/>
+  <xacro:property name="lidar_col_mid" value="${(lidar_col_s0 + lidar_col_s1)/2}"/>
   <!--
     Massless reference frame for TF purposes only. An explicit epsilon-mass
@@ -86,33 +102,60 @@
     </visual>
     <!--
-      Collision as three boxes rather than one. The head mesh fills only 10.4% of
-      its 0.226 x 0.134 x 0.116 bounding box (it is an open bracket cage with a
-      pod at the front), so a single wrapping box would claim a great deal of
-      empty space on a part that now protrudes 0.21 m ahead of the chassis. Since
-      this is the body that strikes obstacles, and near-field obstacle response is
-      the open problem, faithfulness here is worth three primitives.
+      Collision as two primitives, each shaped like the thing it stands for: a
+      box for the carry handle on top, a cylinder for the LiDAR below it. The
+      head mesh fills only 10.4% of its 0.226 x 0.134 x 0.116 bounding box (it
+      is an open bracket cage), so a single wrapping box would claim a great
+      deal of empty space on a part that protrudes 0.21 m ahead of the chassis.
+      Since this is the body that strikes obstacles, and near-field obstacle
+      response is the open problem, shape faithfulness is worth the extra
+      primitive.
       Measured sub-regions, in the Head frame:
-        deck   x 0.000..0.226  y +/-0.055  z -0.0045..0.008
-        pod    x 0.113..0.166  y +/-0.067  z -0.092..-0.006
-        nose   x 0.166..0.218  y +/-0.032  z -0.093..-0.029
-      The thin strut below the deck (x 0.008..0.113, y +/-0.010) is left out: it
-      is tucked under the deck box and is not a plausible contact point.
+        handle x 0.000..0.226  y +/-0.045  z  0.000..0.008
+        cage   x 0.113..0.152  y +/-0.067  z -0.092..-0.006
+        shroud x 0.165..0.230  y +/-0.032  z -0.093..-0.029  (coaxial with the
+               spin axis; its 64.4 mm width is the CAD aperture, 64.3 mm)
+      The thin strut below the handle (x 0.008..0.113, y +/-0.010) is left out:
+      it is tucked under the handle box and is not a plausible contact point.
+      The cage's side walls (|y| 0.033..0.067) are left out too: they are thin
+      sheet either side of the sensor, and wrapping them cost a 611 cm3 box.
+      The top box is the CARRY HANDLE above the LiDAR, sized to the part rather
+      than to the head's bounding box: 8 mm thick (the measured plate is
+      z 0.000..0.008, not the 0.0125 an earlier revision claimed) and y +/-0.045
+      (the two rails and the centre spine span 0.090, not 0.110). It runs the
+      full length of the head, x 0.000..0.226, back to the chassis.
+      It is seated 4 mm ABOVE the measured plate, at Base-frame z 0.0540..0.0620
+      rather than 0.0500..0.0580, so its top face is flush with the Base
+      collision box's top surface (+0.0620). Reason: the handle's rear passes
+      over the two front hips, and Head is a separate rigid body
+      (merge_fixed_joints=False), so Head<->Hip is a non-adjacent pair PhysX
+      leaves active - it feeds both head_contact and base_contact (the hips are
+      in that termination's body list). Under HAA the hip cylinder's inboard end
+      swings up to z=+0.0534, which lands inside the plate's true 0.0500..0.0580
+      band; the cylinder comes up INTO the handle rather than passing under it,
+      so no thinning or narrowing clears it. Lifting the box to start at 0.0540
+      does, across the whole HAA range (-30..+30 deg on both front legs), with
+      0.5 mm to spare over the 0.0535 boundary - and without shortening the
+      handle or shrinking the hip cylinder below the coverage its exposed
+      underside needs.
+      The real parts never touch: Head.STL to LF_Hip.STL holds 2.0 mm at every
+      HAA angle, so this is wrapper-vs-wrapper, not a hardware constraint. The
+      offset trades the plate's lower 4 mm for 4 mm of air beneath the chassis
+      top plane, both shielded approaches.
     -->
     <collision>
-      <origin xyz="0.113 0 0.00175" rpy="0 0 0"/>
+      <origin xyz="0.113 0 0.008" rpy="0 0 0"/>
       <geometry>
-        <box size="0.226 0.110 0.0125"/>
+        <box size="0.226 0.090 0.008"/>
       </geometry>
     </collision>
+    <!-- LiDAR: one cylinder on the spin axis, replacing the pod + nose boxes it
+         used to take (823 -> 352 cm3). rpy sends the cylinder's own +z onto the
+         axis direction (12/13, 0, -5/13); the origin is the span's midpoint
+         measured along that axis from the Head origin. -->
     <collision>
-      <origin xyz="0.1395 0 -0.049" rpy="0 0 0"/>
+      <origin xyz="${lidar_col_mid * cos(lidar_pitch)} 0 ${-lidar_col_mid * sin(lidar_pitch)}"
+              rpy="0 ${M_PI/2 + lidar_pitch} 0"/>
       <geometry>
-        <box size="0.053 0.134 0.086"/>
-      </geometry>
-    </collision>
-    <collision>
-      <origin xyz="0.192 0 -0.061" rpy="0 0 0"/>
-      <geometry>
-        <box size="0.052 0.064 0.064"/>
+        <cylinder radius="${lidar_col_r}" length="${lidar_col_s1 - lidar_col_s0}"/>
       </geometry>
     </collision>
