Commit message: Describe one robot, Ayg 1.3: no version argument, no per-version subtree
The 1.2 model (urdf/1.2, meshes/1.2, mujoco/1.2, config/1.2, ayg1.2.xacro and
its flat URDF) is deleted; it stays on the ayg-1.2 branch. The 1.3 files move
to unversioned paths: meshes/, mujoco/ayg.xml, config/config.rviz,
urdf/{legs,lidar,initial_configuration}.xacro, and urdf/ayg.urdf, regenerated
from urdf/ayg.xacro (element for element the former ayg1.3.urdf, without the
<model_version> tag). ayg1.3.xacro's Base and IMU are now in urdf/ayg.xacro
itself; the version and camera (D555) xacro arguments and the version launch
argument of rviz.launch.py are gone. sim_ros2_control.xacro reads Ayg's
ayg_control/config/gazebo/ayg_sw_controllers.yaml, the controllers file's path
on Ayg's main once the version directories are flattened there.

Co-Authored-By: Claude Opus 5.5 <noreply@anthropic.com>
Claude-Session: https://claude.ai/code/session_01BPTiRWtULNSh3rQggqowaa

File: urdf/ayg.urdf (robot description, URDF)
Before this commit: robot ayg, 20 links, 19 joints
Links:
- link Base: geometry collision box size=0.423 0.239 0.15; visual mesh filename=package://ayg_description/meshes/Base.STL
- link Head: geometry collision box size=0.226 0.090 0.008; collision cylinder length=0.10299999999999998 radius=0.033
- link LF_Hip: geometry collision cylinder length=0.145 radius=0.047; visual mesh filename=package://ayg_description/meshes/LF_Hip.STL
- link LF_Shank: geometry collision box size=0.040 0.017 0.180; collision cylinder length=0.019 radius=0.030
- link LF_Thigh: geometry collision box size=0.052 0.016 0.170; visual mesh filename=package://ayg_description/meshes/L_Thigh.STL
- link LH_Hip: geometry collision cylinder length=0.145 radius=0.047; visual mesh filename=package://ayg_description/meshes/LH_Hip.STL
- link LH_Shank: geometry collision box size=0.040 0.017 0.180; collision cylinder length=0.019 radius=0.030
- link LH_Thigh: geometry collision box size=0.052 0.016 0.170; visual mesh filename=package://ayg_description/meshes/L_Thigh.STL
- link RF_Hip: geometry collision cylinder length=0.145 radius=0.047; visual mesh filename=package://ayg_description/meshes/RF_Hip.STL
- link RF_Shank: geometry collision box size=0.040 0.017 0.180; collision cylinder length=0.019 radius=0.030
- link RF_Thigh: geometry collision box size=0.052 0.016 0.170; visual mesh filename=package://ayg_description/meshes/R_Thigh.STL
- link RH_Hip: geometry collision cylinder length=0.145 radius=0.047; visual mesh filename=package://ayg_description/meshes/RH_Hip.STL
- link RH_Shank: geometry collision box size=0.040 0.017 0.180; collision cylinder length=0.019 radius=0.030
- link RH_Thigh: geometry collision box size=0.052 0.016 0.170; visual mesh filename=package://ayg_description/meshes/R_Thigh.STL

File: urdf/ayg.xacro (robot description, xacro)
@@ -5,20 +5,10 @@
   <xacro:arg name="sim_backend" default="gazebo" />
   <xacro:property name="sim_backend" value="$(arg sim_backend)" />
-  <!-- Which Ayg model to build: "1.2" or "1.3". Selects the whole per-version
-       subtree (root xacro, legs, meshes, mujoco/rviz configs) - see the
-       dispatch include at the bottom of this file.
-       Default mirrors ayg_utils.robot_version.DEFAULT in the Ayg repo. -->
-  <xacro:arg name="version" default="1.2" />
-  <!-- Ayg 1.2's RealSense D555 depth camera. Consumed only by urdf/1.2/*;
-       a harmless no-op when version:=1.3. -->
-  <xacro:arg name="camera" default="True" />
-  <xacro:property name="camera" default="$(arg camera)" />
-  <!-- Ayg 1.3 replaced the D555 depth camera with a LiDAR on a new front
-       mount; the argument follows the hardware. Consumed only by
-       urdf/1.3/*; a harmless no-op when version:=1.2. -->
+  <!-- The LiDAR's sensor frame (lidar_link) on the front head; the head itself
+       is always present. -->
   <xacro:arg name="lidar" default="True" />
   <xacro:property name="lidar" default="$(arg lidar)" />
-  <!-- Payload carried on Base, in kg (Ayg 1.3 only; a no-op when version:=1.2).
-       0 is the bare robot; set it in simulation to test a policy under load. -->
+  <!-- Payload carried on Base, in kg. 0 is the bare robot; set it in
+       simulation to test a policy under load. -->
   <xacro:arg name="payload_mass" default="0.0" />
   <xacro:arg name="initial_configuration" default="lying_down" />
@@ -37,7 +27,4 @@
   <xacro:property name="velocity_lim" value="10.0" />
   <xacro:property name="PI" value="3.1415926535897931" />
-  <!-- $(arg version) substituted as TEXT, not read back through a property:
-       see the dispatch include below for why. -->
-  <model_version>$(arg version)</model_version>
   <xacro:if value="${sim}">
     <xacro:include filename="$(find ayg_description)/urdf/sim_ros2_control.xacro" />
@@ -57,12 +44,120 @@
     />
   </xacro:unless>
-  <!-- Per-version dispatch (Base/IMU/battery/legs/camera-or-lidar): urdf/ayg1.2.xacro
-       or urdf/ayg1.3.xacro, chosen by substituting $(arg version) into the
-       INCLUDE FILENAME, as plain text before xacro ever runs. This must stay a
-       filename substitution and NEVER become a `${version == '1.3'}` xacro:if -
-       xacro coerces xacro:property values that parse as numbers, so a property
-       built from $(arg version) holds the FLOAT 1.3 and an equality check
-       against the string '1.3' silently evaluates false. Confirmed in the
-       container; do not "simplify" this. -->
-  <xacro:include filename="$(find ayg_description)/urdf/ayg$(arg version).xacro" />
+  <!-- ============================ Base and IMU ============================ -->
+  <!-- Unmodelled-hardware allowance. The real robot weighs ~24.8 kg on a scale
+       against this CAD export's 23.809; the difference is the wiring harness and
+       other hardware absent from SolidWorks. It is carried on Base rather than as
+       its own link, with the CAD figures kept separate so the export stays
+       auditable. Set extra_base_mass to 0 for the pure CAD robot.
+       Where the extra mass sits is unknown, so it is modelled as uniform over
+       the Base collision box, centred on the CAD centre of mass: with every
+       position inside the trunk equally likely, that is the expected inertia.
+       Each diagonal term gains m (a^2 + b^2) / 12; the centre of mass and the
+       products of inertia keep their CAD values.
+       The payload_mass xacro arg (default 0) adds a carried load on top of it,
+       modelled the same way: uniform over the Base box at the CAD centre of
+       mass. -->
+  <xacro:property name="base_mass_cad"   value="11.02" />
+  <xacro:property name="extra_base_mass" value="1.0" />
+  <xacro:property name="payload_mass"    value="$(arg payload_mass)" />
+  <xacro:property name="added_base_mass" value="${extra_base_mass + payload_mass}" />
+  <xacro:property name="base_mass"       value="${base_mass_cad + added_base_mass}" />
+  <xacro:property name="base_box_x"      value="0.423" />
+  <xacro:property name="base_box_y"      value="0.239" />
+  <xacro:property name="base_box_z"      value="0.150" />
+  <link
+    name="Base">
+    <inertial>
+      <!-- SolidWorks export CF-AYG-1.3-00-000-URDF-7. Batteries are
+           rigidly fixed inside the chassis and are lumped into this Base
+           mass/inertia (no separate Battery links), so the trunk is a single
+           rigid body. Whole-robot CAD mass 23.809 kg across 20 links. The mass
+           and inertia diagonal below add the extra_base_mass allowance defined
+           above, spread uniformly over the collision box; the
+           origin and products of inertia are the CAD export's. The Base mesh
+           envelope is unchanged from URDF-6, so the collision box below still
+           fits. -->
+      <origin
+        xyz="-0.0005817 -1.9934E-05 -0.0020067"
+        rpy="0 0 0" />
+      <mass
+        value="${base_mass}" />
+      <inertia
+        ixx="${round(0.035479 + added_base_mass * (base_box_y**2 + base_box_z**2) / 12, 6)}"
+        ixy="-3.4801E-06"
+        ixz="8.3812E-05"
+        iyy="${round(0.032555 + added_base_mass * (base_box_x**2 + base_box_z**2) / 12, 6)}"
+        iyz="0.00043953"
+        izz="${round(0.055613 + added_base_mass * (base_box_x**2 + base_box_y**2) / 12, 6)}" />
+    </inertial>
+    <visual>
+      <origin
+        xyz="0 0 0"
+        rpy="0 0 0" />
+      <geometry>
+        <mesh
+          filename="package://ayg_description/meshes/Base.STL" />
+      </geometry>
+      <material
+        name="">
+        <color
+          rgba="0.69804 0.69804 0.69804 1" />
+      </material>
+    </visual>
+    <!-- Trunk collision: axis-aligned box wrapping the Base mesh body. Measured
+         AABB is 0.423 x 0.239 x 0.180 (x -0.2125..0.2105, y +/-0.1195,
+         z -0.088..0.092), but everything above z=0.062 is a single 8 mm rear tab
+         at x~-0.208, so the box stops there (z -0.088..0.062, centred -0.013)
+         rather than over-claiming the empty space beside the tab. -->
+    <collision>
+      <origin
+        xyz="-0.001 0 -0.013"
+        rpy="0 0 0" />
+      <geometry>
+        <box size="${base_box_x} ${base_box_y} ${base_box_z}" />
+      </geometry>
+    </collision>
+  </link>
+  <!-- IMU is a massless-ish reference frame only: it is rigidly fixed to Base,
+       its mesh is inside the chassis (not visible) so no <visual>, and the
+       Gazebo/real IMU sensor is defined on the Base link (see
+       sim_ros2_control.xacro), not on this link. Mass/inertia are the
+       CAD-export values (bare module, ~1.35 g); negligible vs the 24 kg total.
+       URDF-7 moved the module 19 mm down (z -0.00983 -> -0.02883). -->
+  <link
+    name="IMU">
+    <inertial>
+      <origin
+        xyz="-0.00099712 0.00015501 -0.00052021"
+        rpy="0 0 0" />
+      <mass
+        value="0.0013495" />
+      <inertia
+        ixx="4.0133E-08"
+        ixy="-6.9859E-14"
+        ixz="8.9554E-12"
+        iyy="5.9906E-08"
+        iyz="-1.4567E-14"
+        izz="9.917E-08" />
+    </inertial>
+  </link>
+  <joint
+    name="Base_2_IMU"
+    type="fixed">
+    <origin
+      xyz="0 0 -0.02883"
+      rpy="0 0 0" />
+    <parent
+      link="Base" />
+    <child
+      link="IMU" />
+    <axis
+      xyz="0 0 0" />
+  </joint>
+  <xacro:include filename="$(find ayg_description)/urdf/legs.xacro" />
+  <!-- Unconditional: the head is structural chassis (0.81801 kg fixed to
+       Base, reaching 0.425 m forward).
+       Leaving it out would hand ayg_kindyn/Pinocchio a robot missing that mass
+       and its pitch moment. The `lidar` arg inside gates only the sensor frame. -->
+  <xacro:include filename="$(find ayg_description)/urdf/lidar.xacro" />
 </robot>

File: urdf/initial_configuration.xacro (robot description, xacro)
@@ -1,17 +1,13 @@
 <?xml version="1.0"?>
-<!-- Ayg 1.3 initial_configuration poses, included by urdf/sim_ros2_control.xacro
-     (shared file) via filename substitution on $(arg version). -->
+<!-- The initial_configuration poses, included by urdf/sim_ros2_control.xacro. -->
 <robot xmlns:xacro="http://www.ros.org/wiki/xacro">
     <!--
-        Ayg 1.3 poses. Both were re-solved for the 0.510 m leg (was 0.443 m);
-        the 1.2 values no longer produce the pose they are named after. In this
-        convention front and hind take the SAME joint values to reach the same
-        leg pose in the Base frame (both thigh frames are Base-aligned), so the
-        legs no longer need front/hind-specific numbers.
+        Both poses are solved for the 0.510 m leg. Front and hind take the
+        SAME joint values to reach the same leg pose in the Base frame (both
+        thigh frames are Base-aligned).
         lying_down: knee near its 1.4085 limit, hip folded so the foot sits
         under the HFE (foot 3 mm ahead of it). Base 0.1196 m, i.e. 32 mm of
         belly clearance under the trunk collision box - folded as far as the
-        knee limit allows. The 1.2 values (-0.36/1.09) now leave the base at
-        0.192 m, standing on part-folded legs rather than lying down.
+        knee limit allows.
     -->
     <xacro:if value="${initial_configuration == 'lying_down'}">
@@ -31,5 +27,5 @@
     <!--
         standing: the zero pose, feet directly below their HFE origins at a
-        0.4245 m base height (URDF-7; 0.4225 on URDF-6). This is the 1.3
+        0.4245 m base height (URDF-7; 0.4225 on URDF-6). This is the
         nominal stance: it equals the cf_lab training init (every episode
         resets to all-zero joints), it clears the JT128's 0.35 m near-field

File: urdf/legs.xacro (robot description, xacro)
@@ -2,5 +2,5 @@
 <robot xmlns:xacro="http://www.ros.org/wiki/xacro">
   <!--
-    Legs, Ayg 1.3 (SolidWorks export CF-AYG-1.3-00-000-URDF-7).
+    Legs (SolidWorks export CF-AYG-1.3-00-000-URDF-7).
     One macro instantiated four times. `sx` = +1 front / -1 hind, `sy` = +1 left /
     -1 right; every joint origin and mirrored inertia term is written as an export
@@ -41,5 +41,5 @@
         <origin xyz="0 0 0" rpy="0 0 0" />
         <geometry>
-          <mesh filename="package://ayg_description/meshes/1.3/${side}${FH}_Hip.STL" />
+          <mesh filename="package://ayg_description/meshes/${side}${FH}_Hip.STL" />
         </geometry>
         <material name="">
@@ -49,8 +49,8 @@
       <!-- Hip housing AND HFE motor barrel: ONE cylinder about y, spanning the
            whole HAA-to-HFE assembly (hip mesh y -0.0376..0.0250, barrel y
-           0.0215..0.1071 in this frame). This is the pre-1.3 arrangement: the
-           barrel is coaxial with the HFE axis, so carrying it on the parent link
-           is kinematically identical to carrying it on the thigh, and it keeps
-           one collider per hip instead of two.
+           0.0215..0.1071 in this frame). The barrel is coaxial with the HFE
+           axis, so carrying it on the parent link is kinematically identical
+           to carrying it on the thigh, and it keeps one collider per hip
+           instead of two.
            The housing mesh is near-symmetric in z (-0.0520..+0.0513) but its two
            sides are not: the top is roofed by the Head deck collider (underside
@@ -120,5 +120,5 @@
         <origin xyz="0 0 0" rpy="0 0 0" />
         <geometry>
-          <mesh filename="package://ayg_description/meshes/1.3/${side}_Thigh.STL" />
+          <mesh filename="package://ayg_description/meshes/${side}_Thigh.STL" />
         </geometry>
         <material name="">
@@ -172,5 +172,5 @@
         <origin xyz="0 ${0.015582*(sy-1)} 0" rpy="0 0 0" />
         <geometry>
-          <mesh filename="package://ayg_description/meshes/1.3/Shank.STL" />
+          <mesh filename="package://ayg_description/meshes/Shank.STL" />
         </geometry>
         <material name="">

File: urdf/lidar.xacro (robot description, xacro)
@@ -2,7 +2,6 @@
 <robot xmlns:xacro="http://www.ros.org/wiki/xacro">
   <!--
-    Ayg 1.3 front head + LiDAR.
-    Replaces camera.xacro (Intel RealSense D555). The 1.3 chassis carries a HESAI
-    JT128 on a new front mount; ayg_lidar drives it (see ros/src/ayg_lidar) and
+    The front head + LiDAR.
+    The chassis carries a HESAI JT128 on the front mount; ayg_lidar drives it (see ros/src/ayg_lidar) and
     stamps clouds in `lidar_link`.
     The `Head` link is the mount, taken verbatim from the SolidWorks export
@@ -11,7 +10,5 @@
     91 g and moves the CoM 15 mm back and 13 mm up) - do not add sensor mass on
     top. The mount geometry (axis, face distance, Base_2_Head) is unchanged.
-    The link is named `Head` (the export's name), not `Camera` as the D555 era
-    used. Anything that referenced the old body name must follow - notably
-    cf_lab's head-contact termination (body_names="Camera").
+    The link is named `Head`, the export's name.
   -->
   <xacro:property name="M_PI" value="3.1415926535897931"/>
@@ -72,7 +69,6 @@
     Massless reference frame for TF purposes only. An explicit epsilon-mass
     inertial is required because physics simulators (Isaac Sim, Gazebo) silently
-    assign a 1.0 kg default to any link without <inertial>. Across 14 D555
-    reference frames that silently injected +14 kg rigid-fixed to Base - enough
-    to faceplant the AYG locomotion policy in Isaac Lab. Real hardware /
+    assign a 1.0 kg default to any link without <inertial>, which would add a
+    rigid kilogram to Base per frame. Real hardware /
     robot_state_publisher are unaffected (TF-only consumers ignore inertia).
   -->
@@ -97,5 +93,5 @@
       <origin xyz="0 0 0" rpy="0 0 0"/>
       <geometry>
-        <mesh filename="package://ayg_description/meshes/1.3/Head.STL"/>
+        <mesh filename="package://ayg_description/meshes/Head.STL"/>
       </geometry>
       <material name="">
@@ -164,7 +160,6 @@
     </collision>
   </link>
-  <!-- Export Base_2_Head, verbatim. No rotation: unlike the D555 mount, which
-       carried a 90 deg roll to set up the RealSense optical-frame subtree, the
-       head is a plain rigid body and the export places it axis-aligned. -->
+  <!-- Export Base_2_Head, verbatim. No rotation: the head is a plain rigid
+       body and the export places it axis-aligned. -->
   <joint name="Base_2_Head" type="fixed">
     <origin xyz="0.199 0 0.05" rpy="0 0 0"/>
@@ -177,8 +172,6 @@
        structural and always present. -->
   <xacro:if value="${lidar}">
-  <!-- The frame ayg_lidar stamps /lidar/points and /lidar/imu in. Its README
-       states the production stack gets base_link -> lidar_link from the URDF;
-       before 1.3 that TF did not exist anywhere and the bench launch faked it
-       with an identity static_transform_publisher. -->
+  <!-- The frame ayg_lidar stamps /lidar/points_raw and /lidar/imu in; the
+       production stack gets Base -> lidar_link from this URDF. -->
   <xacro:massless_frame name="lidar_link"/>
   <joint name="Head_2_lidar" type="fixed">

File: urdf/sim_ros2_control.xacro (robot description, xacro)
@@ -27,13 +27,9 @@
             <plugin>${system_plugin}</plugin>
             <xacro:if value="${sim_backend == 'mujoco'}">
-                <param name="mujoco_model_path">$(find ayg_description)/mujoco/$(arg version)/ayg.xml</param>
+                <param name="mujoco_model_path">$(find ayg_description)/mujoco/ayg.xml</param>
             </xacro:if>
         </hardware>
-        <!-- initial_configuration poses (lying_down / standing) are per-version:
-             the 1.2 and 1.3 leg geometries need different joint values to reach
-             the same named pose (see each version's file for the derivation).
-             Filename substitution on $(arg version), same convention and same
-             reason as the ayg$(arg version).xacro dispatch in ayg.xacro. -->
-        <xacro:include filename="$(find ayg_description)/urdf/$(arg version)/initial_configuration.xacro" />
+        <!-- initial_configuration poses (lying_down / standing). -->
+        <xacro:include filename="$(find ayg_description)/urdf/initial_configuration.xacro" />
         <sensor name="imu_sensor">
             <state_interface name="orientation.x"/>
@@ -54,8 +50,5 @@
             <gazebo>
                 <plugin filename="libgz_ros2_control-system.so" name="gz_ros2_control::GazeboSimROS2ControlPlugin">
-                    <!-- ayg_control#306 split this config per-version; $(arg version)
-                         text substitution, same convention as the dispatch sites above
-                         (do NOT read this back through a ${...} property). -->
-                    <parameters>$(find ayg_control)/config/$(arg version)/gazebo/ayg_sw_controllers.yaml</parameters>
+                    <parameters>$(find ayg_control)/config/gazebo/ayg_sw_controllers.yaml</parameters>
                 </plugin>
             </gazebo>
