Commit message: Updated camera position, also Updated the camera optical/depth offset

File: urdf/camera.xacro (robot description, xacro)
@@ -33,8 +33,10 @@
     export). The link keeps the name "Camera" so the D555 optical-frame tree,
     Gazebo sensors, realsense2_camera camera_name and all /camera/Camera/* topics
-    are unchanged. The Head mesh is exported base-aligned; because Base_2_Camera
-    carries a +90 deg roll (needed by the optical frames below), the visual and
-    inertial are expressed with a compensating -90 deg roll so the head renders
-    upright. Mass/CoM/inertia are the export Head values rolled into this frame.
+    are unchanged. The Head mesh already bakes in the 15 deg D555 bracket pitch
+    (its front-face normal sits 15 deg below horizontal), so the mount joint must
+    NOT tilt it again. Because Base_2_Camera carries a +90 deg roll (needed by the
+    optical frames below), the visual and inertial are expressed with a compensating
+    -90 deg roll so the head renders as in the CAD. Mass/CoM/inertia are the export
+    Head values rolled into this frame.
   -->
   <link name="Camera">
@@ -68,12 +70,14 @@
     </collision>
   </link>
-  <!-- Ayg 1.3 head mount (export Base_2_Head at 0.257 0 0.095). rpy = +90 deg roll
-       (for the optical-frame subtree below) + 15 deg pitch-down = the physical D555
-       bracket, so the depth/color frames look 15 deg below horizontal. This is the
-       single source of truth for the tilt: Gazebo, Isaac, RViz TF and the real
-       robot all agree (the cf_lab depth-camera prim offset is identity). z=0.095 is
+  <!-- Ayg 1.3 head mount, matches the CAD Base_2_Head (0.257 0 0.095). rpy is a
+       +90 deg roll ONLY (to set up the optical-frame subtree below); it carries NO
+       pitch. The 15 deg D555 bracket pitch is already baked into the Head.STL mesh,
+       so the housing renders tilted straight from the geometry (adding pitch here
+       would double it to 30 deg). The matching 15 deg for the depth/color optical
+       frames is applied once, in Camera_depth_joint. Gazebo, Isaac, RViz TF and the
+       real robot agree (the cf_lab depth-camera prim offset is identity). z=0.095 is
        the CAD-confirmed camera height. -->
   <joint name="Base_2_Camera" type="fixed">
-    <origin xyz="0.257 0 0.095" rpy="1.5708 0.2618 0"/>
+    <origin xyz="0.257 0 0.095" rpy="1.5708 0 0"/>
     <parent link="Base"/>
     <child link="Camera"/>
@@ -81,14 +85,16 @@
   </joint>
   <!--
-    Camera frame post-Base_2_Camera is (X-fwd, Y-up, Z-right) due to the
-    90 deg roll in the parent joint. Camera_depth_frame undoes that roll so
-    the RealSense optical-frame convention (rpy="-pi/2 0 -pi/2" => Z-fwd)
-    works as in realsense2_description, and doubles as the D450 optical-module
-    reference (depth origin = left-IR origin in the module).
-    The xyz=(0.0527 -0.024 0) translation places the depth origin at the
-    optical-module reference inside the housing: +5.27 cm forward and -2.4 cm
-    vertical (down) from the Camera link origin in robot body convention (nominal
+    Camera frame post-Base_2_Camera is (X-fwd, Y-up, Z-right) due to the 90 deg
+    roll in the parent joint. Camera_depth_joint's -pi/2 roll undoes that roll, and
+    its -pi/12 yaw (about this frame's Z = Base "right") pitches the optical subtree
+    15 deg below horizontal; the D555 bracket tilt is applied here ONCE so it is not
+    double-counted with the Head mesh's baked-in tilt. The RealSense optical-frame
+    convention (rpy="-pi/2 0 -pi/2" => Z-fwd) then works as in realsense2_description,
+    and doubles as the D450 optical-module reference (depth origin = left-IR origin).
+    The xyz=(0.0538 -0.0124 0) translation places the depth origin at the
+    optical-module reference inside the housing: +5.38 cm forward and -1.24 cm
+    vertical (down) from the Camera link origin in robot body convention (the
     D555 optical-module offset inside the housing). Camera link's local Y axis is Base +Z
-    (up) due to the 90 deg roll above, so -0.024 along local Y = 2.4 cm down
+    (up) due to the 90 deg roll above, so -0.0124 along local Y = 1.24 cm down
     in body frame; local Z is Base -Y, so 0 leaves the optical module on the
     body centerline.
@@ -103,5 +109,5 @@
   <xacro:massless_frame name="Camera_depth_frame"/>
   <joint name="Camera_depth_joint" type="fixed">
-    <origin xyz="0.0527 -0.024 0" rpy="${-M_PI/2} 0 0"/>
+    <origin xyz="0.0538 -0.0124 0" rpy="${-M_PI/2} 0 ${-M_PI/12}"/>
     <parent link="Camera"/>
     <child link="Camera_depth_frame"/>

Commit message: camera: carry 15° mount tilt into depth/color frames + add 80x60 policy depth sensor

File: urdf/camera.xacro (robot description, xacro)
@@ -11,4 +11,12 @@
   <xacro:property name="M_PI" value="3.1415926535897931"/>
   <xacro:property name="d555_depth_to_color_offset" value="-0.0475"/>
+  <!--
+    Mount-bracket pitch-down. The Camera.STL housing is exported from CAD
+    already tilted 15 deg about the lateral axis (front-face normal measures
+    15.0 deg from link +X), so the tilt must NOT be added to Base_2_Camera
+    (the mesh would double-tilt). It must, however, be carried by the
+    depth/color sensor frames: the optical module tilts with the housing.
+  -->
+  <xacro:property name="d555_mount_tilt" value="${15.0 * M_PI / 180.0}"/>
   <!--
     Massless reference frame for TF purposes only (depth/color/infra/IMU
@@ -87,7 +95,16 @@
     calibrated TF tree at runtime, which supersedes any nominal URDF values.
   -->
+  <!--
+    The yaw component (-d555_mount_tilt, applied about the Camera link's local
+    Z = the robot's lateral axis) pitches the depth frame 15 deg down with the
+    housing. URDF rpy is extrinsic XYZ, so rpy=(-pi/2, 0, -tilt) composes as
+    Rz(-tilt) * Rx(-pi/2): roll into the depth-frame convention first, then
+    tilt in Camera-link coordinates. This matches the Isaac Lab training
+    camera, which spawns at this frame's origin with a 15 deg pitch-down
+    offset (rough_student_env_cfg.py depth_camera offset).
+  -->
   <xacro:massless_frame name="Camera_depth_frame"/>
   <joint name="Camera_depth_joint" type="fixed">
-    <origin xyz="0.0527 -0.024 0" rpy="${-M_PI/2} 0 0"/>
+    <origin xyz="0.0527 -0.024 0" rpy="${-M_PI/2} 0 ${-d555_mount_tilt}"/>
     <parent link="Camera"/>
     <child link="Camera_depth_frame"/>
@@ -167,4 +184,42 @@
   </gazebo>
   <!--
+    Policy depth sensor: the exact camera the vision student was trained with
+    in Isaac Lab (rough_student_env_cfg.py): 80x60 (4:3, ~71 deg vertical FoV),
+    87 deg horizontal FoV, 0.26-9.0 m clip. This is NOT a resize of the
+    640x360 stream above - that sensor is 16:9 (~56 deg VFoV) and physically
+    cannot cover the training image's vertical extent. Sim-only; the real
+    D555 shares the same 16:9 limitation, which is an open sim-to-real gap.
+  -->
+  <gazebo reference="Camera_depth_frame">
+    <sensor name="d555_policy_depth" type="depth_camera">
+      <update_rate>30</update_rate>
+      <topic>camera/Camera/depth/policy_image</topic>
+      <gz_frame_id>Camera_depth_optical_frame</gz_frame_id>
+      <camera>
+        <horizontal_fov>1.5184</horizontal_fov>  <!-- 87 deg -->
+        <lens>
+          <intrinsics>
+            <fx>42.151</fx>
+            <fy>42.151</fy>
+            <cx>40.0</cx>
+            <cy>30.0</cy>
+            <s>0.0</s>
+          </intrinsics>
+        </lens>
+        <image>
+          <width>80</width>
+          <height>60</height>
+          <format>R_FLOAT32</format>
+        </image>
+        <clip>
+          <near>0.26</near>
+          <far>9.0</far>
+        </clip>
+      </camera>
+      <always_on>1</always_on>
+      <visualize>false</visualize>
+    </sensor>
+  </gazebo>
+  <!--
     RGB color sensor. Without this the /camera/Camera/color/image_raw topic
     has no producer in Gazebo (the image reads black). gz_frame_id +

Commit message: camera: add Camera_link + stereo IR frames and sim sensors for cuVSLAM

File: urdf/camera.xacro (robot description, xacro)
@@ -11,4 +11,6 @@
   <xacro:property name="M_PI" value="3.1415926535897931"/>
   <xacro:property name="d555_depth_to_color_offset" value="-0.0475"/>
+  <!-- Stereo IR baseline (D555 datasheet v1.1): infra1 (left) to infra2 (right). -->
+  <xacro:property name="d555_stereo_baseline" value="0.095"/>
   <!--
     Mount-bracket pitch-down. The Camera.STL housing is exported from CAD
@@ -87,11 +89,16 @@
     in body frame; local Z is Base -Y, so 0 leaves the optical module on the
     body centerline.
-    Only the depth and color frames are modeled here (the two Gazebo sensors
-    below reference Camera_depth_frame / Camera_color_frame and publish in the
-    matching *_optical_frame). The infra1/infra2/accel/gyro/imu frames that
-    realsense2_description also declares are omitted: nothing in this repo
-    consumes them in sim, and on real hardware realsense2_camera (launched
-    with camera_name=Camera, see ayg_camera.launch.py) publishes its own
-    calibrated TF tree at runtime, which supersedes any nominal URDF values.
+    The depth, color and stereo-IR (infra1/infra2) frames are modeled here; the
+    accel/gyro/imu frames realsense2_description also declares are omitted since
+    nothing consumes them.
+    This URDF is the SINGLE TF authority for the camera subtree: ayg_camera
+    launches realsense2_camera with publish_tf:=false. Letting the driver publish
+    too would fork the tree — it roots its frames at Camera_link, which has no
+    path to Base, while re-parenting Camera_depth_frame / Camera_color_frame away
+    from this tree. cuVSLAM needs Base -> Camera_infra{1,2}_optical_frame and
+    abort()s outright when the lookup fails, so a forked tree is not survivable.
+    The cost is that the extrinsics here are nominal D450-module values rather
+    than the driver's per-unit calibration; cuVSLAM recovers the precise stereo
+    baseline from camera_info regardless.
   -->
   <!--
@@ -128,4 +135,51 @@
     <parent link="Camera_color_frame"/>
     <child link="Camera_color_optical_frame"/>
+  </joint>
+  <!--
+    Camera_link: the frame realsense2_camera roots its own tree at (it names
+    frames <camera_name>_*, and ayg_camera passes camera_name=Camera). Declared
+    here so any consumer that expects the driver's naming still resolves against
+    Base. On a D4xx optical module camera_link coincides with the depth origin,
+    hence the identity joint (realsense2_camera publishes camera_link ->
+    camera_depth_frame as identity).
+  -->
+  <xacro:massless_frame name="Camera_link"/>
+  <joint name="Camera_link_joint" type="fixed">
+    <origin xyz="0 0 0" rpy="0 0 0"/>
+    <parent link="Camera_depth_frame"/>
+    <child link="Camera_link"/>
+  </joint>
+  <!--
+    Stereo IR pair — the cuVSLAM input (src/ayg_vslam). infra1 is the LEFT
+    imager and IS the depth origin on a D4xx module (the driver publishes
+    camera_link -> camera_infra1_frame as identity), so it sits at
+    Camera_depth_frame. infra2 is the right imager, one baseline away along the
+    depth frame's -Y (frame convention here is X-forward / Y-left / Z-up, so
+    -Y is to the robot's right).
+    Both carry the 15 deg housing tilt for free by hanging off Camera_depth_frame.
+  -->
+  <xacro:massless_frame name="Camera_infra1_frame"/>
+  <joint name="Camera_infra1_joint" type="fixed">
+    <origin xyz="0 0 0" rpy="0 0 0"/>
+    <parent link="Camera_depth_frame"/>
+    <child link="Camera_infra1_frame"/>
+  </joint>
+  <xacro:massless_frame name="Camera_infra1_optical_frame"/>
+  <joint name="Camera_infra1_optical_joint" type="fixed">
+    <origin xyz="0 0 0" rpy="${-M_PI/2} 0 ${-M_PI/2}"/>
+    <parent link="Camera_infra1_frame"/>
+    <child link="Camera_infra1_optical_frame"/>
+  </joint>
+  <xacro:massless_frame name="Camera_infra2_frame"/>
+  <joint name="Camera_infra2_joint" type="fixed">
+    <origin xyz="0 ${-d555_stereo_baseline} 0" rpy="0 0 0"/>
+    <parent link="Camera_depth_frame"/>
+    <child link="Camera_infra2_frame"/>
+  </joint>
+  <xacro:massless_frame name="Camera_infra2_optical_frame"/>
+  <joint name="Camera_infra2_optical_joint" type="fixed">
+    <origin xyz="0 0 0" rpy="${-M_PI/2} 0 ${-M_PI/2}"/>
+    <parent link="Camera_infra2_frame"/>
+    <child link="Camera_infra2_optical_frame"/>
   </joint>
   <!--
@@ -256,4 +310,58 @@
     </sensor>
   </gazebo>
+  <!--
+    Stereo IR pair for Visual SLAM (src/ayg_vslam -> cuVSLAM). Two mono sensors
+    one baseline apart, sharing intrinsics, so the pair is rectified by
+    construction (identical rotation, pure lateral offset) — which is what
+    cuVSLAM is configured for (rectified_images: true).
+    Topic names match real hardware (realsense2_camera, camera_name=Camera,
+    enable_infra1/2): /camera/Camera/infra{1,2}/image_rect_raw. gz leaves
+    CameraInfo.P at its default, so ayg_gazebo's stereo_camera_info node fixes P
+    up and writes the right camera's Tx = -fx * baseline — see
+    ayg_gazebo/scripts/fix_depth_camera_info.py.
+    The real projector must be OFF for stereo VO (its dot pattern is a
+    camera-fixed texture that corrupts feature tracking); in sim there is no
+    projector, so nothing to disable.
+    Intrinsics deliberately match the depth sensor above (fx=fy=337.2 at
+    640x360, 87 deg HFoV) so sim and hardware present the same geometry.
+  -->
+  <xacro:macro name="infra_sensor" params="name frame optical_frame">
+    <gazebo reference="${frame}">
+      <sensor name="${name}" type="camera">
+        <update_rate>30</update_rate>
+        <topic>camera/Camera/${name}/image_rect_raw</topic>
+        <gz_frame_id>${optical_frame}</gz_frame_id>
+        <camera>
+          <horizontal_fov>1.5184</horizontal_fov>  <!-- 87 deg -->
+          <lens>
+            <intrinsics>
+              <fx>337.2</fx>
+              <fy>337.2</fy>
+              <cx>320.0</cx>
+              <cy>180.0</cy>
+              <s>0.0</s>
+            </intrinsics>
+          </lens>
+          <image>
+            <width>640</width>
+            <height>360</height>
+            <format>L8</format>  <!-- mono8: matches the real IR streams -->
+          </image>
+          <clip>
+            <near>0.1</near>
+            <far>100.0</far>
+          </clip>
+        </camera>
+        <always_on>1</always_on>
+        <visualize>false</visualize>
+      </sensor>
+    </gazebo>
+  </xacro:macro>
+  <xacro:infra_sensor name="infra1"
+                      frame="Camera_infra1_frame"
+                      optical_frame="Camera_infra1_optical_frame"/>
+  <xacro:infra_sensor name="infra2"
+                      frame="Camera_infra2_frame"
+                      optical_frame="Camera_infra2_optical_frame"/>
   </xacro:if>
 </robot>
