Commit message: Add 1 kg unmodelled-hardware allowance to the Ayg 1.3 Base
The real Ayg 1.3 weighs ~24.8 kg on a scale against the CAD export's
23.809 kg. The difference is the wiring harness and other hardware
absent from SolidWorks, spread through the Base interior.

Parameterise the Base mass in urdf/ayg1.3.xacro as
base_mass_cad + extra_base_mass (11.02 + 1.0) and scale the CAD inertia
tensor by base_mass / base_mass_cad, keeping the CAD figure visible and
the correction a single tunable number. The centre of mass is unchanged.
Regenerate urdf/ayg1.3.urdf; the only differences are the Base inertial
block and its comment. Whole-robot mass 23.80928 -> 24.80928 kg.

Ayg 1.2 is untouched.

Co-Authored-By: Claude Fable 5.1 <noreply@anthropic.com>

File: urdf/ayg1.3.urdf (robot description, URDF)
Before this commit: robot ayg, 20 links, 19 joints
Links:
- link Base: mass 11.02 -> 12.02

File: urdf/ayg1.3.xacro (robot description, xacro)
@@ -6,4 +6,16 @@
      dispatcher owns those). -->
 <robot xmlns:xacro="http://www.ros.org/wiki/xacro">
+  <!-- Unmodelled-hardware allowance. The real robot weighs ~24.8 kg on a scale
+       against this CAD export's 23.809; the difference is the wiring harness and
+       other hardware absent from SolidWorks. It is carried on Base rather than as
+       its own link, with the CAD figure kept separate so the export stays
+       auditable. Set extra_base_mass to 0 for the pure CAD robot.
+       The inertia is scaled by the same ratio, which assumes the extra mass is
+       distributed like the existing trunk contents - a lower-bound assumption,
+       since the CAD trunk is battery-heavy and centrally concentrated. -->
+  <xacro:property name="base_mass_cad"      value="11.02" />
+  <xacro:property name="extra_base_mass"    value="1.0" />
+  <xacro:property name="base_mass"          value="${base_mass_cad + extra_base_mass}" />
+  <xacro:property name="base_inertia_scale" value="${base_mass / base_mass_cad}" />
   <link
     name="Base">
@@ -12,19 +24,20 @@
            rigidly fixed inside the chassis and are lumped into this Base
            mass/inertia (no separate Battery links), so the trunk is a single
-           rigid body. Whole-robot mass 23.809 kg across 19 links. The Base
-           mesh envelope is unchanged from URDF-6, so the collision box below
-           still fits. -->
+           rigid body. Whole-robot mass 24.809 kg across 19 links, of which
+           23.809 is the CAD export and 1.0 is the extra_base_mass allowance
+           defined in urdf/ayg1.3.xacro. The Base mesh envelope is unchanged
+           from URDF-6, so the collision box below still fits. -->
       <origin
         xyz="-0.0005817 -1.9934E-05 -0.0020067"
         rpy="0 0 0" />
       <mass
-        value="11.02" />
+        value="${base_mass}" />
       <inertia
-        ixx="0.035479"
-        ixy="-3.4801E-06"
-        ixz="8.3812E-05"
-        iyy="0.032555"
-        iyz="0.00043953"
-        izz="0.055613" />
+        ixx="${0.035479    * base_inertia_scale}"
+        ixy="${-3.4801E-06 * base_inertia_scale}"
+        ixz="${8.3812E-05  * base_inertia_scale}"
+        iyy="${0.032555    * base_inertia_scale}"
+        iyz="${0.00043953  * base_inertia_scale}"
+        izz="${0.055613    * base_inertia_scale}" />
     </inertial>
     <visual>
