Commit message: Restructure ayg_description to carry both Ayg 1.2 and 1.3
Add a version arg (default 1.2) that dispatches, by filename text
substitution, to a per-version root xacro (ayg1.2.xacro / ayg1.3.xacro):
Base/IMU links, the battery macro (1.2 only), legs, and camera/lidar.
sim_ros2_control.xacro (renamed from ayg_sim_ros2_control.xacro) stays
shared, with only the initial_configuration pose blocks split out per
version. Fix the model_version tag, hardcoded to 1.3 on both branches
previously, to track the version arg. Regenerate and commit both flat
URDFs; delete the old unversioned urdf/ayg.urdf. Bump package version
to 2.0.0 and update the README and rviz launch file accordingly.

File: urdf/1.2/camera.xacro (robot description, xacro)
@@ -40,5 +40,5 @@
       <origin xyz="0 0 0" rpy="0 0 0"/>
       <geometry>
-        <mesh filename="package://ayg_description/meshes/Camera.STL"/>
+        <mesh filename="package://ayg_description/meshes/1.2/Camera.STL"/>
       </geometry>
       <material name="">

File: urdf/1.2/legs.xacro (robot description, xacro)
@@ -32,9 +32,9 @@
           <xacro:if value="${FH == 'F'}">
             <mesh
-              filename="package://ayg_description/meshes/L_Hip.STL" />
+              filename="package://ayg_description/meshes/1.2/L_Hip.STL" />
           </xacro:if>
           <xacro:unless value="${FH == 'F'}">
             <mesh
-              filename="package://ayg_description/meshes/R_Hip.STL" />
+              filename="package://ayg_description/meshes/1.2/R_Hip.STL" />
           </xacro:unless>
         </geometry>
@@ -124,5 +124,5 @@
         <geometry>
           <mesh
-            filename="package://ayg_description/meshes/L_Thigh.STL" />
+            filename="package://ayg_description/meshes/1.2/L_Thigh.STL" />
         </geometry>
         <material
@@ -197,5 +197,5 @@
         <geometry>
           <mesh
-            filename="package://ayg_description/meshes/L_Shank.STL" />
+            filename="package://ayg_description/meshes/1.2/L_Shank.STL" />
         </geometry>
         <material
@@ -323,9 +323,9 @@
           <xacro:if value="${FH == 'F'}">
             <mesh
-              filename="package://ayg_description/meshes/R_Hip.STL" />
+              filename="package://ayg_description/meshes/1.2/R_Hip.STL" />
           </xacro:if>
           <xacro:unless value="${FH == 'F'}">
             <mesh
-              filename="package://ayg_description/meshes/L_Hip.STL" />
+              filename="package://ayg_description/meshes/1.2/L_Hip.STL" />
           </xacro:unless>
         </geometry>
@@ -415,5 +415,5 @@
         <geometry>
           <mesh
-            filename="package://ayg_description/meshes/R_Thigh.STL" />
+            filename="package://ayg_description/meshes/1.2/R_Thigh.STL" />
         </geometry>
         <material
@@ -488,5 +488,5 @@
         <geometry>
           <mesh
-            filename="package://ayg_description/meshes/R_Shank.STL" />
+            filename="package://ayg_description/meshes/1.2/R_Shank.STL" />
         </geometry>
         <material

File: urdf/1.3/legs.xacro (robot description, xacro)
@@ -41,5 +41,5 @@
         <origin xyz="0 0 0" rpy="0 0 0" />
         <geometry>
-          <mesh filename="package://ayg_description/meshes/${side}${FH}_Hip.STL" />
+          <mesh filename="package://ayg_description/meshes/1.3/${side}${FH}_Hip.STL" />
         </geometry>
         <material name="">
@@ -120,5 +120,5 @@
         <origin xyz="0 0 0" rpy="0 0 0" />
         <geometry>
-          <mesh filename="package://ayg_description/meshes/${side}_Thigh.STL" />
+          <mesh filename="package://ayg_description/meshes/1.3/${side}_Thigh.STL" />
         </geometry>
         <material name="">
@@ -172,5 +172,5 @@
         <origin xyz="0 ${0.015582*(sy-1)} 0" rpy="0 0 0" />
         <geometry>
-          <mesh filename="package://ayg_description/meshes/Shank.STL" />
+          <mesh filename="package://ayg_description/meshes/1.3/Shank.STL" />
         </geometry>
         <material name="">

File: urdf/1.3/lidar.xacro (robot description, xacro)
@@ -97,5 +97,5 @@
       <origin xyz="0 0 0" rpy="0 0 0"/>
       <geometry>
-        <mesh filename="package://ayg_description/meshes/Head.STL"/>
+        <mesh filename="package://ayg_description/meshes/1.3/Head.STL"/>
       </geometry>
       <material name="">

File: urdf/ayg1.3.urdf (robot description, URDF)
Before this commit: robot ayg, 20 links, 19 joints
Links:
- link Base: geometry collision box size=0.423 0.239 0.150; visual mesh filename=package://ayg_description/meshes/1.3/Base.STL
- link Head: geometry collision box size=0.226 0.090 0.008; collision cylinder length=0.10299999999999998 radius=0.033
- link LF_Hip: geometry collision cylinder length=0.145 radius=0.047; visual mesh filename=package://ayg_description/meshes/1.3/LF_Hip.STL
- link LF_Shank: geometry collision box size=0.040 0.017 0.180; collision cylinder length=0.019 radius=0.030
- link LF_Thigh: geometry collision box size=0.052 0.016 0.170; visual mesh filename=package://ayg_description/meshes/1.3/L_Thigh.STL
- link LH_Hip: geometry collision cylinder length=0.145 radius=0.047; visual mesh filename=package://ayg_description/meshes/1.3/LH_Hip.STL
- link LH_Shank: geometry collision box size=0.040 0.017 0.180; collision cylinder length=0.019 radius=0.030
- link LH_Thigh: geometry collision box size=0.052 0.016 0.170; visual mesh filename=package://ayg_description/meshes/1.3/L_Thigh.STL
- link RF_Hip: geometry collision cylinder length=0.145 radius=0.047; visual mesh filename=package://ayg_description/meshes/1.3/RF_Hip.STL
- link RF_Shank: geometry collision box size=0.040 0.017 0.180; collision cylinder length=0.019 radius=0.030
- link RF_Thigh: geometry collision box size=0.052 0.016 0.170; visual mesh filename=package://ayg_description/meshes/1.3/R_Thigh.STL
- link RH_Hip: geometry collision cylinder length=0.145 radius=0.047; visual mesh filename=package://ayg_description/meshes/1.3/RH_Hip.STL
- link RH_Shank: geometry collision box size=0.040 0.017 0.180; collision cylinder length=0.019 radius=0.030
- link RH_Thigh: geometry collision box size=0.052 0.016 0.170; visual mesh filename=package://ayg_description/meshes/1.3/R_Thigh.STL

File: urdf/ayg1.3.xacro (robot description, xacro)
@@ -1,41 +1,9 @@
 <?xml version="1.0" encoding="utf-8"?>
-<robot name="ayg" xmlns:xacro="http://www.ros.org/wiki/xacro">
-  <xacro:arg name="sim" default="False" />
-  <xacro:property name="sim" default="$(arg sim)" />
-  <xacro:arg name="sim_backend" default="gazebo" />
-  <xacro:property name="sim_backend" value="$(arg sim_backend)" />
-  <xacro:arg name="gazebo_version" default="fortress" />
-  <xacro:property name="gazebo_version" value="$(arg gazebo_version)" />
-  <!-- Ayg 1.3 replaced the D555 depth camera with a LiDAR on a new front mount;
-       the argument follows the hardware. Default True, as `camera` was. -->
-  <xacro:arg name="lidar" default="True" />
-  <xacro:property name="lidar" default="$(arg lidar)" />
-  <xacro:arg name="initial_configuration" default="lying_down" />
-  <xacro:property name="initial_configuration" value="$(arg initial_configuration)" />
-  <xacro:arg name="controller" default="default" />
-  <xacro:property name="controller" default="$(arg controller)" />
-  <xacro:arg name="use_csp" default="false" />
-  <xacro:property name="effort_lim" value="50.0" />
-  <xacro:property name="velocity_lim" value="10.0" />
-  <xacro:property name="PI" value="3.1415926535897931" />
-  <xacro:property name="model_version" value="1.3" />
-  <model_version>${model_version}</model_version>
-  <xacro:if value="${sim}">
-    <xacro:include filename="$(find ayg_description)/urdf/ayg_sim_ros2_control.xacro" />
-  </xacro:if>
-  <xacro:unless value="${sim}">
-    <xacro:include filename="$(find robstride_hardware)/urdf/robstride_ros2_control.xacro"/>
-    <xacro:robstride_ros2_control
-      lf_can_interface="can0"
-      rf_can_interface="can1"
-      lh_can_interface="can2"
-      rh_can_interface="can3"
-      actuator_type="3"
-      default_kp="40.0"
-      default_kd="1.0"
-      use_csp="$(arg use_csp)"
-      calibration_file="$(find robstride_hardware)/calibration/joint_calibration.yaml"
-    />
-  </xacro:unless>
+<!-- Ayg 1.3 per-version root: Base, IMU. No battery links - the 1.3 chassis
+     lumps the batteries into Base (see the mass note below). Included by
+     urdf/ayg.xacro via filename substitution on $(arg version); do not run
+     this file directly (no `sim`/`camera`/etc. args are declared here, the
+     dispatcher owns those). -->
+<robot xmlns:xacro="http://www.ros.org/wiki/xacro">
   <link
     name="Base">
@@ -66,5 +34,5 @@
       <geometry>
         <mesh
-          filename="package://ayg_description/meshes/Base.STL" />
+          filename="package://ayg_description/meshes/1.3/Base.STL" />
       </geometry>
       <material
@@ -124,9 +92,9 @@
       xyz="0 0 0" />
   </joint>
-  <xacro:include filename="$(find ayg_description)/urdf/legs.xacro" />
+  <xacro:include filename="$(find ayg_description)/urdf/1.3/legs.xacro" />
   <!-- Unconditional: unlike the optional D555 it replaces, the 1.3 head is
        structural chassis (0.81801 kg fixed to Base, reaching 0.425 m forward).
        Leaving it out would hand ayg_kindyn/Pinocchio a robot missing that mass
        and its pitch moment. The `lidar` arg inside gates only the sensor frame. -->
-  <xacro:include filename="$(find ayg_description)/urdf/lidar.xacro" />
+  <xacro:include filename="$(find ayg_description)/urdf/1.3/lidar.xacro" />
 </robot>

File: urdf/sim_ros2_control.xacro (robot description, xacro)
@@ -30,56 +30,10 @@
             </xacro:if>
         </hardware>
-        <!--
-            Ayg 1.3 poses. Both were re-solved for the 0.510 m leg (was 0.443 m);
-            the 1.2 values no longer produce the pose they are named after. In this
-            convention front and hind take the SAME joint values to reach the same
-            leg pose in the Base frame (both thigh frames are Base-aligned), so the
-            legs no longer need front/hind-specific numbers.
-            lying_down: knee near its 1.4085 limit, hip folded so the foot sits
-            under the HFE (foot 3 mm ahead of it). Base 0.1196 m, i.e. 32 mm of
-            belly clearance under the trunk collision box - folded as far as the
-            knee limit allows. The 1.2 values (-0.36/1.09) now leave the base at
-            0.192 m, standing on part-folded legs rather than lying down.
-        -->
-        <xacro:if value="${initial_configuration == 'lying_down'}">
-            <xacro:ros2_control_joint joint_name="LF_HAA" effort_lim="${effort_lim}" initial_value=" 0.00"/>
-            <xacro:ros2_control_joint joint_name="LF_HFE" effort_lim="${effort_lim}" initial_value="-0.70"/>
-            <xacro:ros2_control_joint joint_name="LF_KFE" effort_lim="${effort_lim}" initial_value=" 1.40"/>
-            <xacro:ros2_control_joint joint_name="RF_HAA" effort_lim="${effort_lim}" initial_value=" 0.00"/>
-            <xacro:ros2_control_joint joint_name="RF_HFE" effort_lim="${effort_lim}" initial_value="-0.70"/>
-            <xacro:ros2_control_joint joint_name="RF_KFE" effort_lim="${effort_lim}" initial_value=" 1.40"/>
-            <xacro:ros2_control_joint joint_name="LH_HAA" effort_lim="${effort_lim}" initial_value=" 0.00"/>
-            <xacro:ros2_control_joint joint_name="LH_HFE" effort_lim="${effort_lim}" initial_value="-0.70"/>
-            <xacro:ros2_control_joint joint_name="LH_KFE" effort_lim="${effort_lim}" initial_value=" 1.40"/>
-            <xacro:ros2_control_joint joint_name="RH_HAA" effort_lim="${effort_lim}" initial_value=" 0.00"/>
-            <xacro:ros2_control_joint joint_name="RH_HFE" effort_lim="${effort_lim}" initial_value="-0.70"/>
-            <xacro:ros2_control_joint joint_name="RH_KFE" effort_lim="${effort_lim}" initial_value=" 1.40"/>
-        </xacro:if>
-        <!--
-            standing: the zero pose, feet directly below their HFE origins at a
-            0.4245 m base height (URDF-7; 0.4225 on URDF-6). This is the 1.3
-            nominal stance: it equals the cf_lab training init (every episode
-            resets to all-zero joints), it clears the JT128's 0.35 m near-field
-            threshold (sensor at 0.415 m vs 0.330 m at the earlier 0.340 m
-            carry-over), and it holds the lowest static KFE torque of the
-            workable range (9.2 vs 11.4 N*m per leg at the URDF-6 masses).
-            The KFE extension stop still leaves 0.565 rad (7.6 cm of base rise)
-            beyond it. Requires spawn_height above 0.4245 (simulate_ayg uses
-            0.45).
-        -->
-        <xacro:if value="${initial_configuration == 'standing'}">
-            <xacro:ros2_control_joint joint_name="LF_HAA" effort_lim="${effort_lim}" initial_value="0.0"/>
-            <xacro:ros2_control_joint joint_name="LF_HFE" effort_lim="${effort_lim}" initial_value="0.0"/>
-            <xacro:ros2_control_joint joint_name="LF_KFE" effort_lim="${effort_lim}" initial_value="0.0"/>
-            <xacro:ros2_control_joint joint_name="RF_HAA" effort_lim="${effort_lim}" initial_value="0.0"/>
-            <xacro:ros2_control_joint joint_name="RF_HFE" effort_lim="${effort_lim}" initial_value="0.0"/>
-            <xacro:ros2_control_joint joint_name="RF_KFE" effort_lim="${effort_lim}" initial_value="0.0"/>
-            <xacro:ros2_control_joint joint_name="LH_HAA" effort_lim="${effort_lim}" initial_value="0.0"/>
-            <xacro:ros2_control_joint joint_name="LH_HFE" effort_lim="${effort_lim}" initial_value="0.0"/>
-            <xacro:ros2_control_joint joint_name="LH_KFE" effort_lim="${effort_lim}" initial_value="0.0"/>
-            <xacro:ros2_control_joint joint_name="RH_HAA" effort_lim="${effort_lim}" initial_value="0.0"/>
-            <xacro:ros2_control_joint joint_name="RH_HFE" effort_lim="${effort_lim}" initial_value="0.0"/>
-            <xacro:ros2_control_joint joint_name="RH_KFE" effort_lim="${effort_lim}" initial_value="0.0"/>
-        </xacro:if>
+        <!-- initial_configuration poses (lying_down / standing) are per-version:
+             the 1.2 and 1.3 leg geometries need different joint values to reach
+             the same named pose (see each version's file for the derivation).
+             Filename substitution on $(arg version), same convention and same
+             reason as the ayg$(arg version).xacro dispatch in ayg.xacro. -->
+        <xacro:include filename="$(find ayg_description)/urdf/$(arg version)/initial_configuration.xacro" />
         <sensor name="imu_sensor">
             <state_interface name="orientation.x"/>
